File: B3/_autosave-B3.kicad_pcb (KiCad board)
At the start: 4 copper layers, 100 x 100 mm, 86 parts, among them U301 74HC00, U302 74HC125, U303 74HC74, U304 74HC74, U305 74HC74, U306 74HC32, U307 74HC299, U308 74HC193, U309 74HC00, U310 74HC244, U311 74HC377, U312 74HC244, U313 74HC299, U314 74HC32, U315 74HC193, U316 74HC00, U317 74HC74, U318 74HC08, U319 74HC32, U320 74HC00, U321 74HC00, U322 74HC00, U323 74HC00, U324 74HC00, U325 74HC08, U326 74HC08, U327 74HC377, U328 74HC00, U329 74HC00, U330 74HC74, U331 74HC74, U332 74HC74, U333 74HC74, U334 74HC74, U335 74HC04, U336 74HC244, U337 74HC08, U338 74HC32, U339 74HC08

Commit message: .
Connections:
- U309 pad 10: /sdr/sdrController/~{FULL} -> GND
- U309 pad 8: Net-(U309-Pad8) -> unconnected-(U309-Pad8)
- U309 pad 9: /sdr/sdrController/~{WRITE} -> GND
- U311 pad 1: Net-(U309-Pad8) -> Net-(U311-Pad1)
- U325 pad 1: GND -> /sdr/sdrController/~{WRITE}
- U325 pad 2: GND -> /sdr/sdrController/~{FULL}
- U325 pad 3: unconnected-(U325-Pad3) -> Net-(U311-Pad1)
Routing:
- net /sdr/sdrController/~{FULL}: track 79.4 -> 0.00 mm, vias 3 -> 0
- net Net-(U309-Pad8): track 31.8 -> 0.00 mm, vias 2 -> 0
- net /sdr/sdrController/~{WRITE}: track 40.1 -> 20.9 mm, vias 2 -> 0
- net GND: track 79.7 -> 70.0 mm, vias 91 -> 90
- net Net-(U324-Pad11): track 22.9 -> 23.8 mm
- net Net-(U324-Pad3): track 24.1 -> 23.4 mm
