File: B3/B3.kicad_sch (KiCad schematic)
At the start: 0 parts

Commit message: Updates to B3
Parts:
- added U301: 74HC04, Package_SO:SO-14_3.9x8.65mm_P1.27mm, symbol 74xx:74HC04
- added U302: 74HC125, Package_SO:SO-14_3.9x8.65mm_P1.27mm, symbol 74xx:74LS125
- added U316: 74HC00, Package_SO:SO-14_3.9x8.65mm_P1.27mm, symbol 74xx:74HC00
Connections:
- new net PHI2: U301.13
- new net ~{PHI2}: U301.12
Other:
- added sheet power (power.kicad_sch)
- added sheet sdr (sdr.kicad_sch)
- sheet buses ports: added DZ[0..7], D[0..7], ~{EN[0..15]}; removed {DATABUS}, {ENABLEBUS}
- title: (none) -> 74HCT6526 Board 3

Commit message: B3 added. First revision
Still not verified.
Parts:
- removed U301: 74HC04, Package_SO:SO-14_3.9x8.65mm_P1.27mm, symbol 74xx:74HC04
- removed U302: 74HC125, Package_SO:SO-14_3.9x8.65mm_P1.27mm, symbol 74xx:74LS125
Connections:
- net PHI2: now also U316.12, U316.13
- net ~{PHI2}: now also U316.11
Other:
- added sheet icr (icr.kicad_sch)
- moved on the sheet: U316D

Commit message: .
Parts:
- removed U316: 74HC00, Package_SO:SO-14_3.9x8.65mm_P1.27mm, symbol 74xx:74HC00
- added U328: 74HC00, Package_SO:SO-14_3.9x8.65mm_P1.27mm, symbol 74xx:74HC00
Connections:
- net PHI2: now also U328.10, U328.9
- net ~{PHI2}: now also U328.8
Other:
- company: (none) -> Daniel Molina
Changed lines of the file:
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@@
   (title_block
     (title "74HCT6526 Board 3")
-    (date "2022-09-11")
-    (rev "0.1")
+    (date "2022-10-08")
+    (rev "0.1.2")
+    (company "Daniel Molina")
+    (comment 1 "https://github.com/dmolinagarcia/74HCT6526")
   )
   (bus_alias "ENABLEBUS" (members "~{EN[0..15]}"))
+  (bus_alias "CONTROLBUS" (members "TASTART" "CNT" "SP" "PHI2" "~{FLAG}" "TOD" "TAPULSE" "TBPULSE" "TODIRQ" "~{IRQ}" "PB6ON" "PB7ON" "TAOUT" "TBOUT" "SPMODE" "TODIN" "ALARM" "ENABLE_NAND" "TARUNMODE" "~{RES}"))
   (bus_alias "DATABUS" (members "D[0..7]" "DZ[0..7]"))
-  (bus_alias "CONTROLBUS" (members "TASTART" "CNT" "SP" "PHI2" "~{FLAG}" "TOD" "TAPULSE" "TBPULSE" "TODIRQ" "~{IRQ}" "PB6ON" "PB7ON" "TAOUT" "TBOUT" "SPMODE" "TODIN" "ALARM" "ENABLE_NAND" "TARUNMODE" "~{RES}"))
+  (junction (at 83.82 33.02) (diameter 0) (color 0 0 0 0)
+  )
   (junction (at 187.96 20.32) (diameter 0) (color 0 0 0 0)
   )
@@
   )
   (wire (pts (xy 185.42 60.96) (xy 190.5 60.96))
+    (stroke (width 0) (type default) (color 0 0 0 0))
+  )
+  (wire (pts (xy 83.82 33.02) (xy 180.34 33.02))
     (stroke (width 0) (type default) (color 0 0 0 0))
   )
@@
     )
   )
-  (symbol (lib_id "74xx:74HC00") (at 68.58 33.02 0) (unit 4)
-    (in_bom yes) (on_board yes) (fields_autoplaced)
-    (property "Reference" "U316" (id 0) (at 68.58 24.13 0))
-    (property "Value" "74HC00" (id 1) (at 68.58 26.67 0))
+  (symbol (lib_id "74xx:74HC00") (at 68.58 33.02 0) (unit 3)
+    (in_bom yes) (on_board yes)
+    (property "Reference" "U328" (id 0) (at 68.04 28.3383 0))
+    (property "Value" "74HC00" (id 1) (at 68.58 38.1 0))
     (property "Footprint" "Package_SO:SO-14_3.9x8.65mm_P1.27mm" (id 2) (at 68.58 33.02 0)
       (effects (font (size 1.27 1.27)) hide)
@@
       (reference "#PWR0106") (unit 1) (value "GND") (footprint "")
     )
+    (path "/a512fa78-7ea1-40a6-bd2e-d62d1f66c73d/c579a6fd-3fc6-4d69-9825-f95a77e227a6"
+      (reference "#PWR0107") (unit 1) (value "GND") (footprint "")
+    )
     (path "/108743f5-032b-46ed-a6db-6b8bf543e425/19d721ab-3834-4525-89b4-bdad6f6db2b8/69ec6aa9-f040-4049-9991-dcde06a46222"
       (reference "#PWR0301") (unit 1) (value "VCC") (footprint "")
@@
       (reference "#PWR0356") (unit 1) (value "GND") (footprint "")
     )
+    (path "/6ac12df0-6226-4d30-947c-27d74eb345ea/75690eac-5e88-44d0-90e0-6b3ef565756f/0d4d31d7-8229-4110-a32f-5a4c1f2200b4"
+      (reference "#PWR0357") (unit 1) (value "GND") (footprint "")
+    )
+    (path "/6ac12df0-6226-4d30-947c-27d74eb345ea/75690eac-5e88-44d0-90e0-6b3ef565756f/587ee2a1-9687-487f-af89-5a27cf693c01"
+      (reference "#PWR0358") (unit 1) (value "GND") (footprint "")
+    )
+    (path "/6ac12df0-6226-4d30-947c-27d74eb345ea/75690eac-5e88-44d0-90e0-6b3ef565756f/123ad7db-c0aa-4245-857e-98514493bc9e"
+      (reference "#PWR0359") (unit 1) (value "GND") (footprint "")
+    )
     (path "/c7e691f1-3826-4fda-8caf-e0d6c99d6f96/5e5b35b2-2cee-4f8a-a15f-d82163ba3fc5"
       (reference "C301") (unit 1) (value "100n") (footprint "Capacitor_SMD:C_0603_1608Metric")
@@
       (reference "C339") (unit 1) (value "100n") (footprint "Capacitor_SMD:C_0603_1608Metric")
     )
+    (path "/a512fa78-7ea1-40a6-bd2e-d62d1f66c73d/97ba3ce4-cff2-40fa-bd3d-a664d6ce034c"
+      (reference "C340") (unit 1) (value "100n") (footprint "Capacitor_SMD:C_0603_1608Metric")
+    )
     (path "/a512fa78-7ea1-40a6-bd2e-d62d1f66c73d/4cb2fad4-88a7-4b24-a682-b7083f1fbcca"
       (reference "CONTROLBUS3") (unit 1) (value "Conn_02x10_Odd_Even") (footprint "Connector_PinHeader_2.54mm:PinHeader_2x10_P2.54mm_Vertical")
@@
       (reference "U309") (unit 2) (value "74HC00") (footprint "Package_SO:SO-14_3.9x8.65mm_P1.27mm")
     )
-    (path "/108743f5-032b-46ed-a6db-6b8bf543e425/3047b525-dc7f-4569-aaa8-1bacf6f9cf0f/4af2477e-4939-40d4-9201-e9c6bdc27e23"
+    (path "/c7e691f1-3826-4fda-8caf-e0d6c99d6f96/99af0ead-ffba-47bc-b406-5410fdfc2706"
       (reference "U309") (unit 3) (value "74HC00") (footprint "Package_SO:SO-14_3.9x8.65mm_P1.27mm")
     )
@@
       (reference "U316") (unit 3) (value "74HC00") (footprint "Package_SO:SO-14_3.9x8.65mm_P1.27mm")
     )
-    (path "/6f9850af-0677-4e04-b98f-e695a335ba3d"
+    (path "/c7e691f1-3826-4fda-8caf-e0d6c99d6f96/e9e07058-34a8-470c-a7cf-5a2cf0cdddc0"
       (reference "U316") (unit 4) (value "74HC00") (footprint "Package_SO:SO-14_3.9x8.65mm_P1.27mm")
     )
@@
       (reference "U324") (unit 5) (value "74HC00") (footprint "Package_SO:SO-14_3.9x8.65mm_P1.27mm")
     )
-    (path "/c7e691f1-3826-4fda-8caf-e0d6c99d6f96/12008a93-9e90-45cf-8eb7-69a38fab3c70"
+    (path "/108743f5-032b-46ed-a6db-6b8bf543e425/3047b525-dc7f-4569-aaa8-1bacf6f9cf0f/9ba088ea-82d3-474b-84c9-66bdc00bf2be"
       (reference "U325") (unit 1) (value "74HC08") (footprint "Package_SO:SO-14_3.9x8.65mm_P1.27mm")
     )
@@
       (reference "U328") (unit 2) (value "74HC00") (footprint "Package_SO:SO-14_3.9x8.65mm_P1.27mm")
     )
-    (path "/c7e691f1-3826-4fda-8caf-e0d6c99d6f96/580b4225-b319-4c9a-a81c-124790bf2feb"
+    (path "/0275355d-7efc-47a4-80e1-0ca0e32dbe5e"
       (reference "U328") (unit 3) (value "74HC00") (footprint "Package_SO:SO-14_3.9x8.65mm_P1.27mm")
     )

Commit message: .
Other:
- sheet icr ports: added ~{SDRIRQ}; removed SDRIRQ
- sheet sdr ports: added ~{SDRIRQ}; removed SDRIRQ
Changed lines of the file:
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@@
   )
   (bus_alias "ENABLEBUS" (members "~{EN[0..15]}"))
+  (bus_alias "DATABUS" (members "D[0..7]" "DZ[0..7]"))
   (bus_alias "CONTROLBUS" (members "TASTART" "CNT" "SP" "PHI2" "~{FLAG}" "TOD" "TAPULSE" "TBPULSE" "TODIRQ" "~{IRQ}" "PB6ON" "PB7ON" "TAOUT" "TBOUT" "SPMODE" "TODIN" "ALARM" "ENABLE_NAND" "TARUNMODE" "~{RES}"))
-  (bus_alias "DATABUS" (members "D[0..7]" "DZ[0..7]"))
   (junction (at 83.82 33.02) (diameter 0) (color 0 0 0 0)
   )
@@
     (effects (font (size 1.27 1.27)) (justify left bottom))
   )
-  (label "SDRIRQ" (at 152.4 96.52 0)
+  (label "~{SDRIRQ}" (at 152.4 96.52 0)
     (effects (font (size 1.27 1.27)) (justify left bottom))
   )
@@
       (effects (font (size 1.27 1.27)) (justify left))
     )
-    (pin "SDRIRQ" output (at 149.86 96.52 0)
+    (pin "~{SDRIRQ}" output (at 149.86 96.52 0)
       (effects (font (size 1.27 1.27)) (justify right))
     )
@@
       (effects (font (size 1.27 1.27)) (justify left))
     )
-    (pin "SDRIRQ" input (at 190.5 96.52 180)
+    (pin "~{SDRIRQ}" input (at 190.5 96.52 180)
       (effects (font (size 1.27 1.27)) (justify left))
     )
@@
       (reference "U316") (unit 3) (value "74HC00") (footprint "Package_SO:SO-14_3.9x8.65mm_P1.27mm")
     )
-    (path "/c7e691f1-3826-4fda-8caf-e0d6c99d6f96/e9e07058-34a8-470c-a7cf-5a2cf0cdddc0"
+    (path "/108743f5-032b-46ed-a6db-6b8bf543e425/08cd0747-3624-4251-9104-81e81adf48f3/006d0d53-2980-46fc-9296-d4a5612be9c7"
       (reference "U316") (unit 4) (value "74HC00") (footprint "Package_SO:SO-14_3.9x8.65mm_P1.27mm")
     )
@@
       (reference "U335") (unit 2) (value "74HC04") (footprint "Package_SO:SO-14_3.9x8.65mm_P1.27mm")
     )
-    (path "/6ac12df0-6226-4d30-947c-27d74eb345ea/de5d14ee-70d2-45ec-9f9c-f4568d1a6c84/3184a564-686d-48c3-907b-2ee2127eb850"
+    (path "/c7e691f1-3826-4fda-8caf-e0d6c99d6f96/cafb36af-fa7e-4a81-8a3a-a73d830c5f36"
       (reference "U335") (unit 3) (value "74HC04") (footprint "Package_SO:SO-14_3.9x8.65mm_P1.27mm")
     )
