File: B3/B3.kicad_pcb (KiCad board)
At the start: 4 copper layers, 100 x 100 mm, 86 parts, among them U301 74HC00, U302 74HC125, U303 74HC74, U304 74HC74, U305 74HC74, U306 74HC32, U307 74HC299, U308 74HC193, U309 74HC00, U310 74HC244, U311 74HC377, U312 74HC244, U313 74HC299, U314 74HC32, U315 74HC193, U316 74HC00, U317 74HC74, U318 74HC08, U319 74HC32, U320 74HC00, U321 74HC00, U322 74HC00, U323 74HC00, U324 74HC00, U325 74HC08, U326 74HC08, U327 74HC377, U328 74HC00, U329 74HC00, U330 74HC74, U331 74HC74, U332 74HC74, U333 74HC74, U334 74HC74, U335 74HC04, U336 74HC244, U337 74HC08, U338 74HC32, U339 74HC08

Commit message: B0 ready for v0.2.0 release.
Connections:
- U333 pad 1: Net-(U333-Pad1) -> Net-(U333-Pad8)
- U333 pad 10: Net-(U333-Pad1) -> Net-(U333-Pad10)
- U333 pad 6: Net-(U333-Pad1) -> Net-(U333-Pad10)
- U333 pad 8: unconnected-(U333-Pad8) -> Net-(U333-Pad8)
Routing:
- net Net-(U333-Pad1): track 17.3 -> 0.00 mm
- net Net-(U333-Pad8): track 0.00 -> 14.3 mm
- net Net-(U333-Pad10): track 0.00 -> 5.48 mm
Changed lines of the file:
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@@
   (net 196 "Net-(U324-Pad8)")
   (net 197 "Net-(U328-Pad12)")
-  (net 198 "Net-(U333-Pad1)")
+  (net 198 "Net-(U333-Pad8)")
   (net 199 "Net-(U333-Pad3)")
   (net 200 "unconnected-(U333-Pad5)")
-  (net 201 "unconnected-(U333-Pad8)")
+  (net 201 "Net-(U333-Pad10)")
   (net 202 "Net-(U335-Pad9)")
   (net 203 "Net-(U337-Pad11)")
@@
     (fp_line (start 1.95 -4.325) (end 1.95 4.325) (layer "F.Fab") (width 0.1))
     (pad "1" smd roundrect (at -2.475 -3.81) (size 1.95 0.6) (layers "F.Cu" "F.Paste" "F.Mask") (roundrect_rratio 0.25)
-      (net 198 "Net-(U333-Pad1)") (pinfunction "~{R}") (pintype "input"))
+      (net 198 "Net-(U333-Pad8)") (pinfunction "~{R}") (pintype "input"))
     (pad "2" smd roundrect (at -2.475 -2.54) (size 1.95 0.6) (layers "F.Cu" "F.Paste" "F.Mask") (roundrect_rratio 0.25)
       (net 29 "VCC") (pinfunction "D") (pintype "input"))
@@
       (net 200 "unconnected-(U333-Pad5)") (pinfunction "Q") (pintype "output+no_connect"))
     (pad "6" smd roundrect (at -2.475 2.54) (size 1.95 0.6) (layers "F.Cu" "F.Paste" "F.Mask") (roundrect_rratio 0.25)
-      (net 198 "Net-(U333-Pad1)") (pinfunction "~{Q}") (pintype "output"))
+      (net 201 "Net-(U333-Pad10)") (pinfunction "~{Q}") (pintype "output"))
     (pad "7" smd roundrect (at -2.475 3.81) (size 1.95 0.6) (layers "F.Cu" "F.Paste" "F.Mask") (roundrect_rratio 0.25)
       (net 30 "GND") (pinfunction "GND") (pintype "power_in"))
     (pad "8" smd roundrect (at 2.475 3.81) (size 1.95 0.6) (layers "F.Cu" "F.Paste" "F.Mask") (roundrect_rratio 0.25)
-      (net 201 "unconnected-(U333-Pad8)") (pinfunction "~{Q}") (pintype "output+no_connect"))
+      (net 198 "Net-(U333-Pad8)") (pinfunction "~{Q}") (pintype "output"))
     (pad "9" smd roundrect (at 2.475 2.54) (size 1.95 0.6) (layers "F.Cu" "F.Paste" "F.Mask") (roundrect_rratio 0.25)
       (net 128 "/icr/icrControl/ICR4") (pinfunction "Q") (pintype "output"))
     (pad "10" smd roundrect (at 2.475 1.27) (size 1.95 0.6) (layers "F.Cu" "F.Paste" "F.Mask") (roundrect_rratio 0.25)
-      (net 198 "Net-(U333-Pad1)") (pinfunction "~{S}") (pintype "input"))
+      (net 201 "Net-(U333-Pad10)") (pinfunction "~{S}") (pintype "input"))
     (pad "11" smd roundrect (at 2.475 0) (size 1.95 0.6) (layers "F.Cu" "F.Paste" "F.Mask") (roundrect_rratio 0.25)
       (net 29 "VCC") (pinfunction "C") (pintype "input"))
@@
   (segment (start 166.9 104.8) (end 169.105 104.8) (width 0.127) (layer "F.Cu") (net 196))
   (segment (start 169.125 114.1) (end 164.175 114.1) (width 0.127) (layer "F.Cu") (net 197))
-  (segment (start 137.461468 113.44) (end 138.04 114.018532) (width 0.127) (layer "F.Cu") (net 198))
-  (segment (start 134.11 116.64) (end 136.305 116.64) (width 0.127) (layer "F.Cu") (net 198))
-  (segment (start 138.04 116.21) (end 137.61 116.64) (width 0.127) (layer "F.Cu") (net 198))
-  (segment (start 131.355 111.56) (end 132.43 111.56) (width 0.127) (layer "F.Cu") (net 198))
-  (segment (start 131.355 117.91) (end 132.84 117.91) (width 0.127) (layer "F.Cu") (net 198))
-  (segment (start 137.61 116.64) (end 136.305 116.64) (width 0.127) (layer "F.Cu") (net 198))
   (segment (start 134.31 113.44) (end 137.461468 113.44) (width 0.127) (layer "F.Cu") (net 198))
-  (segment (start 132.84 117.91) (end 134.11 116.64) (width 0.127) (layer "F.Cu") (net 198))
+  (segment (start 138.04 114.018532) (end 138.04 118.6) (width 0.127) (layer "F.Cu") (net 198))
+  (segment (start 138.04 118.6) (end 137.46 119.18) (width 0.127) (layer "F.Cu") (net 198))
   (segment (start 132.43 111.56) (end 134.31 113.44) (width 0.127) (layer "F.Cu") (net 198))
-  (segment (start 138.04 114.018532) (end 138.04 116.21) (width 0.127) (layer "F.Cu") (net 198))
+  (segment (start 137.461468 113.44) (end 138.04 114.018532) (width 0.127) (layer "F.Cu") (net 198))
+  (segment (start 137.46 119.18) (end 136.305 119.18) (width 0.127) (layer "F.Cu") (net 198))
+  (segment (start 131.355 111.56) (end 132.43 111.56) (width 0.127) (layer "F.Cu") (net 198))
   (segment (start 112.23 127.82) (end 115.52 127.82) (width 0.127) (layer "F.Cu") (net 199))
   (segment (start 126.77 117.24) (end 129.91 114.1) (width 0.127) (layer "F.Cu") (net 199))
@@
   (segment (start 109.475 128.48) (end 111.57 128.48) (width 0.127) (layer "F.Cu") (net 199))
   (segment (start 122.585008 116.11354) (end 123.711468 117.24) (width 0.127) (layer "F.Cu") (net 199))
+  (segment (start 134.11 116.64) (end 136.305 116.64) (width 0.127) (layer "F.Cu") (net 201))
+  (segment (start 131.355 117.91) (end 132.84 117.91) (width 0.127) (layer "F.Cu") (net 201))
+  (segment (start 132.84 117.91) (end 134.11 116.64) (width 0.127) (layer "F.Cu") (net 201))
   (segment (start 116.6 132.29) (end 117.58 133.27) (width 0.127) (layer "F.Cu") (net 202))
   (segment (start 143.1 133.27) (end 145.87646 130.49354) (width 0.127) (layer "F.Cu") (net 202))

Commit message: B3 ready for v0.2.0 release
Parts:
- added C300: 100n, Capacitor_SMD:C_0603_1608Metric, F.Cu at (190.7, 106.8)
- added U340: 74HC74, Package_SO:SO-14_3.9x8.65mm_P1.27mm, F.Cu at (190.7, 100.2)
- moved C340 13.3 mm to (193.6, 94.0), turned to 90 degrees
Connections:
- C340 pad 1: ~{RES} -> VCC
- CONTROLBUS3 pad 18: TARUNMODE -> unconnected-(CONTROLBUS3-Pad18)
- U302 pad 4: Net-(U302-Pad4) -> Net-(U301-Pad10)
- U303 pad 6: unconnected-(U303-Pad6) -> Net-(U303-Pad6)
- U304 pad 1: Net-(U304-Pad1) -> VCC
- U304 pad 13: Net-(U304-Pad1) -> /sdr/sdrController/~{FULL}
- U304 pad 4: VCC -> Net-(U304-Pad4)
- U304 pad 8: Net-(U304-Pad1) -> Net-(U304-Pad4)
- U305 pad 1: Net-(U303-Pad10) -> Net-(U303-Pad6)
- U305 pad 12: Net-(U302-Pad4) -> Net-(U305-Pad12)
- U305 pad 8: Net-(U302-Pad4) -> Net-(U305-Pad12)
- U313 pad 19: /sdr/sdrController/~{SDRCOUNT} -> Net-(U313-Pad19)
- U314 pad 10: Net-(U302-Pad4) -> Net-(U305-Pad12)
- U315 pad 5: Net-(U302-Pad4) -> Net-(U305-Pad12)
Routing:
- net Net-(U302-Pad4): track 72.0 -> 0.00 mm, vias 2 -> 0
- net Net-(U313-Pad19): track 0.00 -> 70.7 mm, vias 0 -> 2
- net Net-(U305-Pad12): track 0.00 -> 51.3 mm, vias 0 -> 2
- net Net-(U301-Pad10): track 30.2 -> 63.1 mm, vias 2 -> 4
- net /~{PHI2}: track 170.9 -> 198.7 mm, vias 9 -> 10
- net Net-(U304-Pad1): track 14.4 -> 0.00 mm
- net Net-(U303-Pad6): track 0.00 -> 13.7 mm, vias 0 -> 2
- net Net-(U303-Pad10): track 15.9 -> 7.16 mm
- net VCC: track 258.5 -> 249.8 mm, vias 46 -> 48
- net /sdr/sdrController/~{SDRCOUNT}: track 105.5 -> 114.2 mm
- net Net-(U304-Pad4): track 0.00 -> 6.00 mm, vias 0 -> 2
- net /sdr/sdrController/~{FULL}: track 97.9 -> 103.7 mm
- net GND: track 80.1 -> 75.6 mm, vias 90 -> 92
- net SPMODE: track 128.5 -> 130.5 mm
- net DZ2: track 158.6 -> 156.8 mm
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Other:
- board text added: "74HCT6526 Board 3 v0.2.0"
- board text removed: "74HCT6526 Board 3 v0.1.2"

Commit message: Ready for v0.2.1
Parts:
- added SW301: SW_SPDT, Button_Switch_SMD:SW_SPDT_PCM12, F.Cu at (166.7, 142.7)
Connections:
- U334 pad 6: unconnected-(U334-Pad6) -> Net-(U334-Pad6)
- U334 pad 8: ~{IRQ} -> Net-(U334-Pad8)
Routing:
- net Net-(U334-Pad6): track 0.00 -> 11.7 mm
- net Net-(U334-Pad8): track 0.00 -> 8.80 mm
- net ~{IRQ}: track 46.9 -> 55.2 mm
- net Net-(U334-Pad4): track 57.2 -> 52.1 mm
- net /icr/icrControl/ICR4: track 60.0 -> 61.0 mm
Other:
- board text added: "74HCT6526 Board 3 v0.2.1"
- board text added: "NEW OLD"
- board text removed: "74HCT6526 Board 3 v0.2.0"

Commit message: B2 refactored. B4 Added. TOD sch completed.
Routing:
- net Net-(U333-Pad3): track 33.4 -> 31.6 mm
- net TBPULSE: track 131.9 -> 131.3 mm
- net Net-(U332-Pad4): track 20.3 -> 19.7 mm
Changed lines of the file:
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@@
   (segment (start 192.5 117.42) (end 191.38 118.54) (width 0.127) (layer "B.Cu") (net 13))
   (segment (start 191.955 123.675) (end 193.135 123.675) (width 0.127) (layer "B.Cu") (net 13))
-  (segment (start 113 125.34) (end 113.6 125.94) (width 0.127) (layer "F.Cu") (net 15))
-  (segment (start 113 125.34) (end 111.01 125.34) (width 0.127) (layer "F.Cu") (net 15))
-  (via (at 111.01 125.34) (size 0.57) (drill 0.3) (layers "F.Cu" "B.Cu") (net 15))
+  (segment (start 112.6 125.94) (end 114.425 125.94) (width 0.127) (layer "F.Cu") (net 15))
+  (via (at 112.6 125.94) (size 0.57) (drill 0.3) (layers "F.Cu" "B.Cu") (net 15))
+  (segment (start 112.02 125.94) (end 112.6 125.94) (width 0.127) (layer "B.Cu") (net 15))
   (segment (start 194.88648 133.944988) (end 186.594988 142.23648) (width 0.127) (layer "B.Cu") (net 15))
-  (segment (start 111.01 125.34) (end 111.01 126.95) (width 0.127) (layer "B.Cu") (net 15))
   (segment (start 111.04648 142.23648) (end 107.35 138.54) (width 0.127) (layer "B.Cu") (net 15))
   (segment (start 191.12648 123.205012) (end 191.849989 123.92852) (width 0.127) (layer "B.Cu") (net 15))
   (segment (start 192.5 114.88) (end 191.12648 116.25352) (width 0.127) (layer "B.Cu") (net 15))
   (segment (start 111.01 126.95) (end 107.35 130.61) (width 0.127) (layer "B.Cu") (net 15))
+  (segment (start 111.01 126.95) (end 112.02 125.94) (width 0.127) (layer "B.Cu") (net 15))
   (segment (start 107.35 138.54) (end 107.35 130.61) (width 0.127) (layer "B.Cu") (net 15))
   (segment (start 193.029988 123.92852) (end 194.88648 125.785012) (width 0.127) (layer "B.Cu") (net 15))
@@
   (segment (start 188.100011 101.454989) (end 188.085 101.47) (width 0.127) (layer "B.Cu") (net 198))
   (segment (start 188.100011 50.710011) (end 188.100011 101.454989) (width 0.127) (layer "B.Cu") (net 198))
+  (segment (start 115.52 127.82) (end 118.46 124.88) (width 0.127) (layer "F.Cu") (net 199))
+  (segment (start 129.91 114.1) (end 131.355 114.1) (width 0.127) (layer "F.Cu") (net 199))
   (segment (start 112.23 127.82) (end 115.52 127.82) (width 0.127) (layer "F.Cu") (net 199))
-  (segment (start 126.77 117.24) (end 129.91 114.1) (width 0.127) (layer "F.Cu") (net 199))
-  (segment (start 119.313524 116.11354) (end 122.585008 116.11354) (width 0.127) (layer "F.Cu") (net 199))
-  (segment (start 115.52 127.82) (end 118.46 124.88) (width 0.127) (layer "F.Cu") (net 199))
-  (segment (start 118.46 124.88) (end 118.46 116.967064) (width 0.127) (layer "F.Cu") (net 199))
-  (segment (start 123.711468 117.24) (end 126.77 117.24) (width 0.127) (layer "F.Cu") (net 199))
-  (segment (start 118.46 116.967064) (end 119.313524 116.11354) (width 0.127) (layer "F.Cu") (net 199))
   (segment (start 111.57 128.48) (end 112.23 127.82) (width 0.127) (layer "F.Cu") (net 199))
-  (segment (start 129.91 114.1) (end 131.355 114.1) (width 0.127) (layer "F.Cu") (net 199))
+  (segment (start 118.46 124.88) (end 118.46 123) (width 0.127) (layer "F.Cu") (net 199))
+  (segment (start 127.52 121.07) (end 129.325 119.265) (width 0.127) (layer "F.Cu") (net 199))
+  (segment (start 120.39 121.07) (end 127.52 121.07) (width 0.127) (layer "F.Cu") (net 199))
+  (segment (start 118.46 123) (end 120.39 121.07) (width 0.127) (layer "F.Cu") (net 199))
+  (segment (start 129.325 119.265) (end 129.325 114.685) (width 0.127) (layer "F.Cu") (net 199))
+  (segment (start 129.325 114.685) (end 129.91 114.1) (width 0.127) (layer "F.Cu") (net 199))
   (segment (start 109.475 128.48) (end 111.57 128.48) (width 0.127) (layer "F.Cu") (net 199))
-  (segment (start 122.585008 116.11354) (end 123.711468 117.24) (width 0.127) (layer "F.Cu") (net 199))
   (segment (start 134.11 116.64) (end 136.305 116.64) (width 0.127) (layer "F.Cu") (net 201))
   (segment (start 131.355 117.91) (end 132.84 117.91) (width 0.127) (layer "F.Cu") (net 201))
@@
   (segment (start 148.45 128.48) (end 152.26 124.67) (width 0.127) (layer "F.Cu") (net 205))
   (segment (start 147.245 128.48) (end 148.45 128.48) (width 0.127) (layer "F.Cu") (net 205))
+  (segment (start 109.475 125.94) (end 110.6 125.94) (width 0.127) (layer "F.Cu") (net 207))
+  (segment (start 110.6 125.94) (end 111.28 125.26) (width 0.127) (layer "F.Cu") (net 207))
+  (segment (start 117.01 125.26) (end 117.95 124.32) (width 0.127) (layer "F.Cu") (net 207))
+  (segment (start 119.34 115.37) (end 120.415 115.37) (width 0.127) (layer "F.Cu") (net 207))
   (segment (start 117.95 124.32) (end 117.95 116.76) (width 0.127) (layer "F.Cu") (net 207))
-  (segment (start 119.34 115.37) (end 120.415 115.37) (width 0.127) (layer "F.Cu") (net 207))
-  (segment (start 112.31 126.57) (end 115.7 126.57) (width 0.127) (layer "F.Cu") (net 207))
-  (segment (start 109.475 125.94) (end 111.68 125.94) (width 0.127) (layer "F.Cu") (net 207))
-  (segment (start 115.7 126.57) (end 117.95 124.32) (width 0.127) (layer "F.Cu") (net 207))
   (segment (start 117.95 116.76) (end 119.34 115.37) (width 0.127) (layer "F.Cu") (net 207))
-  (segment (start 111.68 125.94) (end 112.31 126.57) (width 0.127) (layer "F.Cu") (net 207))
+  (segment (start 111.28 125.26) (end 117.01 125.26) (width 0.127) (layer "F.Cu") (net 207))
   (segment (start 123.47 116.64) (end 125.365 116.64) (width 0.127) (layer "F.Cu") (net 208))
   (segment (start 118.20352 116.865012) (end 119.208512 115.86002) (width 0.127) (layer "F.Cu") (net 208))
