File: B3/icr.kicad_sch (KiCad schematic)
At the start: 0 parts

Commit message: .
Other:
- company: (none) -> Daniel Molina
- title: (none) -> 74HCT6526 Board 3
Changed lines of the file:
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@@
 (kicad_sch (version 20211123) (generator eeschema)
   (paper "A4")
+  (title_block
+    (title "74HCT6526 Board 3")
+    (date "2022-10-08")
+    (rev "0.1.2")
+    (company "Daniel Molina")
+    (comment 1 "https://github.com/dmolinagarcia/74HCT6526")
+  )
   (junction (at 96.52 58.42) (diameter 0) (color 0 0 0 0)
   )

Commit message: .
Other:
- sheet icrControl ports: added ~{SDRIRQ}; removed SDRIRQ
Changed lines of the file:
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@@
     (effects (font (size 1.27 1.27)) (justify right))
   )
-  (hierarchical_label "SDRIRQ" (shape input) (at 73.66 133.35 180)
+  (hierarchical_label "~{SDRIRQ}" (shape input) (at 73.66 133.35 180)
     (effects (font (size 1.27 1.27)) (justify right))
   )
@@
       (effects (font (size 1.27 1.27)) (justify left))
     )
-    (pin "SDRIRQ" input (at 106.68 133.35 180)
+    (pin "~{SDRIRQ}" input (at 106.68 133.35 180)
       (effects (font (size 1.27 1.27)) (justify left))
     )
