File: B3/icrControl.kicad_sch (KiCad schematic)
At the start: 11 parts, among them U329 74HC00, U330 74HC74, U331 74HC74, U332 74HC74, U333 74HC74, U334 74HC74, U335 74HC04, U336 74HC244, U337 74HC08, U338 74HC32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

Commit message: Fixing ICR
Parts:
- added U341: 74HC157, Package_SO:SO-16_3.9x9.9mm_P1.27mm, symbol Custom 74xx:74HC157
Connections:
- net ~{ICRCLR1}: now also U341.2
- net ~{ICRCLR2}: now also U341.3; no longer U332.13 (~{R})
- new net: U332.13 (~{R}), U341.4
Changed lines of the file:
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@@
   (junction (at 88.9 124.46) (diameter 0) (color 0 0 0 0)
   )
-  (junction (at 88.9 101.6) (diameter 0) (color 0 0 0 0)
+  (junction (at 69.85 102.87) (diameter 0) (color 0 0 0 0)
   )
   (junction (at 88.9 102.87) (diameter 0) (color 0 0 0 0)
@@
   )
   (junction (at 34.29 100.33) (diameter 0) (color 0 0 0 0)
+  )
+  (junction (at 66.04 73.66) (diameter 0) (color 0 0 0 0)
   )
   (junction (at 118.11 91.44) (diameter 0) (color 0 0 0 0)
@@
     (stroke (width 0) (type default) (color 0 0 0 0))
   )
+  (wire (pts (xy 88.9 101.6) (xy 88.9 102.87))
+    (stroke (width 0) (type default) (color 0 0 0 0))
+  )
   (wire (pts (xy 226.06 54.61) (xy 229.87 54.61))
     (stroke (width 0) (type default) (color 0 0 0 0))
@@
     (stroke (width 0) (type default) (color 0 0 0 0))
   )
-  (wire (pts (xy 88.9 102.87) (xy 88.9 101.6))
-    (stroke (width 0) (type default) (color 0 0 0 0))
-  )
   (wire (pts (xy 226.06 52.07) (xy 229.87 52.07))
     (stroke (width 0) (type default) (color 0 0 0 0))
@@
     (stroke (width 0) (type default) (color 0 0 0 0))
   )
-  (wire (pts (xy 88.9 101.6) (xy 88.9 78.74))
-    (stroke (width 0) (type default) (color 0 0 0 0))
-  )
   (wire (pts (xy 160.02 142.24) (xy 157.48 142.24))
     (stroke (width 0) (type default) (color 0 0 0 0))
@@
     (stroke (width 0) (type default) (color 0 0 0 0))
   )
+  (wire (pts (xy 66.04 76.2) (xy 66.04 73.66))
+    (stroke (width 0) (type default) (color 0 0 0 0))
+  )
   (bus (pts (xy 232.41 36.83) (xy 232.41 39.37))
     (stroke (width 0) (type default) (color 0 0 0 0))
@@
     (stroke (width 0) (type default) (color 0 0 0 0))
   )
+  (wire (pts (xy 66.04 76.2) (xy 69.85 76.2))
+    (stroke (width 0) (type default) (color 0 0 0 0))
+  )
   (bus (pts (xy 179.07 114.3) (xy 179.07 128.27))
     (stroke (width 0) (type default) (color 0 0 0 0))
@@
     (stroke (width 0) (type default) (color 0 0 0 0))
   )
-  (wire (pts (xy 88.9 78.74) (xy 125.73 78.74))
-    (stroke (width 0) (type default) (color 0 0 0 0))
-  )
   (wire (pts (xy 160.02 46.99) (xy 200.66 46.99))
     (stroke (width 0) (type default) (color 0 0 0 0))
@@
     (stroke (width 0) (type default) (color 0 0 0 0))
   )
+  (wire (pts (xy 85.09 78.74) (xy 125.73 78.74))
+    (stroke (width 0) (type default) (color 0 0 0 0))
+  )
+  (wire (pts (xy 69.85 102.87) (xy 88.9 102.87))
+    (stroke (width 0) (type default) (color 0 0 0 0))
+  )
   (bus (pts (xy 157.48 123.19) (xy 157.48 125.73))
     (stroke (width 0) (type default) (color 0 0 0 0))
@@
     (stroke (width 0) (type default) (color 0 0 0 0))
   )
+  (wire (pts (xy 69.85 81.28) (xy 69.85 102.87))
+    (stroke (width 0) (type default) (color 0 0 0 0))
+  )
   (wire (pts (xy 124.46 163.83) (xy 127 163.83))
     (stroke (width 0) (type default) (color 0 0 0 0))
@@
     (stroke (width 0) (type default) (color 0 0 0 0))
   )
-  (wire (pts (xy 54.61 102.87) (xy 88.9 102.87))
+  (wire (pts (xy 54.61 102.87) (xy 69.85 102.87))
     (stroke (width 0) (type default) (color 0 0 0 0))
   )
@@
     (pin "14")
     (pin "7")
+  )
+  (symbol (lib_id "Custom 74xx:74HC157") (at -38.1 102.87 0) (unit 2)
+    (in_bom yes) (on_board yes) (fields_autoplaced)
+    (property "Reference" "U341" (id 0) (at -38.1 95.25 0)
+      (effects (font (size 0.889 0.889)))
+    )
+    (property "Value" "74HC157" (id 1) (at -38.1 97.79 0)
+      (effects (font (size 0.889 0.889)))
+    )
+    (property "Footprint" "Package_SO:SO-16_3.9x9.9mm_P1.27mm" (id 2) (at -38.1 102.87 0)
+      (effects (font (size 1.27 1.27)) hide)
+    )
+    (property "Datasheet" "" (id 3) (at -38.1 96.52 0)
+      (effects (font (size 1.27 1.27)) hide)
+    )
+    (pin "2")
+    (pin "3")
+    (pin "4")
+    (pin "5")
+    (pin "6")
+    (pin "7")
+    (pin "10")
+    (pin "11")
+    (pin "9")
+    (pin "12")
+    (pin "13")
+    (pin "14")
+    (pin "1")
+    (pin "15")
+    (pin "16")
+    (pin "8")
   )
   (symbol (lib_id "Custom 74xx:74HC08") (at 195.58 95.25 0) (unit 4)
@@
     (pin "7")
   )
+  (symbol (lib_id "Custom 74xx:74HC157") (at -62.23 90.17 0) (unit 5)
+    (in_bom yes) (on_board yes) (fields_autoplaced)
+    (property "Reference" "U341" (id 0) (at -55.88 89.5349 0)
+      (effects (font (size 0.889 0.889)) (justify left))
+    )
+    (property "Value" "74HC157" (id 1) (at -55.88 92.0749 0)
+      (effects (font (size 0.889 0.889)) (justify left))
+    )
+    (property "Footprint" "Package_SO:SO-16_3.9x9.9mm_P1.27mm" (id 2) (at -62.23 90.17 0)
+      (effects (font (size 1.27 1.27)) hide)
+    )
+    (property "Datasheet" "" (id 3) (at -62.23 83.82 0)
+      (effects (font (size 1.27 1.27)) hide)
+    )
+    (pin "2")
+    (pin "3")
+    (pin "4")
+    (pin "5")
+    (pin "6")
+    (pin "7")
+    (pin "10")
+    (pin "11")
+    (pin "9")
+    (pin "12")
+    (pin "13")
+    (pin "14")
+    (pin "1")
+    (pin "15")
+    (pin "16")
+    (pin "8")
+  )
   (symbol (lib_id "74xx:74HC74") (at 125.73 116.84 0) (unit 2)
     (in_bom yes) (on_board yes) (fields_autoplaced)
@@
     (pin "7")
   )
+  (symbol (lib_id "Custom 74xx:74HC157") (at -38.1 115.57 0) (unit 3)
+    (in_bom yes) (on_board yes) (fields_autoplaced)
+    (property "Reference" "U341" (id 0) (at -38.1 107.95 0)
+      (effects (font (size 0.889 0.889)))
+    )
+    (property "Value" "74HC157" (id 1) (at -38.1 110.49 0)
+      (effects (font (size 0.889 0.889)))
+    )
+    (property "Footprint" "Package_SO:SO-16_3.9x9.9mm_P1.27mm" (id 2) (at -38.1 115.57 0)
+      (effects (font (size 1.27 1.27)) hide)
+    )
+    (property "Datasheet" "" (id 3) (at -38.1 109.22 0)
+      (effects (font (size 1.27 1.27)) hide)
+    )
+    (pin "2")
+    (pin "3")
+    (pin "4")
+    (pin "5")
+    (pin "6")
+    (pin "7")
+    (pin "10")
+    (pin "11")
+    (pin "9")
+    (pin "12")
+    (pin "13")
+    (pin "14")
+    (pin "1")
+    (pin "15")
+    (pin "16")
+    (pin "8")
+  )
   (symbol (lib_id "Custom 74xx:74HC08") (at 195.58 137.16 0) (unit 3)
     (in_bom yes) (on_board yes) (fields_autoplaced)
@@
     (pin "14")
     (pin "7")
+  )
+  (symbol (lib_id "Custom 74xx:74HC157") (at -38.1 127 0) (unit 4)
+    (in_bom yes) (on_board yes) (fields_autoplaced)
+    (property "Reference" "U341" (id 0) (at -38.1 119.38 0)
+      (effects (font (size 0.889 0.889)))
+    )
+    (property "Value" "74HC157" (id 1) (at -38.1 121.92 0)
+      (effects (font (size 0.889 0.889)))
+    )
+    (property "Footprint" "Package_SO:SO-16_3.9x9.9mm_P1.27mm" (id 2) (at -38.1 127 0)
+      (effects (font (size 1.27 1.27)) hide)
+    )
+    (property "Datasheet" "" (id 3) (at -38.1 120.65 0)
+      (effects (font (size 1.27 1.27)) hide)
+    )
+    (pin "2")
+    (pin "3")
+    (pin "4")
+    (pin "5")
+    (pin "6")
+    (pin "7")
+    (pin "10")
+    (pin "11")
+    (pin "9")
+    (pin "12")
+    (pin "13")
+    (pin "14")
+    (pin "1")
+    (pin "15")
+    (pin "16")
+    (pin "8")
   )
   (symbol (lib_id "74xx:74HC04") (at 100.33 156.21 0) (unit 4)
@@
     (pin "7")
   )
+  (symbol (lib_id "Custom 74xx:74HC157") (at 77.47 78.74 0) (unit 1)
+    (in_bom yes) (on_board yes) (fields_autoplaced)
+    (property "Reference" "U341" (id 0) (at 77.47 71.12 0)
+      (effects (font (size 0.889 0.889)))
+    )
+    (property "Value" "74HC157" (id 1) (at 77.47 73.66 0)
+      (effects (font (size 0.889 0.889)))
+    )
+    (property "Footprint" "Package_SO:SO-16_3.9x9.9mm_P1.27mm" (id 2) (at 77.47 78.74 0)
+      (effects (font (size 1.27 1.27)) hide)
+    )
+    (property "Datasheet" "" (id 3) (at 77.47 72.39 0)
+      (effects (font (size 1.27 1.27)) hide)
+    )
+    (pin "2")
+    (pin "3")
+    (pin "4")
+    (pin "5")
+    (pin "6")
+    (pin "7")
+    (pin "10")
+    (pin "11")
+    (pin "9")
+    (pin "12")
+    (pin "13")
+    (pin "14")
+    (pin "1")
+    (pin "15")
+    (pin "16")
+    (pin "8")
+  )
   (symbol (lib_id "Custom 74xx:74HC08") (at 195.58 109.22 0) (unit 4)
     (in_bom yes) (on_board yes) (fields_autoplaced)
@@
     (pin "7")
   )
+  (symbol (lib_id "Custom 74xx:74HC157") (at -62.23 114.3 0) (unit 6)
+    (in_bom yes) (on_board yes) (fields_autoplaced)
+    (property "Reference" "U341" (id 0) (at -54.61 113.6649 0)
+      (effects (font (size 0.889 0.889)) (justify left))
+    )
+    (property "Value" "74HC157" (id 1) (at -54.61 116.2049 0)
+      (effects (font (size 0.889 0.889)) (justify left))
+    )
+    (property "Footprint" "Package_SO:SO-16_3.9x9.9mm_P1.27mm" (id 2) (at -62.23 114.3 0)
+      (effects (font (size 1.27 1.27)) hide)
+    )
+    (property "Datasheet" "" (id 3) (at -62.23 107.95 0)
+      (effects (font (size 1.27 1.27)) hide)
+    )
+    (pin "2")
+    (pin "3")
+    (pin "4")
+    (pin "5")
+    (pin "6")
+    (pin "7")
+    (pin "10")
+    (pin "11")
+    (pin "9")
+    (pin "12")
+    (pin "13")
+    (pin "14")
+    (pin "1")
+    (pin "15")
+    (pin "16")
+    (pin "8")
+  )
   (symbol (lib_id "74xx:74LS32") (at 220.98 130.81 0) (unit 4)

Commit message: .
Parts:
- U335: value 74HC04 -> 74HCT04
Changed lines of the file:
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@@
     (in_bom yes) (on_board yes) (fields_autoplaced)
     (property "Reference" "U335" (id 0) (at 118.11 31.75 0))
-    (property "Value" "74HC04" (id 1) (at 118.11 34.29 0))
+    (property "Value" "74HCT04" (id 1) (at 118.11 34.29 0))
     (property "Footprint" "Package_SO:SO-14_3.9x8.65mm_P1.27mm" (id 2) (at 118.11 40.64 0)
       (effects (font (size 1.27 1.27)) hide)
@@
     (in_bom yes) (on_board yes)
     (property "Reference" "U335" (id 0) (at 114.3 134.62 0))
-    (property "Value" "74HC04" (id 1) (at 114.3 137.16 0))
+    (property "Value" "74HCT04" (id 1) (at 114.3 137.16 0))
     (property "Footprint" "Package_SO:SO-14_3.9x8.65mm_P1.27mm" (id 2) (at 110.49 139.7 0)
       (effects (font (size 1.27 1.27)) hide)
@@
     (in_bom yes) (on_board yes)
     (property "Reference" "U335" (id 0) (at 120.65 58.42 0))
-    (property "Value" "74HC04" (id 1) (at 120.65 60.96 0))
+    (property "Value" "74HCT04" (id 1) (at 120.65 60.96 0))
     (property "Footprint" "Package_SO:SO-14_3.9x8.65mm_P1.27mm" (id 2) (at 118.11 63.5 0)
       (effects (font (size 1.27 1.27)) hide)
@@
     (in_bom yes) (on_board yes)
     (property "Reference" "U335" (id 0) (at 121.92 80.01 0))
-    (property "Value" "74HC04" (id 1) (at 121.92 82.55 0))
+    (property "Value" "74HCT04" (id 1) (at 121.92 82.55 0))
     (property "Footprint" "Package_SO:SO-14_3.9x8.65mm_P1.27mm" (id 2) (at 118.11 86.36 0)
       (effects (font (size 1.27 1.27)) hide)
@@
     (in_bom yes) (on_board yes)
     (property "Reference" "U335" (id 0) (at 104.14 151.13 0))
-    (property "Value" "74HC04" (id 1) (at 104.14 153.67 0))
+    (property "Value" "74HCT04" (id 1) (at 104.14 153.67 0))
     (property "Footprint" "Package_SO:SO-14_3.9x8.65mm_P1.27mm" (id 2) (at 100.33 156.21 0)
       (effects (font (size 1.27 1.27)) hide)

Commit message: Ready for v0.2.2
Parts:
- removed unit 4 of U341
- removed unit 6 of U341
- added SW301: SW_SPDT, Button_Switch_SMD:SW_SPDT_PCM12, symbol Switch:SW_SPDT
- added U342: 74HC74, Package_SO:SO-14_3.9x8.65mm_P1.27mm, symbol 74xx:74HC74
Connections:
- net GND: now also U341.15 (~{E}), SW301.1 (A)
- net ICR1: no longer U337.12
- net ICR7: now also U341.7; no longer U334.9 (Q)
- net TBPULSE: now also U337.12
- net VCC: now also SW301.3 (C), U342.10 (~{S}), U342.2 (D), U342.3 (C); no longer U334.13 (~{R})
- net ~{ICRCLR1}: now also U331.13 (~{R}), U332.1 (~{R}), U333.13 (~{R}), U334.1 (~{R}), U334.13 (~{R}), U342.1 (~{R}), U342.13 (~{R})
- net ~{ICRCLR2}: no longer U331.13 (~{R}), U332.1 (~{R}), U333.13 (~{R}), U334.1 (~{R})
- net ~{IRQ}: now also U341.9; no longer U334.8 (~{Q})
- net ~{PHI2}: now also U342.11 (C)
- net at U341.5: now also U334.12 (D), U334.5 (Q)
- net at U341.6: now also U334.9 (Q)
- net at U334.4 (~{S}), U335.8: now also U342.4 (~{S})
- net at U341.1 (S): now also SW301.2 (B)
- net at U341.10: now also U342.8 (~{Q})
- net at U341.11: now also U342.6 (~{Q})
- new net: U342.12 (D), U342.5 (Q)
- no-connect marks 6 -> 9
Other:
- moved on the sheet: U329A, U329B, U329C, U329D, U330A, U330B, U331A, U331B, U332A, U332B, U333A, U333B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
