File: B3/icrRegister.kicad_sch (KiCad schematic)
At the start: 9 parts, among them U320 74HC00, U321 74HC00, U322 74HC00, U323 74HC00, U324 74HC00, U325 74HC08, U326 74HC08, U327 74HC377, U328 74HC00

Commit message: .
Connections:
- net GND: now also U327.17 (D6), U327.4 (D1), U327.8 (D3)
- net MASK1: now also U327.15 (Q5); no longer U327.5 (Q1)
- no-connect marks 0 -> 3
Other:
- company: (none) -> Daniel Molina
- title: (none) -> 74HCT6526 Board 3
Changed lines of the file:
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@@
 (kicad_sch (version 20211123) (generator eeschema)
   (paper "A4")
+  (title_block
+    (title "74HCT6526 Board 3")
+    (date "2022-10-08")
+    (rev "0.1.2")
+    (company "Daniel Molina")
+    (comment 1 "https://github.com/dmolinagarcia/74HCT6526")
+  )
   (junction (at 106.68 189.23) (diameter 0) (color 0 0 0 0)
   )
@@
   (junction (at 49.53 35.56) (diameter 0) (color 0 0 0 0)
   )
+  (no_connect (at 226.06 74.93))
+  (no_connect (at 226.06 67.31))
+  (no_connect (at 226.06 62.23))
   (bus_entry (at 39.37 182.88) (size 2.54 2.54)
     (stroke (width 0) (type default) (color 0 0 0 0))
@@
     (stroke (width 0) (type default) (color 0 0 0 0))
   )
-  (bus_entry (at 241.3 59.69) (size -2.54 2.54)
+  (bus_entry (at 241.3 69.85) (size -2.54 2.54)
     (stroke (width 0) (type default) (color 0 0 0 0))
   )
@@
     (stroke (width 0) (type default) (color 0 0 0 0))
   )
-  (wire (pts (xy 226.06 62.23) (xy 238.76 62.23))
-    (stroke (width 0) (type default) (color 0 0 0 0))
-  )
-  (bus (pts (xy 241.3 59.69) (xy 241.3 62.23))
+  (wire (pts (xy 226.06 72.39) (xy 238.76 72.39))
+    (stroke (width 0) (type default) (color 0 0 0 0))
+  )
+  (bus (pts (xy 241.3 57.15) (xy 241.3 62.23))
     (stroke (width 0) (type default) (color 0 0 0 0))
   )
@@
     (stroke (width 0) (type default) (color 0 0 0 0))
   )
+  (bus (pts (xy 241.3 69.85) (xy 241.3 74.93))
+    (stroke (width 0) (type default) (color 0 0 0 0))
+  )
   (wire (pts (xy 82.55 93.98) (xy 86.36 93.98))
     (stroke (width 0) (type default) (color 0 0 0 0))
@@
     (stroke (width 0) (type default) (color 0 0 0 0))
   )
-  (bus (pts (xy 241.3 67.31) (xy 241.3 74.93))
+  (bus (pts (xy 241.3 67.31) (xy 241.3 69.85))
     (stroke (width 0) (type default) (color 0 0 0 0))
   )
@@
     (stroke (width 0) (type default) (color 0 0 0 0))
   )
-  (bus (pts (xy 241.3 57.15) (xy 241.3 59.69))
-    (stroke (width 0) (type default) (color 0 0 0 0))
-  )
   (wire (pts (xy 86.36 162.56) (xy 86.36 170.18))
     (stroke (width 0) (type default) (color 0 0 0 0))
@@
     (effects (font (size 1.27 1.27)) (justify left bottom))
   )
-  (label "MASK1" (at 231.14 62.23 0)
+  (label "MASK1" (at 231.14 72.39 0)
     (effects (font (size 1.27 1.27)) (justify left bottom))
   )
@@
     (pin "14")
     (pin "7")
+  )
+  (symbol (lib_id "power:GND") (at 200.66 62.23 270) (unit 1)
+    (in_bom yes) (on_board yes) (fields_autoplaced)
+    (property "Reference" "#PWR0357" (id 0) (at 194.31 62.23 0)
+      (effects (font (size 1.27 1.27)) hide)
+    )
+    (property "Value" "GND" (id 1) (at 196.85 62.2299 90)
+      (effects (font (size 1.27 1.27)) (justify right))
+    )
+    (property "Footprint" "" (id 2) (at 200.66 62.23 0)
+      (effects (font (size 1.27 1.27)) hide)
+    )
+    (property "Datasheet" "" (id 3) (at 200.66 62.23 0)
+      (effects (font (size 1.27 1.27)) hide)
+    )
+    (pin "1")
+  )
+  (symbol (lib_id "power:GND") (at 200.66 74.93 270) (unit 1)
+    (in_bom yes) (on_board yes) (fields_autoplaced)
+    (property "Reference" "#PWR0359" (id 0) (at 194.31 74.93 0)
+      (effects (font (size 1.27 1.27)) hide)
+    )
+    (property "Value" "GND" (id 1) (at 196.85 74.9299 90)
+      (effects (font (size 1.27 1.27)) (justify right))
+    )
+    (property "Footprint" "" (id 2) (at 200.66 74.93 0)
+      (effects (font (size 1.27 1.27)) hide)
+    )
+    (property "Datasheet" "" (id 3) (at 200.66 74.93 0)
+      (effects (font (size 1.27 1.27)) hide)
+    )
+    (pin "1")
   )
   (symbol (lib_id "74xx:74HC00") (at 74.93 162.56 0) (unit 3)
@@
     (pin "7")
   )
+  (symbol (lib_id "power:GND") (at 200.66 67.31 270) (unit 1)
+    (in_bom yes) (on_board yes) (fields_autoplaced)
+    (property "Reference" "#PWR0358" (id 0) (at 194.31 67.31 0)
+      (effects (font (size 1.27 1.27)) hide)
+    )
+    (property "Value" "GND" (id 1) (at 196.85 67.3099 90)
+      (effects (font (size 1.27 1.27)) (justify right))
+    )
+    (property "Footprint" "" (id 2) (at 200.66 67.31 0)
+      (effects (font (size 1.27 1.27)) hide)
+    )
+    (property "Datasheet" "" (id 3) (at 200.66 67.31 0)
+      (effects (font (size 1.27 1.27)) hide)
+    )
+    (pin "1")
+  )
   (symbol (lib_id "Custom 74xx:74HC08") (at 118.11 140.97 0) (unit 2)
