File: B3/sdr.kicad_sch (KiCad schematic)
At the start: 0 parts

Commit message: .
Other:
- company: (none) -> Daniel Molina
Changed lines of the file:
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@@
   (title_block
     (title "74HCT6526 Board 3")
-    (date "2022-09-11")
-    (rev "0.1")
+    (date "2022-10-08")
+    (rev "0.1.2")
+    (company "Daniel Molina")
+    (comment 1 "https://github.com/dmolinagarcia/74HCT6526")
   )
   (junction (at 43.18 162.56) (diameter 0) (color 0 0 0 0)

Commit message: .
Other:
- sheet sdrController ports: added ~{SDRIRQ}; removed SDRIRQ
Changed lines of the file:
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@@
     (effects (font (size 1.27 1.27)) (justify right))
   )
-  (hierarchical_label "SDRIRQ" (shape output) (at 271.78 134.62 0)
+  (hierarchical_label "~{SDRIRQ}" (shape output) (at 271.78 134.62 0)
     (effects (font (size 1.27 1.27)) (justify left))
   )
@@
       (effects (font (size 1.27 1.27)) (justify left))
     )
-    (pin "SDRIRQ" output (at 269.24 134.62 0)
-      (effects (font (size 1.27 1.27)) (justify right))
-    )
     (pin "~{SDRCOUNT}" output (at 220.98 134.62 180)
       (effects (font (size 1.27 1.27)) (justify left))
@@
       (effects (font (size 1.27 1.27)) (justify left))
     )
+    (pin "~{SDRIRQ}" output (at 269.24 134.62 0)
+      (effects (font (size 1.27 1.27)) (justify right))
+    )
   )

Commit message: B0 ready for v0.2.0 release.
Other:
- sheet sdrOutput ports: added ~{PHI2}; removed none
Changed lines of the file:
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@@
   (title_block
     (title "74HCT6526 Board 3")
-    (date "2022-10-08")
-    (rev "0.1.2")
+    (date "2023-01-22")
+    (rev "0.2.0")
     (company "Daniel Molina")
     (comment 1 "https://github.com/dmolinagarcia/74HCT6526")
@@
   (junction (at 40.64 111.76) (diameter 0) (color 0 0 0 0)
   )
+  (junction (at 38.1 109.22) (diameter 0) (color 0 0 0 0)
+  )
   (junction (at 45.72 165.1) (diameter 0) (color 0 0 0 0)
   )
@@
     (stroke (width 0) (type default) (color 0 0 0 0))
   )
+  (wire (pts (xy 38.1 170.18) (xy 134.62 170.18))
+    (stroke (width 0) (type default) (color 0 0 0 0))
+  )
+  (wire (pts (xy 134.62 146.05) (xy 142.24 146.05))
+    (stroke (width 0) (type default) (color 0 0 0 0))
+  )
   (wire (pts (xy 132.08 167.64) (xy 132.08 129.54))
     (stroke (width 0) (type default) (color 0 0 0 0))
@@
     (stroke (width 0) (type default) (color 0 0 0 0))
   )
+  (wire (pts (xy 38.1 109.22) (xy 38.1 170.18))
+    (stroke (width 0) (type default) (color 0 0 0 0))
+  )
   (wire (pts (xy 25.4 165.1) (xy 45.72 165.1))
     (stroke (width 0) (type default) (color 0 0 0 0))
@@
   )
   (wire (pts (xy 25.4 167.64) (xy 48.26 167.64))
+    (stroke (width 0) (type default) (color 0 0 0 0))
+  )
+  (wire (pts (xy 134.62 170.18) (xy 134.62 146.05))
     (stroke (width 0) (type default) (color 0 0 0 0))
   )
@@
       (effects (font (size 1.27 1.27)) (justify right))
     )
-  )
+    (pin "~{PHI2}" input (at 142.24 146.05 180)
+      (effects (font (size 1.27 1.27)) (justify left))
+    )
+  )
