File: B3/sdrInput.kicad_sch (KiCad schematic)
At the start: 8 parts, among them U301 74HC04, U302 74HC125, U303 74HC74, U304 74HC74, U305 74HC74, U306 74HC32, U307 74HC299, U308 74HC193

Commit message: B3 added. First revision
Still not verified.
Parts:
- removed U301: 74HC04, Package_SO:SO-14_3.9x8.65mm_P1.27mm, symbol 74xx:74HC04
- added U301: 74HC00, Package_SO:SO-14_3.9x8.65mm_P1.27mm, symbol 74xx:74HC00
Connections:
- net GND: now also U302.1; no longer U302.4
- net SP: now also U302.2; no longer U302.5
- net VCC: now also U307.18 (Ds7), U307.9 (Mr)
- net ~{RES}: now also U301.1, U301.2; no longer U307.18 (Ds7), U307.9 (Mr)
- net at U306.4: now also U301.3
- net at U307.11 (Ds0): now also U302.3; no longer U302.6
Changed lines of the file:
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@@
   (junction (at 93.98 91.44) (diameter 0) (color 0 0 0 0)
   )
+  (junction (at 149.86 58.42) (diameter 0) (color 0 0 0 0)
+  )
   (junction (at 236.22 119.38) (diameter 0) (color 0 0 0 0)
   )
   (junction (at 152.4 111.76) (diameter 0) (color 0 0 0 0)
   )
-  (junction (at 78.74 96.52) (diameter 0) (color 0 0 0 0)
+  (junction (at 91.44 127) (diameter 0) (color 0 0 0 0)
   )
   (junction (at 152.4 114.3) (diameter 0) (color 0 0 0 0)
@@
   )
   (junction (at 152.4 116.84) (diameter 0) (color 0 0 0 0)
-  )
-  (junction (at 149.86 78.74) (diameter 0) (color 0 0 0 0)
   )
   (no_connect (at 180.34 121.92))
@@
     (stroke (width 0) (type default) (color 0 0 0 0))
   )
+  (wire (pts (xy 144.78 58.42) (xy 149.86 58.42))
+    (stroke (width 0) (type default) (color 0 0 0 0))
+  )
   (wire (pts (xy 210.82 106.68) (xy 223.52 106.68))
     (stroke (width 0) (type default) (color 0 0 0 0))
@@
     (stroke (width 0) (type default) (color 0 0 0 0))
   )
+  (wire (pts (xy 91.44 124.46) (xy 91.44 127))
+    (stroke (width 0) (type default) (color 0 0 0 0))
+  )
   (wire (pts (xy 137.16 132.08) (xy 154.94 132.08))
     (stroke (width 0) (type default) (color 0 0 0 0))
@@
     (stroke (width 0) (type default) (color 0 0 0 0))
   )
+  (wire (pts (xy 149.86 58.42) (xy 154.94 58.42))
+    (stroke (width 0) (type default) (color 0 0 0 0))
+  )
   (wire (pts (xy 152.4 96.52) (xy 236.22 96.52))
     (stroke (width 0) (type default) (color 0 0 0 0))
@@
     (stroke (width 0) (type default) (color 0 0 0 0))
   )
-  (wire (pts (xy 149.86 96.52) (xy 149.86 78.74))
-    (stroke (width 0) (type default) (color 0 0 0 0))
-  )
   (wire (pts (xy 78.74 127) (xy 78.74 96.52))
     (stroke (width 0) (type default) (color 0 0 0 0))
@@
     (stroke (width 0) (type default) (color 0 0 0 0))
   )
-  (wire (pts (xy 149.86 78.74) (xy 149.86 53.34))
+  (wire (pts (xy 149.86 78.74) (xy 149.86 58.42))
     (stroke (width 0) (type default) (color 0 0 0 0))
   )
@@
     (stroke (width 0) (type default) (color 0 0 0 0))
   )
+  (wire (pts (xy 91.44 127) (xy 91.44 129.54))
+    (stroke (width 0) (type default) (color 0 0 0 0))
+  )
   (wire (pts (xy 154.94 127) (xy 144.78 127))
     (stroke (width 0) (type default) (color 0 0 0 0))
@@
     (stroke (width 0) (type default) (color 0 0 0 0))
   )
-  (wire (pts (xy 78.74 96.52) (xy 149.86 96.52))
-    (stroke (width 0) (type default) (color 0 0 0 0))
-  )
   (wire (pts (xy 152.4 111.76) (xy 154.94 111.76))
     (stroke (width 0) (type default) (color 0 0 0 0))
   )
   (wire (pts (xy 187.96 114.3) (xy 190.5 114.3))
+    (stroke (width 0) (type default) (color 0 0 0 0))
+  )
+  (wire (pts (xy 149.86 58.42) (xy 149.86 53.34))
     (stroke (width 0) (type default) (color 0 0 0 0))
   )
@@
     (pin "1")
   )
-  (symbol (lib_id "power:VCC") (at 154.94 58.42 0) (unit 1)
+  (symbol (lib_id "power:VCC") (at 144.78 58.42 0) (unit 1)
     (in_bom yes) (on_board yes)
-    (property "Reference" "#PWR0309" (id 0) (at 154.94 62.23 0)
-      (effects (font (size 1.27 1.27)) hide)
-    )
-    (property "Value" "VCC" (id 1) (at 150.2611 57.8286 0)
-      (effects (font (size 1.27 1.27)) (justify left))
-    )
-    (property "Footprint" "" (id 2) (at 154.94 58.42 0)
-      (effects (font (size 1.27 1.27)) hide)
-    )
-    (property "Datasheet" "" (id 3) (at 154.94 58.42 0)
+    (property "Reference" "#PWR0309" (id 0) (at 144.78 62.23 0)
+      (effects (font (size 1.27 1.27)) hide)
+    )
+    (property "Value" "VCC" (id 1) (at 140.1011 57.8286 0)
+      (effects (font (size 1.27 1.27)) (justify left))
+    )
+    (property "Footprint" "" (id 2) (at 144.78 58.42 0)
+      (effects (font (size 1.27 1.27)) hide)
+    )
+    (property "Datasheet" "" (id 3) (at 144.78 58.42 0)
       (effects (font (size 1.27 1.27)) hide)
     )
@@
     (pin "9")
   )
-  (symbol (lib_id "74xx:74LS125") (at 129.54 50.8 0) (unit 2)
+  (symbol (lib_id "74xx:74LS125") (at 129.54 50.8 0) (unit 1)
     (in_bom yes) (on_board yes) (fields_autoplaced)
     (property "Reference" "U302" (id 0) (at 129.54 41.91 0))
@@
     (pin "1")
   )
+  (symbol (lib_id "74xx:74HC00") (at 99.06 127 0) (unit 1)
+    (in_bom yes) (on_board yes) (fields_autoplaced)
+    (property "Reference" "U301" (id 0) (at 99.06 118.11 0))
+    (property "Value" "74HC00" (id 1) (at 99.06 120.65 0))
+    (property "Footprint" "Package_SO:SO-14_3.9x8.65mm_P1.27mm" (id 2) (at 99.06 127 0)
+      (effects (font (size 1.27 1.27)) hide)
+    )
+    (property "Datasheet" "http://www.ti.com/lit/gpn/sn74hc00" (id 3) (at 99.06 127 0)
+      (effects (font (size 1.27 1.27)) hide)
+    )
+    (pin "1")
+    (pin "2")
+    (pin "3")
+    (pin "4")
+    (pin "5")
+    (pin "6")
+    (pin "10")
+    (pin "8")
+    (pin "9")
+    (pin "11")
+    (pin "12")
+    (pin "13")
+    (pin "14")
+    (pin "7")
+  )
   (symbol (lib_id "power:VCC") (at 167.64 101.6 0) (unit 1)
     (in_bom yes) (on_board yes)
@@
     (pin "1")
   )
-  (symbol (lib_id "74xx:74HC04") (at 99.06 127 0) (unit 2)
-    (in_bom yes) (on_board yes) (fields_autoplaced)
-    (property "Reference" "U301" (id 0) (at 99.06 118.11 0))
-    (property "Value" "74HC04" (id 1) (at 99.06 120.65 0))
-    (property "Footprint" "Package_SO:SO-14_3.9x8.65mm_P1.27mm" (id 2) (at 99.06 127 0)
-      (effects (font (size 1.27 1.27)) hide)
-    )
-    (property "Datasheet" "https://assets.nexperia.com/documents/data-sheet/74HC_HCT04.pdf" (id 3) (at 99.06 127 0)
-      (effects (font (size 1.27 1.27)) hide)
-    )
-    (pin "1")
-    (pin "2")
-    (pin "3")
-    (pin "4")
-    (pin "5")
-    (pin "6")
-    (pin "8")
-    (pin "9")
-    (pin "10")
-    (pin "11")
-    (pin "12")
-    (pin "13")
-    (pin "14")
-    (pin "7")
-  )
   (symbol (lib_id "power:VCC") (at 129.54 83.82 180) (unit 1)

Commit message: .
Other:
- company: (none) -> Daniel Molina
Changed lines of the file:
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@@
   (title_block
     (title "74HCT6526 Board 3")
-    (date "2022-09-11")
-    (rev "0.1")
+    (date "2022-10-08")
+    (rev "0.1.2")
+    (company "Daniel Molina")
+    (comment 1 "https://github.com/dmolinagarcia/74HCT6526")
   )
   (junction (at 236.22 114.3) (diameter 0) (color 0 0 0 0)

Commit message: B0 ready for v0.2.0 release.
Connections:
- net VCC: now also U304.1 (~{R}); no longer U304.4 (~{S})
- net ~{FULL}: now also U304.13 (~{R})
- net at U303.10 (~{S}), U305.6 (~{Q}): no longer U305.1 (~{R})
- net at U303.6 (~{Q}): now also U305.1 (~{R})
- new net: U304.4 (~{S}), U304.8 (~{Q})
- no-connect marks 11 -> 10
Changed lines of the file:
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@@
   (title_block
     (title "74HCT6526 Board 3")
-    (date "2022-10-08")
-    (rev "0.1.2")
+    (date "2023-01-22")
+    (rev "0.2.0")
     (company "Daniel Molina")
     (comment 1 "https://github.com/dmolinagarcia/74HCT6526")
@@
   (junction (at 152.4 109.22) (diameter 0) (color 0 0 0 0)
   )
-  (junction (at 210.82 119.38) (diameter 0) (color 0 0 0 0)
-  )
   (junction (at 144.78 73.66) (diameter 0) (color 0 0 0 0)
   )
   (junction (at 152.4 121.92) (diameter 0) (color 0 0 0 0)
   )
-  (junction (at 86.36 83.82) (diameter 0) (color 0 0 0 0)
-  )
   (junction (at 93.98 91.44) (diameter 0) (color 0 0 0 0)
+  )
+  (junction (at 233.68 114.3) (diameter 0) (color 0 0 0 0)
   )
   (junction (at 149.86 58.42) (diameter 0) (color 0 0 0 0)
@@
   (no_connect (at 180.34 127))
   (no_connect (at 114.3 78.74))
-  (no_connect (at 137.16 78.74))
   (no_connect (at 86.36 73.66))
   (no_connect (at 205.74 114.3))
@@
     (stroke (width 0) (type default) (color 0 0 0 0))
   )
-  (wire (pts (xy 86.36 83.82) (xy 78.74 83.82))
-    (stroke (width 0) (type default) (color 0 0 0 0))
-  )
-  (wire (pts (xy 210.82 127) (xy 210.82 119.38))
+  (wire (pts (xy 210.82 127) (xy 223.52 127))
     (stroke (width 0) (type default) (color 0 0 0 0))
   )
@@
     (stroke (width 0) (type default) (color 0 0 0 0))
   )
-  (wire (pts (xy 210.82 106.68) (xy 223.52 106.68))
-    (stroke (width 0) (type default) (color 0 0 0 0))
-  )
   (wire (pts (xy 180.34 58.42) (xy 195.58 58.42))
     (stroke (width 0) (type default) (color 0 0 0 0))
@@
     (stroke (width 0) (type default) (color 0 0 0 0))
   )
+  (wire (pts (xy 233.68 114.3) (xy 236.22 114.3))
+    (stroke (width 0) (type default) (color 0 0 0 0))
+  )
   (wire (pts (xy 93.98 91.44) (xy 93.98 76.2))
     (stroke (width 0) (type default) (color 0 0 0 0))
   )
+  (wire (pts (xy 78.74 83.82) (xy 78.74 90.17))
+    (stroke (width 0) (type default) (color 0 0 0 0))
+  )
   (wire (pts (xy 236.22 119.38) (xy 243.84 119.38))
     (stroke (width 0) (type default) (color 0 0 0 0))
   )
-  (wire (pts (xy 231.14 114.3) (xy 236.22 114.3))
+  (wire (pts (xy 231.14 114.3) (xy 233.68 114.3))
     (stroke (width 0) (type default) (color 0 0 0 0))
   )
@@
     (stroke (width 0) (type default) (color 0 0 0 0))
   )
-  (wire (pts (xy 198.12 127) (xy 210.82 127))
+  (wire (pts (xy 91.44 78.74) (xy 91.44 68.58))
+    (stroke (width 0) (type default) (color 0 0 0 0))
+  )
+  (wire (pts (xy 78.74 90.17) (xy 139.7 90.17))
     (stroke (width 0) (type default) (color 0 0 0 0))
   )
@@
     (stroke (width 0) (type default) (color 0 0 0 0))
   )
+  (wire (pts (xy 210.82 119.38) (xy 210.82 127))
+    (stroke (width 0) (type default) (color 0 0 0 0))
+  )
   (wire (pts (xy 137.16 132.08) (xy 154.94 132.08))
     (stroke (width 0) (type default) (color 0 0 0 0))
@@
     (stroke (width 0) (type default) (color 0 0 0 0))
   )
-  (wire (pts (xy 86.36 83.82) (xy 91.44 83.82))
-    (stroke (width 0) (type default) (color 0 0 0 0))
-  )
   (wire (pts (xy 180.34 66.04) (xy 195.58 66.04))
     (stroke (width 0) (type default) (color 0 0 0 0))
@@
     (stroke (width 0) (type default) (color 0 0 0 0))
   )
-  (wire (pts (xy 91.44 83.82) (xy 91.44 68.58))
-    (stroke (width 0) (type default) (color 0 0 0 0))
-  )
   (wire (pts (xy 152.4 114.3) (xy 152.4 116.84))
     (stroke (width 0) (type default) (color 0 0 0 0))
@@
     (stroke (width 0) (type default) (color 0 0 0 0))
   )
-  (wire (pts (xy 86.36 78.74) (xy 86.36 83.82))
-    (stroke (width 0) (type default) (color 0 0 0 0))
-  )
   (wire (pts (xy 180.34 76.2) (xy 195.58 76.2))
     (stroke (width 0) (type default) (color 0 0 0 0))
   )
+  (wire (pts (xy 137.16 78.74) (xy 139.7 78.74))
+    (stroke (width 0) (type default) (color 0 0 0 0))
+  )
   (wire (pts (xy 63.5 76.2) (xy 71.12 76.2))
     (stroke (width 0) (type default) (color 0 0 0 0))
   )
+  (wire (pts (xy 223.52 127) (xy 223.52 124.46))
+    (stroke (width 0) (type default) (color 0 0 0 0))
+  )
   (wire (pts (xy 78.74 127) (xy 78.74 96.52))
     (stroke (width 0) (type default) (color 0 0 0 0))
@@
     (stroke (width 0) (type default) (color 0 0 0 0))
   )
+  (wire (pts (xy 139.7 78.74) (xy 139.7 90.17))
+    (stroke (width 0) (type default) (color 0 0 0 0))
+  )
   (wire (pts (xy 91.44 127) (xy 91.44 129.54))
     (stroke (width 0) (type default) (color 0 0 0 0))
   )
+  (wire (pts (xy 233.68 132.08) (xy 233.68 114.3))
+    (stroke (width 0) (type default) (color 0 0 0 0))
+  )
+  (wire (pts (xy 86.36 78.74) (xy 91.44 78.74))
+    (stroke (width 0) (type default) (color 0 0 0 0))
+  )
   (wire (pts (xy 154.94 127) (xy 144.78 127))
     (stroke (width 0) (type default) (color 0 0 0 0))
@@
     (stroke (width 0) (type default) (color 0 0 0 0))
   )
-  (wire (pts (xy 210.82 119.38) (xy 210.82 106.68))
+  (wire (pts (xy 198.12 132.08) (xy 233.68 132.08))
     (stroke (width 0) (type default) (color 0 0 0 0))
   )
@@
     (stroke (width 0) (type default) (color 0 0 0 0))
   )
-  (wire (pts (xy 198.12 124.46) (xy 198.12 127))
+  (wire (pts (xy 198.12 124.46) (xy 198.12 132.08))
     (stroke (width 0) (type default) (color 0 0 0 0))
   )
@@
   )
   (wire (pts (xy 152.4 116.84) (xy 154.94 116.84))
-    (stroke (width 0) (type default) (color 0 0 0 0))
-  )
-  (wire (pts (xy 223.52 106.68) (xy 223.52 109.22))
     (stroke (width 0) (type default) (color 0 0 0 0))
   )
@@
     (pin "1")
   )
-  (symbol (lib_id "power:VCC") (at 223.52 124.46 180) (unit 1)
-    (in_bom yes) (on_board yes) (fields_autoplaced)
-    (property "Reference" "#PWR0318" (id 0) (at 223.52 120.65 0)
-      (effects (font (size 1.27 1.27)) hide)
-    )
-    (property "Value" "VCC" (id 1) (at 226.06 125.7299 0)
-      (effects (font (size 1.27 1.27)) (justify right))
-    )
-    (property "Footprint" "" (id 2) (at 223.52 124.46 0)
-      (effects (font (size 1.27 1.27)) hide)
-    )
-    (property "Datasheet" "" (id 3) (at 223.52 124.46 0)
-      (effects (font (size 1.27 1.27)) hide)
-    )
+  (symbol (lib_id "power:VCC") (at 223.52 109.22 0) (unit 1)
+    (in_bom yes) (on_board yes) (fields_autoplaced)
+    (property "Reference" "#PWR0318" (id 0) (at 223.52 113.03 0)
+      (effects (font (size 1.27 1.27)) hide)
+    )
+    (property "Value" "VCC" (id 1) (at 223.52 104.14 0))
+    (property "Footprint" "" (id 2) (at 223.52 109.22 0)
+      (effects (font (size 1.27 1.27)) hide)
+    )
+    (property "Datasheet" "" (id 3) (at 223.52 109.22 0)
+      (effects (font (size 1.27 1.27)) hide)
+    )

Commit message: .
Parts:
- U302: value 74HC125 -> 74HCT125
- U305: value 74HC74 -> 74HCT74
Changed lines of the file:
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@@
     (in_bom yes) (on_board yes) (fields_autoplaced)
     (property "Reference" "U302" (id 0) (at 129.54 41.91 0))
-    (property "Value" "74HC125" (id 1) (at 129.54 44.45 0))
+    (property "Value" "74HCT125" (id 1) (at 129.54 44.45 0))
     (property "Footprint" "Package_SO:SO-14_3.9x8.65mm_P1.27mm" (id 2) (at 129.54 50.8 0)
       (effects (font (size 1.27 1.27)) hide)
@@
       (effects (font (size 1.27 1.27)) (justify left))
     )
-    (property "Value" "74HC74" (id 1) (at 80.7594 68.58 0)
+    (property "Value" "74HCT74" (id 1) (at 80.7594 68.58 0)
       (effects (font (size 1.27 1.27)) (justify left))
     )
