File: B3/sdrRegister.kicad_sch (KiCad schematic)
At the start: 5 parts, among them U306 74HC32, U309 74HC00, U310 74HC244, U311 74HC377, U312 74HC244

Commit message: B3 added. First revision
Still not verified.
Connections:
- net ~{EN12}: now also U309.1; no longer U309.2
- net ~{RES}: now also U309.2; no longer U309.1
Changed lines of the file:
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@@
     (pin "1")
   )
-  (symbol (lib_id "74xx:74HC00") (at 48.26 129.54 0) (unit 1)
+  (symbol (lib_id "74xx:74HC00") (at 48.26 129.54 0) (mirror x) (unit 1)
     (in_bom yes) (on_board yes) (fields_autoplaced)
     (property "Reference" "U309" (id 0) (at 48.26 120.65 0))

Commit message: .
Parts:
- removed unit 3 of U309
- added U325: 74HC08, Package_SO:SO-14_3.9x8.65mm_P1.27mm, symbol Custom 74xx:74HC08
Connections:
- net ~{FULL}: now also U325.2
- net ~{WRITE}: now also U325.1
- net at U311.1 (~{E}): now also U325.3
Other:
- company: (none) -> Daniel Molina
- moved on the sheet: U306C
Changed lines of the file:
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@@
   (title_block
     (title "74HCT6526 Board 3")
-    (date "2022-09-11")
-    (rev "0.1")
+    (date "2022-10-08")
+    (rev "0.1.2")
+    (company "Daniel Molina")
+    (comment 1 "https://github.com/dmolinagarcia/74HCT6526")
+  )
+  (junction (at 76.2 97.79) (diameter 0) (color 0 0 0 0)
   )
   (junction (at 198.12 99.06) (diameter 0) (color 0 0 0 0)
   )
+  (junction (at 71.12 132.08) (diameter 0) (color 0 0 0 0)
+  )
   (junction (at 33.02 134.62) (diameter 0) (color 0 0 0 0)
   )
-  (junction (at 76.2 99.06) (diameter 0) (color 0 0 0 0)
-  )
   (junction (at 30.48 132.08) (diameter 0) (color 0 0 0 0)
   )
@@
     (stroke (width 0) (type default) (color 0 0 0 0))
   )
+  (wire (pts (xy 68.58 103.505) (xy 68.58 97.79))
+    (stroke (width 0) (type default) (color 0 0 0 0))
+  )
   (wire (pts (xy 106.68 86.36) (xy 124.46 86.36))
     (stroke (width 0) (type default) (color 0 0 0 0))
   )
+  (wire (pts (xy 76.2 97.79) (xy 76.2 96.52))
+    (stroke (width 0) (type default) (color 0 0 0 0))
+  )
   (wire (pts (xy 71.12 132.08) (xy 78.74 132.08))
     (stroke (width 0) (type default) (color 0 0 0 0))
@@
     (stroke (width 0) (type default) (color 0 0 0 0))
   )
-  (wire (pts (xy 27.94 114.3) (xy 73.66 114.3))
+  (wire (pts (xy 27.94 118.745) (xy 66.04 118.745))
     (stroke (width 0) (type default) (color 0 0 0 0))
   )
@@
     (stroke (width 0) (type default) (color 0 0 0 0))
   )
-  (wire (pts (xy 76.2 99.06) (xy 76.2 96.52))
+  (wire (pts (xy 76.2 99.06) (xy 76.2 97.79))
     (stroke (width 0) (type default) (color 0 0 0 0))
   )
@@
     (stroke (width 0) (type default) (color 0 0 0 0))
   )
-  (wire (pts (xy 78.74 114.3) (xy 78.74 132.08))
+  (wire (pts (xy 71.12 118.745) (xy 71.12 132.08))
     (stroke (width 0) (type default) (color 0 0 0 0))
   )
@@
   )
   (wire (pts (xy 27.94 154.94) (xy 86.36 154.94))
+    (stroke (width 0) (type default) (color 0 0 0 0))
+  )
+  (wire (pts (xy 68.58 97.79) (xy 76.2 97.79))
     (stroke (width 0) (type default) (color 0 0 0 0))
   )
@@
     (effects (font (size 1.27 1.27)) (justify left))
   )
-  (hierarchical_label "FULL" (shape input) (at 27.94 114.3 180)
+  (hierarchical_label "FULL" (shape input) (at 27.94 118.745 180)
     (effects (font (size 1.27 1.27)) (justify right))
   )
@@
     (pin "7")
   )
-  (symbol (lib_id "74xx:74HC00") (at 129.54 134.62 0) (unit 3)
-    (in_bom yes) (on_board yes) (fields_autoplaced)
-    (property "Reference" "U309" (id 0) (at 129.54 125.73 0))
-    (property "Value" "74HC00" (id 1) (at 129.54 128.27 0))
-    (property "Footprint" "Package_SO:SO-14_3.9x8.65mm_P1.27mm" (id 2) (at 129.54 134.62 0)
-      (effects (font (size 1.27 1.27)) hide)
-    )
-    (property "Datasheet" "http://www.ti.com/lit/gpn/sn74hc00" (id 3) (at 129.54 134.62 0)
-      (effects (font (size 1.27 1.27)) hide)
-    )
-    (pin "1")
-    (pin "2")
-    (pin "3")
-    (pin "4")
-    (pin "5")
-    (pin "6")
-    (pin "10")
-    (pin "8")
-    (pin "9")
-    (pin "11")
-    (pin "12")
-    (pin "13")
-    (pin "14")
-    (pin "7")
-  )
   (symbol (lib_id "power:GND") (at 162.56 106.68 0) (unit 1)
     (in_bom yes) (on_board yes) (fields_autoplaced)
@@
     (pin "9")
   )
-  (symbol (lib_id "74xx:74LS32") (at 76.2 106.68 270) (mirror x) (unit 3)
+  (symbol (lib_id "74xx:74LS32") (at 68.58 111.125 270) (mirror x) (unit 3)
     (in_bom yes) (on_board yes) (fields_autoplaced)
-    (property "Reference" "U306" (id 0) (at 81.28 105.4099 90)
+    (property "Reference" "U306" (id 0) (at 73.66 109.8549 90)
       (effects (font (size 1.27 1.27)) (justify left))
     )
-    (property "Value" "74HC32" (id 1) (at 81.28 107.9499 90)
+    (property "Value" "74HC32" (id 1) (at 73.66 112.3949 90)
       (effects (font (size 1.27 1.27)) (justify left))
     )
-    (property "Footprint" "Package_SO:SO-14_3.9x8.65mm_P1.27mm" (id 2) (at 76.2 106.68 0)
-      (effects (font (size 1.27 1.27)) hide)
-    )
-    (property "Datasheet" "http://www.ti.com/lit/gpn/sn74LS32" (id 3) (at 76.2 106.68 0)
-      (effects (font (size 1.27 1.27)) hide)
-    )
+    (property "Footprint" "Package_SO:SO-14_3.9x8.65mm_P1.27mm" (id 2) (at 68.58 111.125 0)
+      (effects (font (size 1.27 1.27)) hide)
+    )
+    (property "Datasheet" "http://www.ti.com/lit/gpn/sn74LS32" (id 3) (at 68.58 111.125 0)
+      (effects (font (size 1.27 1.27)) hide)
+    )
+    (pin "1")
+    (pin "2")
+    (pin "3")
+    (pin "4")
+    (pin "5")
+    (pin "6")
+    (pin "10")
+    (pin "8")
+    (pin "9")
+    (pin "11")
+    (pin "12")
+    (pin "13")
+    (pin "14")
+    (pin "7")
+  )
+  (symbol (lib_id "Custom 74xx:74HC08") (at 129.54 134.62 0) (unit 1)
+    (in_bom yes) (on_board yes) (fields_autoplaced)
+    (property "Reference" "U325" (id 0) (at 129.54 125.73 0))
+    (property "Value" "74HC08" (id 1) (at 129.54 128.27 0))
+    (property "Footprint" "Package_SO:SO-14_3.9x8.65mm_P1.27mm" (id 2) (at 129.54 134.62 0)
+      (effects (font (size 1.27 1.27)) hide)
+    )
+    (property "Datasheet" "" (id 3) (at 129.54 128.27 0)
+      (effects (font (size 1.27 1.27)) hide)
+    )
