File: B0/B0.kicad_pcb (KiCad board)
At the start: 4 copper layers, 100 x 100 mm, 76 parts, among them U001 74HCT00, U002 74HCT125, U003 74HCT244, U004 74HCT244, U005 74HCT244, U006 74HCT244, U007 74HCT32, U008 74HCT04, U009 74HCT00, U010 74HCT125, U011 74HCT04, U012 74HCT00, U013 74HCT125, U014 74HCT08, U015 74HCT04, U016 74HCT00, U017 74HCT125, U018 74HCT04, U019 74HCT00, U020 74HCT125, U021 74HCT08, U022 74HCT377, U023 74HCT377, U024 74HCT377, U025 74HCT377, U026 74HCT138, U027 74HCT138, U028 74HCT00, U029 74HCT00, U030 74HCT32, U031 74HCT00, U032 74HCT74

Commit message: v0.1.0 completed
Parts:
- GND1, GND2: value MountingHole_2.2mm_M2_DIN965_Pad -> GND
- VCC1, VCC2: value MountingHole_2.2mm_M2_DIN965_Pad -> VCC
Routing:
- net TOD: track 106.3 -> 107.0 mm
- net ~FLAG: track 111.6 -> 112.2 mm
Other:
- board text added: "74HCT6526 Board 0 v0.1.0"
- board text removed: "74HCT6526 Board 0 v0.1.1"

Commit message: B1 CREGA added
Work started on b1. CREGA added.
Minor changes to B0 schematic properties.
Connections:
- net /ddra/~OE2 renamed /ddra/~{OE2}
- net /ddra/~WE2 renamed /ddra/~{WE2}
- net /ddrb/~OE3 renamed /ddrb/~{OE3}
- net /ddrb/~WE3 renamed /ddrb/~{WE3}
- net /porta/~OE0 renamed /porta/~{OE0}
- net /porta/~WE0 renamed /porta/~{WE0}
- net /portb/~OE1 renamed /portb/~{OE1}
- net /portb/~WE1 renamed /portb/~{WE1}
- net /~CS renamed /~{CS}
- net /~PC renamed /~{PC}
- net /~PHI2 renamed /~{PHI2}
- net ~EN0 renamed ~{EN0}
- net ~EN1 renamed ~{EN1}
- net ~EN10 renamed ~{EN10}
- net ~EN11 renamed ~{EN11}
- net ~EN12 renamed ~{EN12}
- net ~EN13 renamed ~{EN13}
- net ~EN14 renamed ~{EN14}
- net ~EN15 renamed ~{EN15}
- net ~EN2 renamed ~{EN2}
- net ~EN3 renamed ~{EN3}
- net ~EN4 renamed ~{EN4}
- net ~EN5 renamed ~{EN5}
- net ~EN6 renamed ~{EN6}
- net ~EN7 renamed ~{EN7}
- net ~EN8 renamed ~{EN8}
- net ~EN9 renamed ~{EN9}
- net ~FLAG renamed ~{FLAG}
- net ~IRQ renamed ~{IRQ}
- net ~RES renamed ~{RES}

Commit message: B2 almost ready
Connections:
- net /DDRA0 renamed /ddra/DDRA0
- net /DDRA1 renamed /ddra/DDRA1
- net /DDRA2 renamed /ddra/DDRA2
- net /DDRA3 renamed /ddra/DDRA3
- net /DDRA4 renamed /ddra/DDRA4
- net /DDRA5 renamed /ddra/DDRA5
- net /DDRA6 renamed /ddra/DDRA6
- net /DDRA7 renamed /ddra/DDRA7
- net /DDRB0 renamed /ddrb/DDRB0
- net /DDRB1 renamed /ddrb/DDRB1
- net /DDRB2 renamed /ddrb/DDRB2
- net /DDRB3 renamed /ddrb/DDRB3
- net /DDRB4 renamed /ddrb/DDRB4
- net /DDRB5 renamed /ddrb/DDRB5
- net /DDRB6 renamed /ddrb/DDRB6
- net /DDRB7 renamed /ddrb/DDRB7
- net /PA0 renamed /icInterface/PA0
- net /PA1 renamed /icInterface/PA1
- net /PA2 renamed /icInterface/PA2
- net /PA3 renamed /icInterface/PA3
- net /PA4 renamed /icInterface/PA4
- net /PA5 renamed /icInterface/PA5
- net /PA6 renamed /icInterface/PA6
- net /PA7 renamed /icInterface/PA7
- net /PB0 renamed /icInterface/PB0
- net /PB1 renamed /icInterface/PB1
- net /PB2 renamed /icInterface/PB2
- net /PB3 renamed /icInterface/PB3
- net /PB4 renamed /icInterface/PB4
- net /PB5 renamed /icInterface/PB5
- net /PB6 renamed /icInterface/PB6
- net /PB7 renamed /icInterface/PB7
- net /RS0 renamed /icInterface/RS0
- net /RS1 renamed /icInterface/RS1
- net /RS2 renamed /icInterface/RS2
- net /RS3 renamed /icInterface/RS3
- net /~{CS} renamed /icInterface/~{CS}
- net /~{PC} renamed /icInterface/~{PC}
- U002 pad 8: no_connect_169 -> unconnected-(U002-Pad8)
- U008 pad 12: no_connect_170 -> unconnected-(U008-Pad12)
- U008 pad 2: no_connect_171 -> unconnected-(U008-Pad2)
- U015 pad 12: no_connect_172 -> unconnected-(U015-Pad12)
- U015 pad 2: no_connect_173 -> unconnected-(U015-Pad2)
- U018 pad 12: no_connect_174 -> unconnected-(U018-Pad12)
- U018 pad 2: no_connect_175 -> unconnected-(U018-Pad2)
- U030 pad 11: no_connect_176 -> unconnected-(U030-Pad11)
- U030 pad 3: no_connect_177 -> unconnected-(U030-Pad3)
- U032 pad 6: no_connect_178 -> unconnected-(U032-Pad6)
- U032 pad 8: no_connect_179 -> unconnected-(U032-Pad8)
- U032 pad 9: no_connect_180 -> unconnected-(U032-Pad9)
Routing:
- net GND: track 145.2 -> 140.6 mm
- net /icInterface/PB6: track 50.3 -> 48.1 mm
- net ~{EN2}: track 138.5 -> 136.3 mm
- net Net-(U008-Pad4): track 11.3 -> 9.61 mm
- net ~{EN1}: track 136.9 -> 135.2 mm
- net ENABLE_NAND: track 251.8 -> 250.4 mm
- net DZ6: track 97.8 -> 96.5 mm
- net D7: track 138.9 -> 137.8 mm
- net PB6ON: track 106.4 -> 105.7 mm
- net /icInterface/PA0: track 45.2 -> 44.5 mm
- net Net-(U031-Pad10): track 1.91 -> 1.27 mm
- net Net-(U011-Pad2): track 54.5 -> 53.8 mm
- net /portb/PBIN5: track 25.3 -> 24.7 mm
- net ~{EN0}: track 112.4 -> 111.9 mm
Other:
- board text added: "74HCT6526 Board 0 v0.1.1"
- board text removed: "74HCT6526 Board 0 v0.1.0"

Commit message: Almost 0.1.1
Routing:
- net TBOUT: track 38.4 -> 42.5 mm
- net GND: track 140.6 -> 138.1 mm, vias 81 -> 80
Changed lines of the file:
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@@
   (via (at 137.165 102.42) (size 0.5) (drill 0.2) (layers "F.Cu" "B.Cu") (net 12))
   (via (at 151.405 89.1) (size 0.5) (drill 0.2) (layers "F.Cu" "B.Cu") (net 12))
+  (segment (start 172.485 123.02) (end 177.435 123.02) (width 0.2) (layer "F.Cu") (net 13))
   (segment (start 168.37 81.48) (end 166.08 83.77) (width 0.2) (layer "F.Cu") (net 13))
   (segment (start 116.475 91.99) (end 113.87 91.99) (width 0.2) (layer "F.Cu") (net 13))
@@
   (segment (start 115.48 79.96) (end 113.87 79.96) (width 0.2) (layer "F.Cu") (net 13))
   (segment (start 156.225 102.47) (end 155.9465 102.47) (width 0.2) (layer "F.Cu") (net 13))
-  (segment (start 177.435 123.02) (end 179.27 123.02) (width 0.2) (layer "F.Cu") (net 13))
   (segment (start 188.6 54.26) (end 189.86 55.52) (width 0.2) (layer "F.Cu") (net 13))
   (segment (start 111.525 86.31) (end 110.21 86.31) (width 0.2) (layer "F.Cu") (net 13))
@@
   (segment (start 166.24 79.96) (end 166.44 79.76) (width 0.3048) (layer "F.Cu") (net 13))
   (segment (start 162.355 77.145) (end 162.33 77.17) (width 0.2) (layer "F.Cu") (net 13))
-  (segment (start 177.435 123.02) (end 172.485 123.02) (width 0.2) (layer "F.Cu") (net 13))
   (segment (start 154.65 86.325) (end 154.65 87.325) (width 0.2) (layer "F.Cu") (net 13))
   (segment (start 131.44 83.77) (end 132.06 83.15) (width 0.2) (layer "F.Cu") (net 13))
@@
   (segment (start 192.43 55.15) (end 192.43 53.19) (width 0.2) (layer "F.Cu") (net 13))
   (segment (start 132.16 95.04) (end 132.16 95.03) (width 0.2) (layer "F.Cu") (net 13))
+  (segment (start 177.435 124.29) (end 177.435 123.02) (width 0.2) (layer "F.Cu") (net 13))
   (segment (start 133.98 81.23) (end 135.475 81.23) (width 0.2) (layer "F.Cu") (net 13))
   (segment (start 110.35 115.715) (end 111.795 115.715) (width 0.2) (layer "F.Cu") (net 13))
@@
   (segment (start 121.025 99.555) (end 121.05 99.58) (width 0.2) (layer "F.Cu") (net 13))
   (segment (start 192.985 48.68) (end 192.985 48.685) (width 0.2) (layer "F.Cu") (net 13))
-  (segment (start 177.435 124.29) (end 179.24 124.29) (width 0.2) (layer "F.Cu") (net 13))
   (segment (start 136.475 120.705) (end 136.48 120.71) (width 0.2) (layer "F.Cu") (net 13))
   (segment (start 185.325 77.1) (end 185.34 77.1) (width 0.2) (layer "F.Cu") (net 13))
-  (segment (start 179.27 123.02) (end 179.28 123.03) (width 0.2) (layer "F.Cu") (net 13))
   (segment (start 132.16 98.3) (end 133.16 98.3) (width 0.2) (layer "F.Cu") (net 13))
   (segment (start 116.16 59.665) (end 116.145 59.665) (width 0.2) (layer "F.Cu") (net 13))
   (segment (start 165.205 91.96) (end 166.64 91.96) (width 0.2) (layer "F.Cu") (net 13))
-  (segment (start 179.24 124.29) (end 179.28 124.33) (width 0.2) (layer "F.Cu") (net 13))
   (segment (start 166.87 94.96) (end 168.6 93.23) (width 0.2) (layer "F.Cu") (net 13))
   (segment (start 179.475 120.09) (end 179.475 120.115) (width 0.2) (layer "F.Cu") (net 13))
@@
   (via (at 132.06 83.15) (size 0.5) (drill 0.2) (layers "F.Cu" "B.Cu") (net 13))
   (via (at 179.6 132.12) (size 0.5) (drill 0.2) (layers "F.Cu" "B.Cu") (net 13))
-  (via (at 179.28 123.03) (size 0.5) (drill 0.2) (layers "F.Cu" "B.Cu") (net 13))
   (via (at 173.69 102.4) (size 0.5) (drill 0.2) (layers "F.Cu" "B.Cu") (net 13))
   (via (at 163.23 62.09) (size 0.5) (drill 0.2) (layers "F.Cu" "B.Cu") (net 13))
@@
   (via (at 136.98 88.06) (size 0.5) (drill 0.2) (layers "F.Cu" "B.Cu") (net 13))
   (via (at 132.16 98.3) (size 0.5) (drill 0.2) (layers "F.Cu" "B.Cu") (net 13))
-  (via (at 179.28 124.33) (size 0.5) (drill 0.2) (layers "F.Cu" "B.Cu") (net 13))
+  (via (at 178.054 124.33) (size 0.5) (drill 0.2) (layers "F.Cu" "B.Cu") (net 13))
   (via (at 120.76 74.11) (size 0.5) (drill 0.2) (layers "F.Cu" "B.Cu") (net 13))
   (via (at 155.9365 102.48) (size 0.5) (drill 0.2) (layers "F.Cu" "B.Cu") (net 13))
@@
   (segment (start 187.06 56.79) (end 186.025 56.79) (width 0.127) (layer "F.Cu") (net 15))
   (segment (start 137.40802 130.131464) (end 137.40802 140.46802) (width 0.127) (layer "F.Cu") (net 15))
+  (segment (start 166.702 123.62) (end 171.704 118.618) (width 0.127) (layer "F.Cu") (net 16))
   (segment (start 152.435 123.02) (end 153.45 123.02) (width 0.127) (layer "F.Cu") (net 16))
+  (segment (start 171.704 118.618) (end 183.538 118.618) (width 0.127) (layer "F.Cu") (net 16))
   (segment (start 153.45 123.02) (end 154.05 123.62) (width 0.127) (layer "F.Cu") (net 16))
-  (segment (start 154.05 123.62) (end 188.54 123.62) (width 0.127) (layer "F.Cu") (net 16))
-  (segment (start 188.54 123.62) (end 189.96 125.04) (width 0.127) (layer "F.Cu") (net 16))
+  (segment (start 183.538 118.618) (end 189.96 125.04) (width 0.127) (layer "F.Cu") (net 16))
+  (segment (start 154.05 123.62) (end 166.702 123.62) (width 0.127) (layer "F.Cu") (net 16))
   (segment (start 169.75 48.12) (end 169.75 47.89) (width 0.127) (layer "F.Cu") (net 17))
   (segment (start 195.59807 60.670398) (end 195.59807 67.388846) (width 0.127) (layer "F.Cu") (net 17))
@@
   (segment (start 172.535 134.98) (end 171.845 134.98) (width 0.127) (layer "F.Cu") (net 173))
   (segment (start 151.47 136.25) (end 150.82 135.6) (width 0.127) (layer "F.Cu") (net 173))
+  (segment (start 132.42 124.8) (end 132.42 123.94) (width 0.127) (layer "F.Cu") (net 173))
   (segment (start 110.07 119.83) (end 106.44 116.2) (width 0.127) (layer "F.Cu") (net 173))
   (segment (start 152.465 136.28) (end 169.595 136.28) (width 0.127) (layer "F.Cu") (net 173))
@@
   (segment (start 110.4 119.83) (end 130.95 119.83) (width 0.127) (layer "F.Cu") (net 173))
   (segment (start 106.44 96.31) (end 106.44 64.09) (width 0.127) (layer "F.Cu") (net 173))
+  (segment (start 132.465 124.845) (end 132.42 124.8) (width 0.127) (layer "F.Cu") (net 173))
   (segment (start 132.42 121.3) (end 132.42 123.94) (width 0.127) (layer "F.Cu") (net 173))
-  (segment (start 132.42 124.85) (end 132.42 123.94) (width 0.127) (layer "F.Cu") (net 173))
   (segment (start 133.325 126.495) (end 132.42 125.59) (width 0.127) (layer "F.Cu") (net 173))
-  (segment (start 133.325 124.845) (end 134.575 124.845) (width 0.127) (layer "F.Cu") (net 173))
   (segment (start 109.22 62.505) (end 108.025 62.505) (width 0.127) (layer "F.Cu") (net 173))
   (segment (start 171.845 134.98) (end 170.545 136.28) (width 0.127) (layer "F.Cu") (net 173))
   (segment (start 151.54 136.25) (end 151.47 136.25) (width 0.127) (layer "F.Cu") (net 173))
   (segment (start 130.95 119.83) (end 132.42 121.3) (width 0.127) (layer "F.Cu") (net 173))
-  (segment (start 133.325 124.845) (end 133.32 124.85) (width 0.127) (layer "F.Cu") (net 173))
   (segment (start 110.4 119.83) (end 110.07 119.83) (width 0.127) (layer "F.Cu") (net 173))
   (segment (start 106.44 116.2) (end 106.44 114.65) (width 0.127) (layer "F.Cu") (net 173))
   (segment (start 106.44 114.65) (end 106.44 96.31) (width 0.127) (layer "F.Cu") (net 173))
   (segment (start 133.6 126.77) (end 133.325 126.495) (width 0.127) (layer "F.Cu") (net 173))
-  (segment (start 133.32 124.85) (end 132.42 124.85) (width 0.127) (layer "F.Cu") (net 173))
+  (segment (start 132.42 124.85) (end 132.42 124.8) (width 0.127) (layer "F.Cu") (net 173))
   (segment (start 135.93 126.77) (end 133.6 126.77) (width 0.127) (layer "F.Cu") (net 173))
   (segment (start 132.42 125.59) (end 132.42 124.85) (width 0.127) (layer "F.Cu") (net 173))
   (segment (start 144.76 135.6) (end 135.93 126.77) (width 0.127) (layer "F.Cu") (net 173))
   (segment (start 150.82 135.6) (end 144.76 135.6) (width 0.127) (layer "F.Cu") (net 173))
+  (segment (start 134.575 124.845) (end 132.465 124.845) (width 0.127) (layer "F.Cu") (net 173))
   (segment (start 152.435 136.25) (end 152.465 136.28) (width 0.127) (layer "F.Cu") (net 173))
   (segment (start 112.34 137.5) (end 110.42 135.58) (width 0.127) (layer "F.Cu") (net 174))

Commit message: .
Parts:
- added C033: 100n, Capacitor_SMD:C_0603_1608Metric, F.Cu at (187.2, 110.6)
Routing:
- net ~{RES}: track 166.7 -> 169.4 mm
- net GND: track 138.1 -> 139.1 mm, vias 80 -> 81
- net ~{EN4}: track 18.8 -> 19.3 mm
- net ~{EN5}: track 11.8 -> 12.4 mm
Other:
- board text added: "74HCT6526 Board 0 v0.1.2"
- board text removed: "74HCT6526 Board 0 v0.1.1"

Commit message: B0 ready for v0.2.0 release.
Parts:
- removed C033: 100n, Capacitor_SMD:C_0603_1608Metric
- added C000: 100n, Capacitor_SMD:C_0603_1608Metric, F.Cu at (187.2, 110.6)
Connections:
- CONTROLBUS0 pad 18: TARUNMODE -> unconnected-(CONTROLBUS0-Pad18)
Routing:
- net GND: track 139.1 -> 134.1 mm
- net /portb/PBIN0: track 31.6 -> 27.9 mm
- net ~{EN9}: track 15.9 -> 12.7 mm
- net DZ0: track 113.1 -> 109.9 mm
- net ~{EN1}: track 135.2 -> 132.3 mm
- net ~{EN3}: track 168.6 -> 165.8 mm
- net D7: track 137.8 -> 135.4 mm
- net ~{EN12}: track 14.1 -> 16.4 mm
- net /ddra/DDRA3: track 59.7 -> 57.5 mm
- net /icInterface/PB1: track 56.2 -> 58.4 mm
- net Net-(EXT1-Pad25): track 28.6 -> 26.5 mm
- net /icInterface/PA1: track 49.9 -> 47.9 mm
- net /icInterface/PB3: track 65.4 -> 67.4 mm
- net Net-(U015-Pad10): track 12.1 -> 10.2 mm
- net VCC: track 85.4 -> 83.6 mm
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Other:
- board text added: "74HCT6526 Board 0 v0.2.0"
- board text removed: "74HCT6526 Board 0 v0.1.2"
