File: B0/B0.kicad_sch (KiCad schematic)
At the start: 0 parts

Commit message: B1 CREGA added
Work started on b1. CREGA added.
Minor changes to B0 schematic properties.
Other:
- sheet ddra ports: added ~{EN2}, ~{RES}; removed ~EN2, ~RES
- sheet ddrb ports: added ~{EN3}, ~{RES}; removed ~EN3, ~RES
- sheet icInterface ports: added ~{CS}, ~{FLAG}, ~{IRQ}, ~{PC}, ~{PHI2}, ~{RES}; removed ~CS, ~FLAG, ~IRQ, ~PC, ~PHI2, ~RES
- sheet porta ports: added ~{EN0}, ~{PHI2}, ~{RES}; removed ~EN0, ~PHI2, ~RES
- sheet portb ports: added ~{EN1}, ~{PC}, ~{PHI2}, ~{RES}; removed ~EN1, ~PC, ~PHI2, ~RES
- sheet regDecoder ports: added ~{CS}, ~{EN[0..15]}, ~{PHI2}; removed ~CS, ~EN[0..15], ~PHI2
- sheet resetData ports: added ~{RES}; removed ~RES

Commit message: B2 almost ready
Other:
- sheet buses ports: added DZ[0..7], D[0..7], ~{EN[0..15]}; removed {DATABUS}, {ENABLEBUS}

Commit message: .
Changed lines of the file:
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@@
   (title_block
     (title "74HCT6526 Board 0")
-    (date "2022-08-17")
-    (rev "0.4")
+    (date "2022-10-08")
+    (rev "0.1.2")
     (company "Daniel Molina")
     (comment 1 "https://github.com/dmolinagarcia/74HCT6526")
@@
     (effects (font (size 1.27 1.27)) (justify left bottom))
   )
-  (label "~{PHI2}" (at 281.94 25.4 180)
+  (label "~{PHI2}" (at 284.48 25.4 180)
     (effects (font (size 1.27 1.27)) (justify right bottom))
   )
@@
       (reference "#PWR0114") (unit 1) (value "VCC") (footprint "")
     )
+    (path "/8ab4ca08-d71d-4254-8eb7-31fef72c2a95/abf49d68-554a-4336-9604-1b81f0c2389a"
+      (reference "#PWR0115") (unit 1) (value "GND") (footprint "")
+    )
     (path "/8d4bae2f-b118-40a6-8955-6b06f32615aa/d5d77f31-0456-4b05-b49a-1b52e4ace104"
       (reference "#PWR0123") (unit 1) (value "GND") (footprint "")
@@
       (reference "C032") (unit 1) (value "C") (footprint "74hct6526.footprints:0603_SMD")
     )
+    (path "/8ab4ca08-d71d-4254-8eb7-31fef72c2a95/182e5014-3833-462f-bbe2-3830e8c34674"
+      (reference "C033") (unit 1) (value "100n") (footprint "Capacitor_SMD:C_0603_1608Metric")
+    )
     (path "/8ab4ca08-d71d-4254-8eb7-31fef72c2a95/7f45c487-1782-49bd-9ad2-e522697f4099"
