File: B0/porta.kicad_sch (KiCad schematic)
At the start: 11 parts, among them U004 74HCT244, U007 74HCT32, U008 74HCT04, U009 74HCT00, U010 74HCT125, U015 74HCT04, U016 74HCT00, U017 74HCT125, U022 74HCT377, U031 74HCT00

Commit message: B1 CREGA added
Work started on b1. CREGA added.
Minor changes to B0 schematic properties.
Connections:
- net ~EN0 renamed ~{EN0}
- net ~OE0 renamed ~{OE0}
- net ~PHI2 renamed ~{PHI2}
- net ~RES renamed ~{RES}
- net ~WE0 renamed ~{WE0}

Commit message: Ready for v0.2.1
Parts:
- RN1: value R_Network08 -> 3k
Changed lines of the file:
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@@
   (title_block
     (title "74HCT6526 Board 0")
-    (date "2023-01-22")
-    (rev "0.2.0")
+    (date "2023-03-25")
+    (rev "0.2.1")
     (company "Daniel Molina")
     (comment 1 "https://github.com/dmolinagarcia/74HCT6526")
@@
     (in_bom yes) (on_board yes)
     (property "Reference" "RN1" (id 0) (at 232.41 23.7298 90))
-    (property "Value" "R_Network08" (id 1) (at 232.41 26.0285 90))
+    (property "Value" "3k" (id 1) (at 232.41 26.0285 90))
     (property "Footprint" "Resistor_THT:R_Array_SIP9" (id 2) (at 232.41 51.435 90)
       (effects (font (size 1.27 1.27)) hide)

Commit message: .
Parts:
- U004: value 74HCT244 -> 74HC244
- U007: value 74HCT32 -> 74HC32
- U008, U015: value 74HCT04 -> 74HC04
- U009, U016, U031: value 74HCT00 -> 74HC00
- U010, U017: value 74HCT125 -> 74HC125
- U022: value 74HCT377 -> 74HC377
