File: B0/portb.kicad_sch (KiCad schematic)
At the start: 15 parts, among them U006 74HCT244, U007 74HCT32, U011 74HCT04, U012 74HCT00, U013 74HCT125, U018 74HCT04, U019 74HCT00, U020 74HCT125, U024 74HCT377, U028 74HCT00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

Commit message: B1 CREGA added
Work started on b1. CREGA added.
Minor changes to B0 schematic properties.
Connections:
- net ~EN1 renamed ~{EN1}
- net ~OE1 renamed ~{OE1}
- net ~PC renamed ~{PC}
- net ~PHI2 renamed ~{PHI2}
- net ~RES renamed ~{RES}
- net ~WE1 renamed ~{WE1}

Commit message: Ready for v0.2.1
Parts:
- RN2: value R_Network08 -> 1k
Changed lines of the file:
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@@
   (title_block
     (title "74HCT6526 Board 0")
-    (date "2023-01-22")
-    (rev "0.2.0")
+    (date "2023-03-25")
+    (rev "0.2.1")
     (company "Daniel Molina")
     (comment 1 "https://github.com/dmolinagarcia/74HCT6526")
@@
     (in_bom yes) (on_board yes)
     (property "Reference" "RN2" (id 0) (at 229.87 51.2002 90))
-    (property "Value" "R_Network08" (id 1) (at 229.87 48.9015 90))
+    (property "Value" "1k" (id 1) (at 229.87 48.9015 90))
     (property "Footprint" "Resistor_THT:R_Array_SIP9" (id 2) (at 229.87 23.495 90)
       (effects (font (size 1.27 1.27)) hide)

Commit message: .
Parts:
- U006: value 74HCT244 -> 74HC244
- U007, U030: value 74HCT32 -> 74HC32
- U011, U018: value 74HCT04 -> 74HC04
- U012, U019, U028, U029, U031: value 74HCT00 -> 74HC00
- U013, U020: value 74HCT125 -> 74HC125
- U024: value 74HCT377 -> 74HC377
- U032: value 74HCT74 -> 74HC74
