File: B0/regDecoder.kicad_sch (KiCad schematic)
At the start: 2 parts, among them U026 74HCT138, U027 74HCT138

Commit message: B1 CREGA added
Work started on b1. CREGA added.
Minor changes to B0 schematic properties.
Connections:
- net ~CS renamed ~{CS}
- net ~EN0 renamed ~{EN0}
- net ~EN1 renamed ~{EN1}
- net ~EN10 renamed ~{EN10}
- net ~EN11 renamed ~{EN11}
- net ~EN12 renamed ~{EN12}
- net ~EN13 renamed ~{EN13}
- net ~EN14 renamed ~{EN14}
- net ~EN15 renamed ~{EN15}
- net ~EN2 renamed ~{EN2}
- net ~EN3 renamed ~{EN3}
- net ~EN4 renamed ~{EN4}
- net ~EN5 renamed ~{EN5}
- net ~EN6 renamed ~{EN6}
- net ~EN7 renamed ~{EN7}
- net ~EN8 renamed ~{EN8}
- net ~EN9 renamed ~{EN9}
- net ~PHI2 renamed ~{PHI2}
