File: B2/B2.kicad_pcb (KiCad board)
At the start: 4 copper layers, 100 x 100 mm, 65 parts, among them U201 74HC244, U202 74HC244, U203 74HCT32, U204 74HCT32, U205 74HC244, U206 74HC688, U207 74HC688, U208 74HC32, U209 74HC74, U210 74HC04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

Commit message: Updates to B3
Routing:
- net ~{RES}: track 157.4 -> 155.8 mm
- net /resetData/DO6: track 140.6 -> 141.3 mm
- net /resetData/DO1: track 136.6 -> 137.3 mm
- net /resetData/DO7: track 134.6 -> 135.3 mm
- net /TBINMODE0: track 75.1 -> 75.6 mm
- net DZ0: track 54.4 -> 54.9 mm

Commit message: Added ICR. B2 fixes
Parts:
- U229: value 74HC08 -> 74HCT08
Changed lines of the file:
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@@
       (effects (font (size 1 1) (thickness 0.15)))
     )
-    (fp_text value "74HC244" (at 0 7.35) (layer "F.Fab")
+    (fp_text value "74HC244" (at 0 7.35) (layer "F.SilkS")
       (effects (font (size 1 1) (thickness 0.15)))
     )
@@
       (effects (font (size 1 1) (thickness 0.15)))
     )
-    (fp_text value "74HC08" (at 0 5.28) (layer "F.SilkS")
-      (effects (font (size 1 1) (thickness 0.15)))
-    )
+    (fp_text value "74HCT08" (at 0 5.28) (layer "F.SilkS")
+      (effects (font (size 1 1) (thickness 0.15)))
+    )

Commit message: .
Parts:
- added C230: 100n, Capacitor_SMD:C_0603_1608Metric, F.Cu at (189.9, 105.9)
Routing:
- net ~{RES}: track 155.8 -> 157.6 mm
- net GND: track 205.0 -> 205.1 mm, vias 64 -> 65
Other:
- board text added: "74HCT6526 Board 2 v0.1.2"
- board text removed: "74HCT6526 Board 2 v0.1.1"
Changed lines of the file:
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@@
   )
   (footprint "Capacitor_SMD:C_0603_1608Metric" (layer "F.Cu")
+    (at 189.94 105.94 90)
+    (descr "Capacitor SMD 0603 (1608 Metric), square (rectangular) end terminal, IPC_7351 nominal, (Body size source: IPC-SM-782 page 76, https://www.pcb-3d.com/wordpress/wp-content/uploads/ipc-sm-782a_amendment_1_and_2.pdf), generated with kicad-footprint-generator")
+    (tags "capacitor")
+    (property "Sheetfile" "buses.kicad_sch")
+    (property "Sheetname" "buses")
+    (attr smd)
+    (fp_text reference "C230" (at 0 -1.43 90) (layer "F.Fab")
+      (effects (font (size 1 1) (thickness 0.15)))
+    )
+    (fp_text value "100n" (at 0 1.43 90) (layer "F.Fab")
+      (effects (font (size 1 1) (thickness 0.15)))
+    )
+    (fp_text user "${REFERENCE}" (at 0 0 90) (layer "F.Fab")
+      (effects (font (size 0.4 0.4) (thickness 0.06)))
+    )
+    (fp_line (start -0.14058 0.51) (end 0.14058 0.51) (layer "F.SilkS") (width 0.12))
+    (fp_line (start -0.14058 -0.51) (end 0.14058 -0.51) (layer "F.SilkS") (width 0.12))
+    (fp_line (start 1.48 -0.73) (end 1.48 0.73) (layer "F.CrtYd") (width 0.05))
+    (fp_line (start 1.48 0.73) (end -1.48 0.73) (layer "F.CrtYd") (width 0.05))
+    (fp_line (start -1.48 -0.73) (end 1.48 -0.73) (layer "F.CrtYd") (width 0.05))
+    (fp_line (start -1.48 0.73) (end -1.48 -0.73) (layer "F.CrtYd") (width 0.05))
+    (fp_line (start -0.8 -0.4) (end 0.8 -0.4) (layer "F.Fab") (width 0.1))
+    (fp_line (start -0.8 0.4) (end -0.8 -0.4) (layer "F.Fab") (width 0.1))
+    (fp_line (start 0.8 -0.4) (end 0.8 0.4) (layer "F.Fab") (width 0.1))
+    (fp_line (start 0.8 0.4) (end -0.8 0.4) (layer "F.Fab") (width 0.1))
+    (pad "1" smd roundrect (at -0.775 0 90) (size 0.9 0.95) (layers "F.Cu" "F.Paste" "F.Mask") (roundrect_rratio 0.25)
+      (net 20 "~{RES}") (pintype "passive"))
+    (pad "2" smd roundrect (at 0.775 0 90) (size 0.9 0.95) (layers "F.Cu" "F.Paste" "F.Mask") (roundrect_rratio 0.25)
+      (net 30 "GND") (pintype "passive"))
+    (model "${KICAD6_3DMODEL_DIR}/Capacitor_SMD.3dshapes/C_0603_1608Metric.wrl"
+      (offset (xyz 0 0 0))
+      (scale (xyz 1 1 1))
+      (rotate (xyz 0 0 0))
+    )
+  )
+  (footprint "Capacitor_SMD:C_0603_1608Metric" (layer "F.Cu")
     (at 119.888 47.8282)
     (descr "Capacitor SMD 0603 (1608 Metric), square (rectangular) end terminal, IPC_7351 nominal, (Body size source: IPC-SM-782 page 76, https://www.pcb-3d.com/wordpress/wp-content/uploads/ipc-sm-782a_amendment_1_and_2.pdf), generated with kicad-footprint-generator")
@@
       (effects (font (size 1 1) (thickness 0.15)))
     )
-    (fp_text value "74HC74" (at 0 5.28) (layer "F.Fab")
+    (fp_text value "74HC74" (at -4.72722 0.37 90) (layer "F.SilkS")
       (effects (font (size 1 1) (thickness 0.15)))
     )
@@
     (property "Sheetname" "power")
     (attr smd)
-    (fp_text reference "C307" (at 0 -1.43) (layer "F.SilkS")
+    (fp_text reference "C307" (at 0 -1.43) (layer "F.Fab")
       (effects (font (size 1 1) (thickness 0.15)))
     )
@@
   (gr_line (start 99.981802 45.005538) (end 99.981802 145.005538) (layer "Edge.Cuts") (width 0.05))
   (gr_line (start 199.981802 145.005538) (end 199.981802 45.005538) (layer "Edge.Cuts") (width 0.05))
-  (gr_text "74HCT6526\nBoard 2\nv0.1.1" (at 149.86 140.716) (layer "F.SilkS")
+  (gr_text "74HCT6526\nBoard 2\nv0.1.2" (at 149.86 140.716) (layer "F.SilkS")
     (effects (font (size 1 1) (thickness 0.25) italic))
   )
@@
   (segment (start 163.576 130.048) (end 162.814 130.81) (width 0.127) (layer "B.Cu") (net 16))
   (segment (start 167.089079 68.448179) (end 165.65222 68.448179) (width 0.127) (layer "F.Cu") (net 20))
+  (segment (start 191.75083 106.715) (end 191.757915 106.722085) (width 0.127) (layer "F.Cu") (net 20))
   (segment (start 179.961411 73.528179) (end 184.272179 73.528179) (width 0.127) (layer "F.Cu") (net 20))
   (segment (start 191.757915 108.002085) (end 189.96 109.8) (width 0.127) (layer "F.Cu") (net 20))
+  (segment (start 191.757915 106.722085) (end 191.757915 108.002085) (width 0.127) (layer "F.Cu") (net 20))
   (segment (start 145.411161 126.9112) (end 147.2312 126.9112) (width 0.127) (layer "F.Cu") (net 20))
   (segment (start 163.068 68.58) (end 163.199821 68.448179) (width 0.127) (layer "F.Cu") (net 20))
+  (segment (start 191.757915 93.930587) (end 191.757915 106.722085) (width 0.127) (layer "F.Cu") (net 20))
   (segment (start 147.2312 126.9112) (end 148.5012 128.1812) (width 0.127) (layer "F.Cu") (net 20))
   (segment (start 148.5012 128.1812) (end 150.361161 128.1812) (width 0.127) (layer "F.Cu") (net 20))
@@
   (segment (start 179.961411 73.528179) (end 178.938179 73.528179) (width 0.127) (layer "F.Cu") (net 20))
   (segment (start 187.35349 89.526162) (end 191.757915 93.930587) (width 0.127) (layer "F.Cu") (net 20))
-  (segment (start 191.757915 93.930587) (end 191.757915 108.002085) (width 0.127) (layer "F.Cu") (net 20))
   (segment (start 158.776166 121.909074) (end 158.75762 121.92762) (width 0.127) (layer "F.Cu") (net 20))
   (segment (start 171.600134 72.959234) (end 167.089079 68.448179) (width 0.127) (layer "F.Cu") (net 20))
@@
   (segment (start 150.361161 128.1812) (end 154.12984 128.1812) (width 0.127) (layer "F.Cu") (net 20))
   (segment (start 154.12984 128.1812) (end 157.85084 131.9022) (width 0.127) (layer "F.Cu") (net 20))
+  (segment (start 189.94 106.715) (end 191.75083 106.715) (width 0.127) (layer "F.Cu") (net 20))
   (via (at 158.75 138.176) (size 0.5) (drill 0.2) (layers "F.Cu" "B.Cu") (net 20))
   (via (at 163.068 68.58) (size 0.5) (drill 0.2) (layers "F.Cu" "B.Cu") (net 20))
@@
   (segment (start 165.60142 86.2306) (end 165.60142 87.5006) (width 0.127) (layer "F.Cu") (net 30))
   (segment (start 167.6784 108.458) (end 167.64 108.458) (width 0.127) (layer "F.Cu") (net 30))
+  (segment (start 189.94 105.165) (end 189.820283 105.165) (width 0.254) (layer "F.Cu") (net 30))
   (segment (start 118.636411 71.0767) (end 125.846411 71.0767) (width 0.127) (layer "F.Cu") (net 30))
   (segment (start 160.65142 81.1506) (end 160.65142 82.4206) (width 0.127) (layer "F.Cu") (net 30))
@@
   (segment (start 133.809759 105.309876) (end 132.980651 105.31094) (width 0.254) (layer "F.Cu") (net 30))
   (segment (start 135.146411 76.1567) (end 136.9493 76.1567) (width 0.127) (layer "F.Cu") (net 30))
+  (segment (start 189.820283 105.165) (end 189.805283 105.18) (width 0.254) (layer "F.Cu") (net 30))
   (segment (start 146.558 82.5246) (end 147.05076 83.01736) (width 0.127) (layer "F.Cu") (net 30))
   (segment (start 135.146411 73.6167) (end 136.95668 73.6167) (width 0.127) (layer "F.Cu") (net 30))
@@
   (via (at 152.4254 65.1256) (size 0.5) (drill 0.2) (layers "F.Cu" "B.Cu") (net 30))
   (via (at 110.0328 79.9592) (size 0.5) (drill 0.2) (layers "F.Cu" "B.Cu") (net 30))
+  (via (at 189.805283 105.18) (size 0.5) (drill 0.2) (layers "F.Cu" "B.Cu") (net 30))
   (via (at 161.2646 104.9528) (size 0.5) (drill 0.2) (layers "F.Cu" "B.Cu") (net 30))
   (via (at 173.5074 61.341) (size 0.5) (drill 0.2) (layers "F.Cu" "B.Cu") (net 30))

Commit message: B0 ready for v0.2.0 release.
Connections:
- U221 pad 10: Net-(U221-Pad1) -> Net-(U221-Pad10)
- U221 pad 6: Net-(U221-Pad1) -> Net-(U221-Pad10)
- U221 pad 8: unconnected-(U221-Pad8) -> Net-(U221-Pad1)
Routing:
- net Net-(U221-Pad10): track 0.00 -> 5.48 mm
- net VCC: track 203.8 -> 199.8 mm, vias 42 -> 43
- net Net-(U216-Pad2): track 29.2 -> 28.6 mm

Commit message: B2 ready for v0.2.0 release
Parts:
- removed C230: 100n, Capacitor_SMD:C_0603_1608Metric
- added C200: 100n, Capacitor_SMD:C_0603_1608Metric, F.Cu at (189.9, 105.9)
Connections:
- CONTROLBUS2 pad 18: TARUNMODE -> unconnected-(CONTROLBUS2-Pad18)
Routing:
- net PHI2: track 171.2 -> 162.0 mm, vias 7 -> 6
- net Net-(U223-Pad11): track 41.5 -> 48.3 mm
- net GND: track 205.1 -> 201.0 mm
- net TBOUT: track 64.2 -> 61.6 mm
- net ~{RES}: track 157.6 -> 155.2 mm
- net /TBINMODE1: track 83.7 -> 86.1 mm
- net DZ1: track 64.6 -> 66.3 mm
- net VCC: track 199.8 -> 198.1 mm
- net D2: track 99.3 -> 97.6 mm
- net /cregb/WE14: track 80.0 -> 78.5 mm
- net TBPULSE: track 78.2 -> 76.8 mm
- net DZ5: track 64.1 -> 65.4 mm
- net DZ7: track 61.5 -> 62.7 mm
- net DZ4: track 53.9 -> 54.9 mm
- net DZ0: track 54.9 -> 56.0 mm
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Other:
- board text added: "74HCT6526 Board 2 v0.2.0"
- board text removed: "74HCT6526 Board 2 v0.1.2"

Commit message: Ready for v0.2.1
Parts:
- added C202: 100n, Capacitor_SMD:C_0603_1608Metric, F.Cu at (157.6, 79.4)
- added U230: 74HC74, Package_SO:SO-14_3.9x8.65mm_P1.27mm, F.Cu at (153.7, 85.0)
- moved U211 3.05 mm to (144.9, 85.0)
- moved C304 3.05 mm to (148.6, 79.3)
Connections:
- U211 pad 10: /TBLOAD -> /cregb/TBUNDERFLOW
- U211 pad 9: /cregb/TBUNDERFLOW -> /TBLOAD
- U216 pad 13: Net-(U211-Pad8) -> /timerb/TBPULSESET
- U217 pad 11: /~{PHI2} -> VCC
- U217 pad 13: Net-(U211-Pad8) -> VCC
- U217 pad 9: Net-(U217-Pad9) -> unconnected-(U217-Pad9)
- U229 pad 4: Net-(U217-Pad9) -> Net-(U229-Pad4)
Routing:
- net Net-(U229-Pad4): track 0.00 -> 58.9 mm, vias 0 -> 2
- net Net-(U217-Pad9): track 37.6 -> 0.00 mm, vias 2 -> 0
- net /timerb/TBPULSESET: track 24.8 -> 57.5 mm, vias 2 -> 3
- net /~{PHI2}: track 172.3 -> 197.3 mm, vias 4 -> 6
- net Net-(U211-Pad8): track 29.4 -> 16.0 mm
- net VCC: track 198.1 -> 210.9 mm, vias 43 -> 44
- net Net-(U230-Pad2): track 0.00 -> 11.5 mm
- net /cregb/TBUNDERFLOW: track 101.7 -> 110.4 mm
- net /TBLOAD: track 45.6 -> 53.2 mm
- net /timerb/TBSTART: track 72.2 -> 76.4 mm
- net GND: track 201.0 -> 197.3 mm, vias 65 -> 66
- net /TBOUTMODE: track 101.4 -> 104.1 mm
- net /TBINMODE1: track 86.1 -> 83.8 mm
- net /timerb/timer16/~{TIMER_UNDERFLOW}: track 20.2 -> 18.8 mm
- net /timerb/~{WETBHI}: track 107.6 -> 108.6 mm
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Other:
- board text added: "74HCT6526 Board 2 v0.2.1"
- board text removed: "74HCT6526 Board 2 v0.2.0"
