File: B2/B2.kicad_sch (KiCad schematic)
At the start: 0 parts

Commit message: B2 almost ready
Parts:
- added U302: 74HC04, Package_SO:SOIC-14_3.9x8.7mm_P1.27mm, symbol 74xx:74HC04
Connections:
- new net PHI2: U302.1
- new net ~{PHI2}: U302.2
Other:
- added sheet cregb (cregb.kicad_sch)
- added sheet power (power.kicad_sch)
- added sheet resetData (resetData.kicad_sch)
- added sheet timerb (timerb.kicad_sch)
- sheet buses ports: added DZ[0..7], D[0..7], ~{EN[0..15]}; removed {DATABUS}, {ENABLEBUS}
- company: (none) -> Daniel Molina
- title: (none) -> 74HCT6526 Board 1

Commit message: Almost 0.1.1
Parts:
- renumbered U302 to U210
Other:
- title: 74HCT6526 Board 1 -> 74HCT6526 Board 2
