File: B2/buses.kicad_sch (KiCad schematic)
At the start: 3 parts

Commit message: B1 CREGA added
Work started on b1. CREGA added.
Minor changes to B0 schematic properties.
Connections:
- net ~EN10 renamed ~{EN10}
- net ~EN11 renamed ~{EN11}
- net ~EN12 renamed ~{EN12}
- net ~EN13 renamed ~{EN13}
- net ~EN14 renamed ~{EN14}
- net ~EN15 renamed ~{EN15}
- net ~EN4 renamed ~{EN4}
- net ~EN5 renamed ~{EN5}
- net ~EN6 renamed ~{EN6}
- net ~EN7 renamed ~{EN7}
- net ~EN8 renamed ~{EN8}
- net ~EN9 renamed ~{EN9}
- net ~FLAG renamed ~{FLAG}
- net ~IRQ renamed ~{IRQ}
- net ~RES renamed ~{RES}

Commit message: B2 almost ready
Parts:
- renumbered CONTROLBUS3 to CONTROLBUS2, DATABUS3 to DATABUS2, ENABLEBUS3 to ENABLEBUS2
Changed lines of the file:
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@@
   (junction (at 152.4 81.28) (diameter 1.016) (color 0 0 0 0)
   )
+  (junction (at 134.62 99.695) (diameter 0) (color 0 0 0 0)
+  )
   (junction (at 111.76 78.74) (diameter 1.016) (color 0 0 0 0)
   )
@@
     (stroke (width 0) (type solid) (color 0 0 0 0))
   )
+  (bus (pts (xy 134.62 88.9) (xy 134.62 99.695))
+    (stroke (width 0) (type default) (color 0 0 0 0))
+  )
   (wire (pts (xy 165.1 68.58) (xy 177.8 68.58))
     (stroke (width 0) (type solid) (color 0 0 0 0))
@@
     (stroke (width 0) (type solid) (color 0 0 0 0))
   )
-  (bus (pts (xy 134.62 73.66) (xy 134.62 81.28))
-    (stroke (width 0) (type solid) (color 0 0 0 0))
-  )
   (bus (pts (xy 180.34 35.56) (xy 180.34 66.04))
     (stroke (width 0) (type solid) (color 0 0 0 0))
@@
     (stroke (width 0) (type solid) (color 0 0 0 0))
   )
+  (bus (pts (xy 134.62 99.695) (xy 180.34 99.695))
+    (stroke (width 0) (type default) (color 0 0 0 0))
+  )
   (wire (pts (xy 81.28 83.82) (xy 99.06 83.82))
     (stroke (width 0) (type solid) (color 0 0 0 0))
   )
+  (bus (pts (xy 27.94 99.695) (xy 134.62 99.695))
+    (stroke (width 0) (type default) (color 0 0 0 0))
+  )
   (wire (pts (xy 165.1 76.2) (xy 177.8 76.2))
     (stroke (width 0) (type solid) (color 0 0 0 0))
   )
-  (bus (pts (xy 180.34 73.66) (xy 180.34 81.28))
-    (stroke (width 0) (type solid) (color 0 0 0 0))
-  )
   (bus (pts (xy 78.74 38.1) (xy 78.74 66.04))
     (stroke (width 0) (type solid) (color 0 0 0 0))
@@
     (stroke (width 0) (type solid) (color 0 0 0 0))
   )
+  (bus (pts (xy 180.34 99.695) (xy 180.34 88.9))
+    (stroke (width 0) (type default) (color 0 0 0 0))
+  )
   (bus (pts (xy 208.28 81.28) (xy 208.28 83.82))
     (stroke (width 0) (type solid) (color 0 0 0 0))
@@
     (effects (font (size 1.27 1.27)) (justify right bottom))
   )
-  (label "{ENABLEBUS}" (at 132.08 38.1 180)
-    (effects (font (size 1.27 1.27)) (justify right bottom))
-  )
   (label "ENABLE_NAND" (at 251.46 86.36 180)
     (effects (font (size 1.27 1.27)) (justify right bottom))
@@
     (effects (font (size 1.27 1.27)) (justify right bottom))
   )
-  (label "{DATABUS}" (at 180.34 35.56 180)
-    (effects (font (size 1.27 1.27)) (justify right bottom))
-  )
   (label "ALARM" (at 251.46 83.82 180)
     (effects (font (size 1.27 1.27)) (justify right bottom))
@@
     (effects (font (size 1.27 1.27)) (justify right bottom))
   )
-  (hierarchical_label "{DATABUS}" (shape bidirectional) (at 27.94 35.56 180)
+  (hierarchical_label "D[0..7]" (shape bidirectional) (at 27.94 35.56 180)
     (effects (font (size 1.27 1.27)) (justify right))
   )
-  (hierarchical_label "{ENABLEBUS}" (shape input) (at 27.94 38.1 180)
+  (hierarchical_label "~{EN[0..15]}" (shape output) (at 27.94 38.1 180)
     (effects (font (size 1.27 1.27)) (justify right))
   )
@@
     (effects (font (size 1.27 1.27)) (justify right))
   )
+  (hierarchical_label "DZ[0..7]" (shape bidirectional) (at 27.94 99.695 180)
+    (effects (font (size 1.27 1.27)) (justify right))
+  )
   (symbol (lib_id "power:GND") (at 118.11 83.82 0) (unit 1)
     (in_bom yes) (on_board yes)
-    (property "Reference" "#PWR010" (id 0) (at 118.11 90.17 0)
+    (property "Reference" "#PWR0303" (id 0) (at 118.11 90.17 0)
       (effects (font (size 1.27 1.27)) hide)
     )
@@
   (symbol (lib_id "Connector_Generic:Conn_02x10_Odd_Even") (at 231.14 78.74 0) (unit 1)
     (in_bom yes) (on_board yes)
-    (property "Reference" "CONTROLBUS3" (id 0) (at 232.41 63.1 0))
+    (property "Reference" "CONTROLBUS2" (id 0) (at 232.41 63.1 0))
     (property "Value" "Conn_02x10_Odd_Even" (id 1) (at 232.41 65.3985 0))
     (property "Footprint" "Connector_PinHeader_2.54mm:PinHeader_2x10_P2.54mm_Vertical" (id 2) (at 231.14 78.74 0)
@@
   (symbol (lib_id "Connector_Generic:Conn_02x10_Odd_Even") (at 157.48 78.74 0) (unit 1)
     (in_bom yes) (on_board yes)
-    (property "Reference" "DATABUS3" (id 0) (at 158.75 63.1 0))
+    (property "Reference" "DATABUS2" (id 0) (at 158.75 63.1 0))
     (property "Value" "Conn_02x10_Odd_Even" (id 1) (at 158.75 65.3985 0))
     (property "Footprint" "Connector_PinHeader_2.54mm:PinHeader_2x10_P2.54mm_Vertical" (id 2) (at 157.48 78.74 0)
@@
   (symbol (lib_id "power:VCC") (at 143.51 81.28 0) (unit 1)
     (in_bom yes) (on_board yes)
-    (property "Reference" "#PWR011" (id 0) (at 143.51 85.09 0)
+    (property "Reference" "#PWR0304" (id 0) (at 143.51 85.09 0)
       (effects (font (size 1.27 1.27)) hide)
     )
@@
   (symbol (lib_id "Connector_Generic:Conn_02x10_Odd_Even") (at 104.14 78.74 0) (unit 1)
     (in_bom yes) (on_board yes)
-    (property "Reference" "ENABLEBUS3" (id 0) (at 105.41 63.1 0))
+    (property "Reference" "ENABLEBUS2" (id 0) (at 105.41 63.1 0))
     (property "Value" "Conn_02x10_Odd_Even" (id 1) (at 105.41 65.3985 0))
     (property "Footprint" "Connector_PinHeader_2.54mm:PinHeader_2x10_P2.54mm_Vertical" (id 2) (at 104.14 78.74 0)
@@
   (symbol (lib_id "power:VCC") (at 118.11 81.28 0) (unit 1)
     (in_bom yes) (on_board yes)
-    (property "Reference" "#PWR09" (id 0) (at 118.11 85.09 0)
+    (property "Reference" "#PWR0302" (id 0) (at 118.11 85.09 0)
       (effects (font (size 1.27 1.27)) hide)
     )
@@
   (symbol (lib_id "power:GND") (at 175.26 78.74 0) (unit 1)
     (in_bom yes) (on_board yes)
-    (property "Reference" "#PWR012" (id 0) (at 175.26 85.09 0)
-      (effects (font (size 1.27 1.27)) hide)
-    )
+    (property "Reference" "#PWR0305" (id 0) (at 175.26 85.09 0)
+      (effects (font (size 1.27 1.27)) hide)
+    )

Commit message: Almost 0.1.1
Other:
- company: (none) -> Daniel Molina
- title: (none) -> 74HCT6526 Board 2
Changed lines of the file:
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@@
 (kicad_sch (version 20211123) (generator eeschema)
   (paper "A4")
+  (title_block
+    (title "74HCT6526 Board 2")
+    (date "2022-08-17")
+    (rev "0.1")
+    (company "Daniel Molina")
+    (comment 1 "https://github.com/dmolinagarcia/74HCT6526")
+  )
   (junction (at 111.76 81.28) (diameter 1.016) (color 0 0 0 0)
   )

Commit message: .
Parts:
- added C230: 100n, Capacitor_SMD:C_0603_1608Metric, symbol Device:C
Connections:
- net GND: now also C230.2
- net ~{RES}: now also C230.1
Changed lines of the file:
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@@
   (title_block
     (title "74HCT6526 Board 2")
-    (date "2022-08-17")
-    (rev "0.1")
+    (date "2022-10-08")
+    (rev "0.1.2")
     (company "Daniel Molina")
     (comment 1 "https://github.com/dmolinagarcia/74HCT6526")
@@
   (junction (at 111.76 81.28) (diameter 1.016) (color 0 0 0 0)
   )
+  (junction (at 248.285 91.44) (diameter 0) (color 0 0 0 0)
+  )
   (junction (at 111.76 88.9) (diameter 1.016) (color 0 0 0 0)
   )
@@
     (stroke (width 0.1524) (type solid) (color 0 0 0 0))
   )
-  (wire (pts (xy 238.76 91.44) (xy 256.54 91.44))
+  (wire (pts (xy 238.76 91.44) (xy 248.285 91.44))
     (stroke (width 0) (type solid) (color 0 0 0 0))
   )
@@
   )
   (wire (pts (xy 165.1 76.2) (xy 177.8 76.2))
+    (stroke (width 0) (type solid) (color 0 0 0 0))
+  )
+  (wire (pts (xy 248.285 91.44) (xy 256.54 91.44))
     (stroke (width 0) (type solid) (color 0 0 0 0))
   )
@@
     (pin "9")
   )
+  (symbol (lib_id "Device:C") (at 248.285 95.25 0) (unit 1)
+    (in_bom yes) (on_board yes) (fields_autoplaced)
+    (property "Reference" "C230" (id 0) (at 251.46 93.9799 0)
+      (effects (font (size 1.27 1.27)) (justify left))
+    )
+    (property "Value" "100n" (id 1) (at 251.46 96.5199 0)
+      (effects (font (size 1.27 1.27)) (justify left))
+    )
+    (property "Footprint" "Capacitor_SMD:C_0603_1608Metric" (id 2) (at 249.2502 99.06 0)
+      (effects (font (size 1.27 1.27)) hide)
+    )
+    (property "Datasheet" "~" (id 3) (at 248.285 95.25 0)
+      (effects (font (size 1.27 1.27)) hide)
+    )
+    (pin "1")
+    (pin "2")
+  )
   (symbol (lib_id "Connector_Generic:Conn_02x10_Odd_Even") (at 157.48 78.74 0) (unit 1)
     (in_bom yes) (on_board yes)
@@
       (effects (font (size 1.27 1.27)) hide)
     )
+    (pin "1")
+  )
+  (symbol (lib_id "power:GND") (at 248.285 99.06 0) (unit 1)
+    (in_bom yes) (on_board yes) (fields_autoplaced)
+    (property "Reference" "#PWR0107" (id 0) (at 248.285 105.41 0)
+      (effects (font (size 1.27 1.27)) hide)
+    )
+    (property "Value" "GND" (id 1) (at 248.285 104.14 0))
+    (property "Footprint" "" (id 2) (at 248.285 99.06 0)
+      (effects (font (size 1.27 1.27)) hide)
+    )
+    (property "Datasheet" "" (id 3) (at 248.285 99.06 0)
+      (effects (font (size 1.27 1.27)) hide)
+    )

Commit message: B0 ready for v0.2.0 release.
Parts:
- renumbered C230 to C200
Connections:
- net TARUNMODE: no longer names the net of CONTROLBUS2.18 (Pin_18)
- no-connect marks 0 -> 1
Changed lines of the file:
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@@
   (title_block
     (title "74HCT6526 Board 2")
-    (date "2022-10-08")
-    (rev "0.1.2")
+    (date "2023-01-22")
+    (rev "0.2.0")
     (company "Daniel Molina")
     (comment 1 "https://github.com/dmolinagarcia/74HCT6526")
@@
   (junction (at 111.76 78.74) (diameter 1.016) (color 0 0 0 0)
   )
+  (no_connect (at 238.76 88.9))
   (bus_entry (at 78.74 78.74) (size 2.54 2.54)
     (stroke (width 0.1524) (type solid) (color 0 0 0 0))
@@
   )
   (bus_entry (at 259.08 83.82) (size -2.54 2.54)
-    (stroke (width 0.1524) (type solid) (color 0 0 0 0))
-  )
-  (bus_entry (at 259.08 86.36) (size -2.54 2.54)
     (stroke (width 0.1524) (type solid) (color 0 0 0 0))
   )
@@
     (stroke (width 0) (type solid) (color 0 0 0 0))
   )
-  (wire (pts (xy 238.76 88.9) (xy 256.54 88.9))
-    (stroke (width 0) (type solid) (color 0 0 0 0))
-  )
   (bus (pts (xy 78.74 83.82) (xy 78.74 86.36))
     (stroke (width 0) (type solid) (color 0 0 0 0))
@@
     (stroke (width 0) (type solid) (color 0 0 0 0))
   )
-  (bus (pts (xy 259.08 83.82) (xy 259.08 86.36))
+  (bus (pts (xy 259.08 83.82) (xy 259.08 88.9))
     (stroke (width 0) (type solid) (color 0 0 0 0))
   )
@@
     (stroke (width 0) (type solid) (color 0 0 0 0))
   )
-  (bus (pts (xy 259.08 86.36) (xy 259.08 88.9))
-    (stroke (width 0) (type solid) (color 0 0 0 0))
-  )
   (bus (pts (xy 78.74 66.04) (xy 78.74 68.58))
     (stroke (width 0) (type solid) (color 0 0 0 0))
@@
   )
   (label "SP" (at 223.52 73.66 180)
-    (effects (font (size 1.27 1.27)) (justify right bottom))
-  )
-  (label "TARUNMODE" (at 251.46 88.9 180)
     (effects (font (size 1.27 1.27)) (justify right bottom))
   )
@@
   (symbol (lib_id "Device:C") (at 248.285 95.25 0) (unit 1)
     (in_bom yes) (on_board yes) (fields_autoplaced)
-    (property "Reference" "C230" (id 0) (at 251.46 93.9799 0)
+    (property "Reference" "C200" (id 0) (at 251.46 93.9799 0)
       (effects (font (size 1.27 1.27)) (justify left))
     )
