File: B2/power.kicad_sch (KiCad schematic)
At the start: 43 parts, among them U103 74HCT32, U104 74HCT32, U108 74HC32, U109 74HC74, U110 74HC04, U113 74HC27, U115 74HC74, U118 74HC74, U119 74HC74, U120 74HC74, U123 74HCT74, U124 74HC00, U125 74HC74, U126 74HC00, U127 74HC08

Commit message: B2 almost ready
Parts:
- removed C103: 100n, Capacitor_SMD:C_0603_1608Metric, symbol Device:C
- removed unit 3 of U110
- removed U120: 74HC74, Package_SO:SO-14_3.9x8.65mm_P1.27mm, symbol 74xx:74HC74
- added C307, C999: 100n, Capacitor_SMD:C_0603_1608Metric, symbol Device:C
- added unit 3 of U302
- added unit 3 of U303
- added U999: 74HC74, Package_SO:SO-14_3.9x8.65mm_P1.27mm, symbol 74xx:74HC74
- renumbered C115 to C302, C104 to C303, C113 to C304, C121 to C305, C119 to C306, C110 to C308, C120 to C309, C102 to C310, C114 to C311, C107 to C312, C127 to C313, C118 to C314, C122 to C315, C112 to C316, C101 to C317, C106 to C318, C128 to C319, C109 to C320, C117 to C321, C111 to C322, C105 to C323, C125 to C324, C126 to C325, C123 to C326, C108 to C327, C116 to C328, C124 to C329, U103 to U203, U104 to U204, U110 to U302, U124 to U303, U108 to U304, U127 to U306, U125 to U308, U126 to U310, U123 to U311, U118 to U312, U113 to U315, U115 to U316, U109 to U317, U119 to U318
Connections:
- net GND: now also C307.2, C999.2, U999.7 (GND)
- net VCC: now also C307.1, C999.1, U302.5, U303.10, U303.9, U999.14 (VCC)
- no-connect marks 2 -> 3

Commit message: Almost 0.1.1
Parts:
- renumbered U304 to U208, U317 to U209, U302 to U210, U315 to U211, U316 to U213, U312 to U216, U318 to U217, U311 to U221, U999 to U222, U308 to U223, U310 to U226, U303 to U227, U306 to U229
Other:
- company: (none) -> Daniel Molina
- title: (none) -> 74HCT6526 Board 2
Changed lines of the file:
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@@
 (kicad_sch (version 20211123) (generator eeschema)
   (paper "A4")
+  (title_block
+    (title "74HCT6526 Board 2")
+    (date "2022-08-17")
+    (rev "0.1")
+    (company "Daniel Molina")
+    (comment 1 "https://github.com/dmolinagarcia/74HCT6526")
+  )
   (junction (at 137.16 63.5) (diameter 0) (color 0 0 0 0)
   )
@@
   (symbol (lib_id "74xx:74HC04") (at 74.93 50.8 0) (unit 7)
     (in_bom yes) (on_board yes) (fields_autoplaced)
-    (property "Reference" "U302" (id 0) (at 80.772 49.8915 0)
+    (property "Reference" "U210" (id 0) (at 80.772 49.8915 0)
       (effects (font (size 1.27 1.27)) (justify left))
     )
@@
   (symbol (lib_id "74xx:74HC00") (at 200.66 50.8 0) (unit 5)
     (in_bom yes) (on_board yes) (fields_autoplaced)
-    (property "Reference" "U310" (id 0) (at 206.502 49.8915 0)
+    (property "Reference" "U226" (id 0) (at 206.502 49.8915 0)
       (effects (font (size 1.27 1.27)) (justify left))
     )
@@
   (symbol (lib_id "74xx:74HC74") (at 158.75 50.8 0) (unit 3)
     (in_bom yes) (on_board yes)
-    (property "Reference" "U999" (id 0) (at 157.48 50.8 0)
+    (property "Reference" "U222" (id 0) (at 157.48 50.8 0)
       (effects (font (size 1.27 1.27)) (justify left))
     )
@@
   (symbol (lib_id "74xx:74HC74") (at 222.25 50.8 0) (unit 3)
     (in_bom yes) (on_board yes) (fields_autoplaced)
-    (property "Reference" "U311" (id 0) (at 228.092 49.8915 0)
+    (property "Reference" "U221" (id 0) (at 228.092 49.8915 0)
       (effects (font (size 1.27 1.27)) (justify left))
     )
@@
   (symbol (lib_id "74xx:74HC74") (at 137.16 82.55 0) (unit 3)
     (in_bom yes) (on_board yes) (fields_autoplaced)
-    (property "Reference" "U317" (id 0) (at 143.002 81.6415 0)
+    (property "Reference" "U209" (id 0) (at 143.002 81.6415 0)
       (effects (font (size 1.27 1.27)) (justify left))
     )
@@
   (symbol (lib_id "74xx:74HC00") (at 72.39 162.56 0) (unit 3)
     (in_bom yes) (on_board yes)
-    (property "Reference" "U303" (id 0) (at 72.39 162.56 0))
+    (property "Reference" "U227" (id 0) (at 72.39 162.56 0))
     (property "Value" "74HC00" (id 1) (at 72.39 157.5586 0))
     (property "Footprint" "Package_SO:SOIC-14_3.9x8.7mm_P1.27mm" (id 2) (at 72.39 162.56 0)
@@
   (symbol (lib_id "74xx:74HC74") (at 157.48 82.55 0) (unit 3)
     (in_bom yes) (on_board yes) (fields_autoplaced)
-    (property "Reference" "U318" (id 0) (at 163.322 81.6415 0)
+    (property "Reference" "U217" (id 0) (at 163.322 81.6415 0)
       (effects (font (size 1.27 1.27)) (justify left))
     )
@@
   (symbol (lib_id "74xx:74HC04") (at 72.39 173.99 0) (unit 3)
     (in_bom yes) (on_board yes)
-    (property "Reference" "U302" (id 0) (at 72.39 173.99 0))
+    (property "Reference" "U210" (id 0) (at 72.39 173.99 0))
     (property "Value" "74HC04" (id 1) (at 72.39 168.9886 0))
     (property "Footprint" "Package_SO:SOIC-14_3.9x8.7mm_P1.27mm" (id 2) (at 72.39 173.99 0)
@@
   (symbol (lib_id "74xx:74HC74") (at 116.84 82.55 0) (unit 3)
     (in_bom yes) (on_board yes) (fields_autoplaced)
-    (property "Reference" "U316" (id 0) (at 122.682 81.6415 0)
+    (property "Reference" "U213" (id 0) (at 122.682 81.6415 0)
       (effects (font (size 1.27 1.27)) (justify left))
     )
@@
   (symbol (lib_id "Custom 74xx:74HC08") (at 137.16 50.8 0) (unit 5)
     (in_bom yes) (on_board yes) (fields_autoplaced)
-    (property "Reference" "U306" (id 0) (at 143.002 49.8915 0)
+    (property "Reference" "U229" (id 0) (at 143.002 49.8915 0)
       (effects (font (size 1.27 1.27)) (justify left))
     )
@@
   (symbol (lib_id "74xx:74LS27") (at 95.25 82.55 0) (unit 4)
     (in_bom yes) (on_board yes) (fields_autoplaced)
-    (property "Reference" "U315" (id 0) (at 101.092 81.6415 0)
+    (property "Reference" "U211" (id 0) (at 101.092 81.6415 0)
       (effects (font (size 1.27 1.27)) (justify left))
     )
@@
   (symbol (lib_id "74xx:74HC04") (at 72.39 151.13 0) (unit 2)
     (in_bom yes) (on_board yes)
-    (property "Reference" "U302" (id 0) (at 72.39 151.13 0))
+    (property "Reference" "U210" (id 0) (at 72.39 151.13 0))
     (property "Value" "74HC04" (id 1) (at 72.39 146.1286 0))
     (property "Footprint" "Package_SO:SOIC-14_3.9x8.7mm_P1.27mm" (id 2) (at 72.39 151.13 0)
@@
   (symbol (lib_id "74xx:74LS32") (at 116.84 50.8 0) (unit 5)
     (in_bom yes) (on_board yes) (fields_autoplaced)
-    (property "Reference" "U304" (id 0) (at 122.682 49.8915 0)
+    (property "Reference" "U208" (id 0) (at 122.682 49.8915 0)
       (effects (font (size 1.27 1.27)) (justify left))
     )
@@
   (symbol (lib_id "74xx:74HC74") (at 74.93 82.55 0) (unit 3)
     (in_bom yes) (on_board yes) (fields_autoplaced)
-    (property "Reference" "U312" (id 0) (at 80.772 81.6415 0)
+    (property "Reference" "U216" (id 0) (at 80.772 81.6415 0)
       (effects (font (size 1.27 1.27)) (justify left))
     )
@@
   (symbol (lib_id "74xx:74HC00") (at 95.25 50.8 0) (unit 5)
     (in_bom yes) (on_board yes) (fields_autoplaced)
-    (property "Reference" "U303" (id 0) (at 101.092 49.8915 0)
+    (property "Reference" "U227" (id 0) (at 101.092 49.8915 0)
       (effects (font (size 1.27 1.27)) (justify left))
     )
@@
   (symbol (lib_id "74xx:74HC74") (at 179.07 50.8 0) (unit 3)
     (in_bom yes) (on_board yes) (fields_autoplaced)
-    (property "Reference" "U308" (id 0) (at 184.912 49.8915 0)
-      (effects (font (size 1.27 1.27)) (justify left))
-    )
+    (property "Reference" "U223" (id 0) (at 184.912 49.8915 0)
+      (effects (font (size 1.27 1.27)) (justify left))
+    )

Commit message: Added ICR. B2 fixes
Parts:
- U229: value 74HC08 -> 74HCT08
Changed lines of the file:
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@@
       (effects (font (size 1.27 1.27)) (justify left))
     )
-    (property "Value" "74HC08" (id 1) (at 143.002 52.6666 0)
+    (property "Value" "74HCT08" (id 1) (at 143.002 52.6666 0)
       (effects (font (size 1.27 1.27)) (justify left))
     )

Commit message: Ready for v0.2.1
Parts:
- added C202: 100n, Capacitor_SMD:C_0603_1608Metric, symbol Device:C
- added unit 2 of U217
- added U230: 74HC74, Package_SO:SO-14_3.9x8.65mm_P1.27mm, symbol 74xx:74HC74
Connections:
- net GND: now also C202.2, U230.7 (GND)
- net VCC: now also C202.1, U217.10 (~{S}), U217.11 (C), U217.12 (D), U217.13 (~{R}), U230.14 (VCC)
- no-connect marks 3 -> 5
Changed lines of the file:
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@@
   (title_block
     (title "74HCT6526 Board 2")
-    (date "2023-01-22")
-    (rev "0.2.0")
+    (date "2023-03-25")
+    (rev "0.2.1")
     (company "Daniel Molina")
     (comment 1 "https://github.com/dmolinagarcia/74HCT6526")
@@
   (junction (at 166.37 125.73) (diameter 0) (color 0 0 0 0)
   )
+  (junction (at 88.9 148.59) (diameter 0) (color 0 0 0 0)
+  )
   (junction (at 86.36 118.11) (diameter 0) (color 0 0 0 0)
   )
@@
   (junction (at 95.25 38.1) (diameter 0) (color 0 0 0 0)
   )
+  (junction (at 88.9 146.05) (diameter 0) (color 0 0 0 0)
+  )
   (junction (at 97.79 133.35) (diameter 0) (color 0 0 0 0)
   )
@@
   (junction (at 95.25 63.5) (diameter 0) (color 0 0 0 0)
   )
+  (junction (at 242.57 63.5) (diameter 0) (color 0 0 0 0)
+  )
   (junction (at 200.66 125.73) (diameter 0) (color 0 0 0 0)
   )
@@
   (junction (at 179.07 95.25) (diameter 0) (color 0 0 0 0)
   )
+  (junction (at 234.95 133.35) (diameter 0) (color 0 0 0 0)
+  )
   (junction (at 212.09 125.73) (diameter 0) (color 0 0 0 0)
   )
   (junction (at 86.36 133.35) (diameter 0) (color 0 0 0 0)
   )
+  (junction (at 222.25 38.1) (diameter 0) (color 0 0 0 0)
+  )
+  (junction (at 88.9 138.43) (diameter 0) (color 0 0 0 0)
+  )
   (junction (at 60.96 160.02) (diameter 0) (color 0 0 0 0)
   )
@@
   (junction (at 60.96 125.73) (diameter 0) (color 0 0 0 0)
   )
+  (junction (at 60.96 138.43) (diameter 0) (color 0 0 0 0)
+  )
   (junction (at 74.93 125.73) (diameter 0) (color 0 0 0 0)
   )
@@
   )
   (junction (at 143.51 118.11) (diameter 0) (color 0 0 0 0)
+  )
+  (junction (at 223.52 125.73) (diameter 0) (color 0 0 0 0)
   )
   (junction (at 97.79 110.49) (diameter 0) (color 0 0 0 0)
@@
   (no_connect (at 80.01 162.56))
   (no_connect (at 80.01 151.13))
+  (no_connect (at 107.95 146.05))
+  (no_connect (at 107.95 151.13))
   (wire (pts (xy 137.16 95.25) (xy 157.48 95.25))
     (stroke (width 0) (type default) (color 0 0 0 0))
@@
     (stroke (width 0) (type default) (color 0 0 0 0))
   )
-  (wire (pts (xy 60.96 125.73) (xy 60.96 151.13))
+  (wire (pts (xy 60.96 125.73) (xy 60.96 138.43))
     (stroke (width 0) (type default) (color 0 0 0 0))
   )
@@
     (stroke (width 0) (type default) (color 0 0 0 0))
   )
+  (wire (pts (xy 88.9 146.05) (xy 88.9 138.43))
+    (stroke (width 0) (type default) (color 0 0 0 0))
+  )
   (wire (pts (xy 200.66 63.5) (xy 179.07 63.5))
     (stroke (width 0) (type default) (color 0 0 0 0))
   )
+  (wire (pts (xy 100.33 138.43) (xy 88.9 138.43))
+    (stroke (width 0) (type default) (color 0 0 0 0))
+  )
   (wire (pts (xy 137.16 69.85) (xy 157.48 69.85))
     (stroke (width 0) (type default) (color 0 0 0 0))
@@
     (stroke (width 0) (type default) (color 0 0 0 0))
   )
+  (wire (pts (xy 100.33 158.75) (xy 88.9 158.75))
+    (stroke (width 0) (type default) (color 0 0 0 0))
+  )
   (wire (pts (xy 177.8 133.35) (xy 189.23 133.35))
     (stroke (width 0) (type default) (color 0 0 0 0))
@@
     (stroke (width 0) (type default) (color 0 0 0 0))
   )
+  (wire (pts (xy 100.33 156.21) (xy 100.33 158.75))
+    (stroke (width 0) (type default) (color 0 0 0 0))
+  )
   (wire (pts (xy 60.96 151.13) (xy 60.96 160.02))
     (stroke (width 0) (type default) (color 0 0 0 0))
@@
     (stroke (width 0) (type default) (color 0 0 0 0))
   )
+  (wire (pts (xy 234.95 133.35) (xy 242.57 133.35))
+    (stroke (width 0) (type default) (color 0 0 0 0))
+  )
   (wire (pts (xy 74.93 125.73) (xy 86.36 125.73))
     (stroke (width 0) (type default) (color 0 0 0 0))
@@
     (stroke (width 0) (type default) (color 0 0 0 0))
   )
+  (wire (pts (xy 222.25 38.1) (xy 242.57 38.1))
+    (stroke (width 0) (type default) (color 0 0 0 0))
+  )
   (wire (pts (xy 200.66 38.1) (xy 222.25 38.1))
     (stroke (width 0) (type default) (color 0 0 0 0))
@@
     (stroke (width 0) (type default) (color 0 0 0 0))
   )
+  (wire (pts (xy 60.96 138.43) (xy 60.96 151.13))
+    (stroke (width 0) (type default) (color 0 0 0 0))
+  )
   (wire (pts (xy 158.75 38.1) (xy 179.07 38.1))
     (stroke (width 0) (type default) (color 0 0 0 0))
@@
     (stroke (width 0) (type default) (color 0 0 0 0))
   )
+  (wire (pts (xy 88.9 148.59) (xy 92.71 148.59))
+    (stroke (width 0) (type default) (color 0 0 0 0))
+  )
   (wire (pts (xy 212.09 125.73) (xy 223.52 125.73))
     (stroke (width 0) (type default) (color 0 0 0 0))
@@
     (stroke (width 0) (type default) (color 0 0 0 0))
   )
+  (wire (pts (xy 242.57 38.1) (xy 242.57 40.64))
+    (stroke (width 0) (type default) (color 0 0 0 0))
+  )
   (wire (pts (xy 222.25 60.96) (xy 222.25 63.5))
     (stroke (width 0) (type default) (color 0 0 0 0))
@@
     (stroke (width 0) (type default) (color 0 0 0 0))
   )
-  (wire (pts (xy 223.52 133.35) (xy 242.57 133.35))
+  (wire (pts (xy 223.52 133.35) (xy 234.95 133.35))
     (stroke (width 0) (type default) (color 0 0 0 0))
   )
@@
     (stroke (width 0) (type default) (color 0 0 0 0))
   )
+  (wire (pts (xy 88.9 138.43) (xy 60.96 138.43))
+    (stroke (width 0) (type default) (color 0 0 0 0))
+  )
   (wire (pts (xy 132.08 133.35) (xy 143.51 133.35))
     (stroke (width 0) (type default) (color 0 0 0 0))
@@
     (stroke (width 0) (type default) (color 0 0 0 0))
   )
+  (wire (pts (xy 242.57 60.96) (xy 242.57 63.5))
+    (stroke (width 0) (type default) (color 0 0 0 0))
+  )
   (wire (pts (xy 60.96 160.02) (xy 60.96 165.1))
     (stroke (width 0) (type default) (color 0 0 0 0))
@@
     (stroke (width 0) (type default) (color 0 0 0 0))
   )
+  (wire (pts (xy 88.9 148.59) (xy 88.9 146.05))
+    (stroke (width 0) (type default) (color 0 0 0 0))
+  )
   (wire (pts (xy 86.36 118.11) (xy 97.79 118.11))
     (stroke (width 0) (type default) (color 0 0 0 0))
@@
     (stroke (width 0) (type default) (color 0 0 0 0))
   )
+  (wire (pts (xy 223.52 125.73) (xy 234.95 125.73))
+    (stroke (width 0) (type default) (color 0 0 0 0))
+  )
   (wire (pts (xy 154.94 118.11) (xy 166.37 118.11))
     (stroke (width 0) (type default) (color 0 0 0 0))
@@
     (stroke (width 0) (type default) (color 0 0 0 0))
   )
+  (wire (pts (xy 100.33 140.97) (xy 100.33 138.43))
+    (stroke (width 0) (type default) (color 0 0 0 0))
+  )
   (wire (pts (xy 60.96 165.1) (xy 60.96 173.99))
     (stroke (width 0) (type default) (color 0 0 0 0))
@@
     (stroke (width 0) (type default) (color 0 0 0 0))
   )
+  (wire (pts (xy 88.9 146.05) (xy 92.71 146.05))
+    (stroke (width 0) (type default) (color 0 0 0 0))
+  )
   (wire (pts (xy 177.8 110.49) (xy 189.23 110.49))
     (stroke (width 0) (type default) (color 0 0 0 0))
@@
   )
   (wire (pts (xy 158.75 63.5) (xy 179.07 63.5))
+    (stroke (width 0) (type default) (color 0 0 0 0))
+  )
+  (wire (pts (xy 88.9 158.75) (xy 88.9 148.59))
     (stroke (width 0) (type default) (color 0 0 0 0))
   )
@@
     (pin "7")
   )
+  (symbol (lib_id "Device:C") (at 234.95 129.54 0) (unit 1)
+    (in_bom yes) (on_board yes) (fields_autoplaced)
+    (property "Reference" "C202" (id 0) (at 237.871 128.6315 0)
+      (effects (font (size 1.27 1.27)) (justify left))
+    )
+    (property "Value" "100n" (id 1) (at 237.871 131.4066 0)
+      (effects (font (size 1.27 1.27)) (justify left))
+    )
+    (property "Footprint" "Capacitor_SMD:C_0603_1608Metric" (id 2) (at 235.9152 133.35 0)
+      (effects (font (size 1.27 1.27)) hide)
+    )
+    (property "Datasheet" "~" (id 3) (at 234.95 129.54 0)
+      (effects (font (size 1.27 1.27)) hide)
+    )
+    (pin "1")
+    (pin "2")
+  )
   (symbol (lib_id "74xx:74LS32") (at 116.84 50.8 0) (unit 5)
     (in_bom yes) (on_board yes) (fields_autoplaced)
@@
     (pin "2")
   )
+  (symbol (lib_id "74xx:74HC74") (at 100.33 148.59 0) (unit 2)
+    (in_bom yes) (on_board yes)
+    (property "Reference" "U217" (id 0) (at 98.425 148.59 0)
+      (effects (font (size 1.27 1.27)) (justify left))
+    )
+    (property "Value" "74HC74" (id 1) (at 102.235 154.94 0)
+      (effects (font (size 1.27 1.27)) (justify left))
+    )
+    (property "Footprint" "Package_SO:SO-14_3.9x8.65mm_P1.27mm" (id 2) (at 100.33 148.59 0)
+      (effects (font (size 1.27 1.27)) hide)
+    )
+    (property "Datasheet" "74xx/74hc_hct74.pdf" (id 3) (at 100.33 148.59 0)
+      (effects (font (size 1.27 1.27)) hide)
+    )
+    (pin "1")
+    (pin "2")
+    (pin "3")
+    (pin "4")
+    (pin "5")
+    (pin "6")
+    (pin "10")
+    (pin "11")
+    (pin "12")
+    (pin "13")
+    (pin "8")
+    (pin "9")
+    (pin "14")
+    (pin "7")
+  )
   (symbol (lib_id "Device:C") (at 74.93 129.54 0) (unit 1)
     (in_bom yes) (on_board yes) (fields_autoplaced)
@@
     (pin "2")
   )
+  (symbol (lib_id "74xx:74HC74") (at 242.57 50.8 0) (unit 3)
+    (in_bom yes) (on_board yes) (fields_autoplaced)
+    (property "Reference" "U230" (id 0) (at 250.19 49.5299 0)
+      (effects (font (size 1.27 1.27)) (justify left))
+    )
+    (property "Value" "74HC74" (id 1) (at 250.19 52.0699 0)
+      (effects (font (size 1.27 1.27)) (justify left))
+    )
+    (property "Footprint" "Package_SO:SO-14_3.9x8.65mm_P1.27mm" (id 2) (at 242.57 50.8 0)
+      (effects (font (size 1.27 1.27)) hide)
+    )
+    (property "Datasheet" "74xx/74hc_hct74.pdf" (id 3) (at 242.57 50.8 0)
+      (effects (font (size 1.27 1.27)) hide)
+    )
+    (pin "1")
+    (pin "2")
+    (pin "3")
+    (pin "4")
+    (pin "5")
+    (pin "6")
+    (pin "10")
+    (pin "11")
+    (pin "12")
+    (pin "13")
+    (pin "8")
+    (pin "9")
+    (pin "14")
+    (pin "7")
+  )
   (symbol (lib_id "power:GND") (at 242.57 139.7 0) (unit 1)
