File: B2/resetData.kicad_sch (KiCad schematic)
At the start: 3 parts, among them U203 74HCT32, U204 74HCT32, U302 74HC04

Commit message: Almost 0.1.1
Parts:
- renumbered U302 to U210
Other:
- company: (none) -> Daniel Molina
- title: (none) -> 74HCT6526 Board 2
Changed lines of the file:
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@@
 (kicad_sch (version 20211123) (generator eeschema)
   (paper "A4")
+  (title_block
+    (title "74HCT6526 Board 2")
+    (date "2022-08-17")
+    (rev "0.1")
+    (company "Daniel Molina")
+    (comment 1 "https://github.com/dmolinagarcia/74HCT6526")
+  )
   (junction (at 133.35 99.06) (diameter 0) (color 0 0 0 0)
   )
@@
   (symbol (lib_id "74xx:74HC04") (at 111.76 52.07 0) (unit 4)
     (in_bom yes) (on_board yes)
-    (property "Reference" "U302" (id 0) (at 110.49 52.07 0))
+    (property "Reference" "U210" (id 0) (at 110.49 52.07 0))
     (property "Value" "74HC04" (id 1) (at 111.76 47.0686 0))
     (property "Footprint" "Package_SO:SOIC-14_3.9x8.7mm_P1.27mm" (id 2) (at 111.76 52.07 0)
