File: B2/timer16.kicad_sch (KiCad schematic)
At the start: 8 parts, among them U201 74HC244, U202 74HC244, U322 74HC193, U323 74HC193, U324 74HC193, U325 74HC193, U328 74HC688, U329 74HC688

Commit message: Almost 0.1.1
Parts:
- renumbered U329 to U206, U328 to U207, U325 to U214, U323 to U215, U324 to U219, U322 to U220
Other:
- company: (none) -> Daniel Molina
- title: (none) -> 74HCT6526 Board 2
Changed lines of the file:
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@@
 (kicad_sch (version 20211123) (generator eeschema)
   (paper "A4")
+  (title_block
+    (title "74HCT6526 Board 2")
+    (date "2022-08-17")
+    (rev "0.1")
+    (company "Daniel Molina")
+    (comment 1 "https://github.com/dmolinagarcia/74HCT6526")
+  )
   (junction (at 237.49 133.35) (diameter 0) (color 0 0 0 0)
   )
@@
   (symbol (lib_id "74xx:74LS193") (at 97.79 173.99 0) (unit 1)
     (in_bom yes) (on_board yes) (fields_autoplaced)
-    (property "Reference" "U325" (id 0) (at 99.8094 157.3235 0)
+    (property "Reference" "U214" (id 0) (at 99.8094 157.3235 0)
       (effects (font (size 1.27 1.27)) (justify left))
     )
@@
   (symbol (lib_id "74xx:74HC688") (at 250.19 120.65 0) (unit 1)
     (in_bom yes) (on_board yes)
-    (property "Reference" "U329" (id 0) (at 252.73 116.6049 0))
+    (property "Reference" "U206" (id 0) (at 252.73 116.6049 0))
     (property "Value" "74HC688" (id 1) (at 252.73 119.38 0))
     (property "Footprint" "Package_SO:SOIC-20W_7.5x12.8mm_P1.27mm" (id 2) (at 250.19 120.65 0)
@@
   (symbol (lib_id "74xx:74LS193") (at 97.79 128.27 0) (unit 1)
     (in_bom yes) (on_board yes) (fields_autoplaced)
-    (property "Reference" "U324" (id 0) (at 99.8094 111.6035 0)
+    (property "Reference" "U219" (id 0) (at 99.8094 111.6035 0)
       (effects (font (size 1.27 1.27)) (justify left))
     )
@@
   (symbol (lib_id "74xx:74LS193") (at 97.79 82.55 0) (unit 1)
     (in_bom yes) (on_board yes) (fields_autoplaced)
-    (property "Reference" "U323" (id 0) (at 99.8094 65.8835 0)
+    (property "Reference" "U215" (id 0) (at 99.8094 65.8835 0)
       (effects (font (size 1.27 1.27)) (justify left))
     )
@@
   (symbol (lib_id "74xx:74HC688") (at 250.19 50.8 0) (unit 1)
     (in_bom yes) (on_board yes)
-    (property "Reference" "U328" (id 0) (at 252.73 46.7549 0))
+    (property "Reference" "U207" (id 0) (at 252.73 46.7549 0))
     (property "Value" "74HC688" (id 1) (at 252.73 49.53 0))
     (property "Footprint" "Package_SO:SOIC-20W_7.5x12.8mm_P1.27mm" (id 2) (at 250.19 50.8 0)
@@
   (symbol (lib_id "74xx:74LS193") (at 97.79 36.83 0) (unit 1)
     (in_bom yes) (on_board yes) (fields_autoplaced)
-    (property "Reference" "U322" (id 0) (at 99.8094 20.1635 0)
+    (property "Reference" "U220" (id 0) (at 99.8094 20.1635 0)
       (effects (font (size 1.27 1.27)) (justify left))
     )

Commit message: B2 refactored. B4 Added. TOD sch completed.
Parts:
- added U229: 74HCT08, Package_SO:SO-14_3.9x8.65mm_P1.27mm, symbol Custom 74xx:74HC08
Connections:
- net CLK: now also U229.13; no longer U220.4 (DOWN)
- net ~{LOAD}: now also U229.4; no longer U214.11 (~{LOAD}), U215.11 (~{LOAD}), U219.11 (~{LOAD}), U220.11 (~{LOAD})
- new net: U214.11 (~{LOAD}), U215.11 (~{LOAD}), U219.11 (~{LOAD}), U220.11 (~{LOAD}), U229.6
- new net: U220.4 (DOWN), U229.11
- new net PHI2: U229.12
- new net ~{RES}: U229.5
Changed lines of the file:
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@@
   (junction (at 237.49 133.35) (diameter 0) (color 0 0 0 0)
   )
+  (junction (at 48.26 85.09) (diameter 0) (color 0 0 0 0)
+  )
+  (junction (at 48.26 39.37) (diameter 0) (color 0 0 0 0)
+  )
   (junction (at 237.49 125.73) (diameter 0) (color 0 0 0 0)
   )
@@
   (junction (at 237.49 123.19) (diameter 0) (color 0 0 0 0)
   )
-  (junction (at 44.45 39.37) (diameter 0) (color 0 0 0 0)
-  )
-  (junction (at 44.45 130.81) (diameter 0) (color 0 0 0 0)
-  )
   (junction (at 237.49 55.88) (diameter 0) (color 0 0 0 0)
   )
@@
   (junction (at 237.49 138.43) (diameter 0) (color 0 0 0 0)
   )
-  (junction (at 44.45 85.09) (diameter 0) (color 0 0 0 0)
-  )
   (junction (at 237.49 66.04) (diameter 0) (color 0 0 0 0)
   )
   (junction (at 237.49 130.81) (diameter 0) (color 0 0 0 0)
+  )
+  (junction (at 48.26 130.81) (diameter 0) (color 0 0 0 0)
   )
   (junction (at 168.91 83.82) (diameter 0) (color 0 0 0 0)
@@
     (stroke (width 0) (type default) (color 0 0 0 0))
   )
+  (wire (pts (xy 24.13 41.91) (xy 27.94 41.91))
+    (stroke (width 0) (type default) (color 0 0 0 0))
+  )
   (wire (pts (xy 162.56 73.66) (xy 168.91 73.66))
     (stroke (width 0) (type default) (color 0 0 0 0))
@@
     (stroke (width 0) (type default) (color 0 0 0 0))
   )
+  (wire (pts (xy 48.26 85.09) (xy 85.09 85.09))
+    (stroke (width 0) (type default) (color 0 0 0 0))
+  )
+  (wire (pts (xy 43.18 49.53) (xy 73.66 49.53))
+    (stroke (width 0) (type default) (color 0 0 0 0))
+  )
   (wire (pts (xy 194.31 76.2) (xy 203.2 76.2))
     (stroke (width 0) (type default) (color 0 0 0 0))
@@
     (stroke (width 0) (type default) (color 0 0 0 0))
   )
-  (wire (pts (xy 44.45 85.09) (xy 44.45 130.81))
+  (wire (pts (xy 48.26 85.09) (xy 48.26 130.81))
     (stroke (width 0) (type default) (color 0 0 0 0))
   )
@@
     (stroke (width 0) (type default) (color 0 0 0 0))
   )
+  (wire (pts (xy 48.26 130.81) (xy 85.09 130.81))
+    (stroke (width 0) (type default) (color 0 0 0 0))
+  )
   (wire (pts (xy 236.22 86.36) (xy 236.22 73.66))
     (stroke (width 0) (type default) (color 0 0 0 0))
@@
     (stroke (width 0) (type default) (color 0 0 0 0))
   )
+  (wire (pts (xy 73.66 49.53) (xy 73.66 46.99))
+    (stroke (width 0) (type default) (color 0 0 0 0))
+  )
   (wire (pts (xy 231.14 105.41) (xy 237.49 105.41))
     (stroke (width 0) (type default) (color 0 0 0 0))
   )
-  (wire (pts (xy 44.45 130.81) (xy 85.09 130.81))
-    (stroke (width 0) (type default) (color 0 0 0 0))
-  )
   (wire (pts (xy 237.49 60.96) (xy 237.49 63.5))
     (stroke (width 0) (type default) (color 0 0 0 0))
@@
     (stroke (width 0) (type default) (color 0 0 0 0))
   )
+  (wire (pts (xy 43.18 39.37) (xy 48.26 39.37))
+    (stroke (width 0) (type default) (color 0 0 0 0))
+  )
   (bus (pts (xy 124.46 120.65) (xy 124.46 118.11))
     (stroke (width 0) (type default) (color 0 0 0 0))
@@
     (stroke (width 0) (type default) (color 0 0 0 0))
   )
+  (wire (pts (xy 73.66 46.99) (xy 85.09 46.99))
+    (stroke (width 0) (type default) (color 0 0 0 0))
+  )
   (wire (pts (xy 110.49 168.91) (xy 121.92 168.91))
     (stroke (width 0) (type default) (color 0 0 0 0))
   )
-  (wire (pts (xy 44.45 39.37) (xy 85.09 39.37))
-    (stroke (width 0) (type default) (color 0 0 0 0))
-  )
   (wire (pts (xy 66.04 163.83) (xy 85.09 163.83))
     (stroke (width 0) (type default) (color 0 0 0 0))
@@
     (stroke (width 0) (type default) (color 0 0 0 0))
   )
+  (wire (pts (xy 24.13 46.99) (xy 27.94 46.99))
+    (stroke (width 0) (type default) (color 0 0 0 0))
+  )
   (bus (pts (xy 124.46 163.83) (xy 124.46 161.29))
     (stroke (width 0) (type default) (color 0 0 0 0))
@@
     (stroke (width 0) (type default) (color 0 0 0 0))
   )
-  (wire (pts (xy 39.37 39.37) (xy 44.45 39.37))
-    (stroke (width 0) (type default) (color 0 0 0 0))
-  )
   (bus (pts (xy 160.02 73.66) (xy 160.02 104.14))
     (stroke (width 0) (type default) (color 0 0 0 0))
@@
     (stroke (width 0) (type default) (color 0 0 0 0))
   )
-  (wire (pts (xy 44.45 176.53) (xy 85.09 176.53))
+  (wire (pts (xy 48.26 176.53) (xy 85.09 176.53))
     (stroke (width 0) (type default) (color 0 0 0 0))
   )
@@
     (stroke (width 0) (type default) (color 0 0 0 0))
   )
-  (wire (pts (xy 44.45 130.81) (xy 44.45 176.53))
+  (wire (pts (xy 24.13 52.07) (xy 27.94 52.07))
+    (stroke (width 0) (type default) (color 0 0 0 0))
+  )
+  (wire (pts (xy 48.26 130.81) (xy 48.26 176.53))
     (stroke (width 0) (type default) (color 0 0 0 0))
   )
@@
     (stroke (width 0) (type default) (color 0 0 0 0))
   )
+  (wire (pts (xy 24.13 36.83) (xy 27.94 36.83))
+    (stroke (width 0) (type default) (color 0 0 0 0))
+  )
   (bus (pts (xy 205.74 68.58) (xy 205.74 71.12))
     (stroke (width 0) (type default) (color 0 0 0 0))
@@
     (stroke (width 0) (type default) (color 0 0 0 0))
   )
-  (wire (pts (xy 74.295 46.99) (xy 85.09 46.99))
-    (stroke (width 0) (type default) (color 0 0 0 0))
-  )
   (wire (pts (xy 162.56 68.58) (xy 168.91 68.58))
     (stroke (width 0) (type default) (color 0 0 0 0))
@@
     (stroke (width 0) (type default) (color 0 0 0 0))
   )
-  (wire (pts (xy 44.45 85.09) (xy 85.09 85.09))
-    (stroke (width 0) (type default) (color 0 0 0 0))
-  )
   (bus (pts (xy 228.6 38.1) (xy 228.6 40.64))
     (stroke (width 0) (type default) (color 0 0 0 0))
@@
     (stroke (width 0) (type default) (color 0 0 0 0))
   )
+  (wire (pts (xy 48.26 39.37) (xy 85.09 39.37))
+    (stroke (width 0) (type default) (color 0 0 0 0))
+  )
   (wire (pts (xy 66.04 168.91) (xy 85.09 168.91))
     (stroke (width 0) (type default) (color 0 0 0 0))
@@
     (stroke (width 0) (type default) (color 0 0 0 0))
   )
-  (wire (pts (xy 44.45 39.37) (xy 44.45 85.09))
+  (wire (pts (xy 48.26 39.37) (xy 48.26 85.09))
     (stroke (width 0) (type default) (color 0 0 0 0))
   )
@@
     )
   )
-  (hierarchical_label "CLK" (shape input) (at 74.295 46.99 180)
+  (hierarchical_label "CLK" (shape input) (at 24.13 46.99 180)
     (effects (font (size 1.27 1.27)) (justify right))
   )
-  (hierarchical_label "~{LOAD}" (shape input) (at 39.37 39.37 180)
+  (hierarchical_label "~{LOAD}" (shape input) (at 24.13 36.83 180)
     (effects (font (size 1.27 1.27)) (justify right))
   )
@@
     (effects (font (size 1.27 1.27)) (justify left))
   )
+  (hierarchical_label "PHI2" (shape input) (at 24.13 52.07 180)
+    (effects (font (size 1.27 1.27)) (justify right))
+  )
   (hierarchical_label "~{OEHI}" (shape input) (at 154.94 132.08 180)
     (effects (font (size 1.27 1.27)) (justify right))
@@
   (hierarchical_label "D[0..7]" (shape output) (at 209.55 52.07 0)
     (effects (font (size 1.27 1.27)) (justify left))
+  )
+  (hierarchical_label "~{RES}" (shape input) (at 24.13 41.91 180)
+    (effects (font (size 1.27 1.27)) (justify right))
   )
   (symbol (lib_id "power:VCC") (at 85.09 90.17 90) (unit 1)
@@
     (pin "1")
   )
+  (symbol (lib_id "Custom 74xx:74HC08") (at 35.56 49.53 0) (mirror x) (unit 4)
+    (in_bom yes) (on_board yes)
+    (property "Reference" "U229" (id 0) (at 34.925 50.165 0))
+    (property "Value" "74HCT08" (id 1) (at 35.56 54.5314 0))
+    (property "Footprint" "Package_SO:SO-14_3.9x8.65mm_P1.27mm" (id 2) (at 35.56 49.53 0)
+      (effects (font (size 1.27 1.27)) hide)
+    )
+    (property "Datasheet" "" (id 3) (at 35.56 55.88 0)
+      (effects (font (size 1.27 1.27)) hide)
+    )
+    (pin "1")
+    (pin "2")
+    (pin "3")
+    (pin "4")
+    (pin "5")
+    (pin "6")
+    (pin "10")
+    (pin "8")
+    (pin "9")
+    (pin "11")
+    (pin "12")
+    (pin "13")
+    (pin "14")
+    (pin "7")
+  )
   (symbol (lib_id "74xx:74HC688") (at 250.19 50.8 0) (unit 1)
     (in_bom yes) (on_board yes)
@@
     (pin "9")
   )
+  (symbol (lib_id "Custom 74xx:74HC08") (at 35.56 39.37 0) (unit 2)
+    (in_bom yes) (on_board yes)
+    (property "Reference" "U229" (id 0) (at 35.56 39.37 0))
+    (property "Value" "74HCT08" (id 1) (at 35.56 41.91 0))
+    (property "Footprint" "Package_SO:SO-14_3.9x8.65mm_P1.27mm" (id 2) (at 35.56 39.37 0)
+      (effects (font (size 1.27 1.27)) hide)
+    )
+    (property "Datasheet" "" (id 3) (at 35.56 33.02 0)
+      (effects (font (size 1.27 1.27)) hide)
+    )
+    (pin "1")
+    (pin "2")
+    (pin "3")
+    (pin "4")
+    (pin "5")
+    (pin "6")
+    (pin "10")
+    (pin "8")
+    (pin "9")
+    (pin "11")
+    (pin "12")
+    (pin "13")
+    (pin "14")
+    (pin "7")
+  )
   (symbol (lib_id "power:VCC") (at 181.61 99.06 0) (unit 1)
