File: B2/timerbPipeline.kicad_sch (KiCad schematic)
At the start: 5 parts, among them U210 74HC04, U211 74HC27, U216 74HC74, U217 74HC74, U230 74HC74

Commit message: Ready for v0.2.2
Other:
- company: (none) -> Daniel Molina
- title: (none) -> 74HCT6526 Board 2
Changed lines of the file:
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@@
 (kicad_sch (version 20211123) (generator eeschema)
   (paper "A4")
+  (title_block
+    (title "74HCT6526 Board 2")
+    (date "2023-06-22")
+    (rev "0.2.2")
+    (company "Daniel Molina")
+    (comment 1 "https://github.com/dmolinagarcia/74HCT6526")
+  )
   (junction (at 92.71 74.93) (diameter 0) (color 0 0 0 0)
   )
