File: B1/B1.kicad_pcb (KiCad board)
At the start: 4 copper layers, 100 x 100 mm, 63 parts, among them U101 74HC244, U102 74HC244, U103 74HCT32, U104 74HCT32, U105 74HC244, U106 74HC688, U107 74HC688, U108 74HC32, U109 74HC74, U110 74HC04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

Commit message: .
Parts:
- added C129: 100n, Capacitor_SMD:C_0603_1608Metric, F.Cu at (189.9, 106.5)
Routing:
- net ~{RES}: track 137.0 -> 139.6 mm
- net GND: track 176.4 -> 177.5 mm, vias 64 -> 65
Other:
- board text added: "74HCT6526 Board 1 v0.1.2"
- board text removed: "74HCT6526 Board 1 v0.1.1"
Changed lines of the file:
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@@
       (net 29 "VCC") (zone_connect 2))
+  )
+  (footprint "Capacitor_SMD:C_0603_1608Metric" (layer "F.Cu")
+    (at 189.89 106.46 90)
+    (descr "Capacitor SMD 0603 (1608 Metric), square (rectangular) end terminal, IPC_7351 nominal, (Body size source: IPC-SM-782 page 76, https://www.pcb-3d.com/wordpress/wp-content/uploads/ipc-sm-782a_amendment_1_and_2.pdf), generated with kicad-footprint-generator")
+    (tags "capacitor")
+    (property "Sheetfile" "buses.kicad_sch")
+    (property "Sheetname" "buses")
+    (attr smd)
+    (fp_text reference "C129" (at 0 -1.43 90) (layer "F.Fab")
+      (effects (font (size 1 1) (thickness 0.15)))
+    )
+    (fp_text value "100n" (at 0 1.43 90) (layer "F.Fab")
+      (effects (font (size 1 1) (thickness 0.15)))
+    )
+    (fp_text user "${REFERENCE}" (at 0 0 90) (layer "F.Fab")
+      (effects (font (size 0.4 0.4) (thickness 0.06)))
+    )
+    (fp_line (start -0.14058 0.51) (end 0.14058 0.51) (layer "F.SilkS") (width 0.12))
+    (fp_line (start -0.14058 -0.51) (end 0.14058 -0.51) (layer "F.SilkS") (width 0.12))
+    (fp_line (start -1.48 0.73) (end -1.48 -0.73) (layer "F.CrtYd") (width 0.05))
+    (fp_line (start 1.48 -0.73) (end 1.48 0.73) (layer "F.CrtYd") (width 0.05))
+    (fp_line (start -1.48 -0.73) (end 1.48 -0.73) (layer "F.CrtYd") (width 0.05))
+    (fp_line (start 1.48 0.73) (end -1.48 0.73) (layer "F.CrtYd") (width 0.05))
+    (fp_line (start 0.8 0.4) (end -0.8 0.4) (layer "F.Fab") (width 0.1))
+    (fp_line (start -0.8 0.4) (end -0.8 -0.4) (layer "F.Fab") (width 0.1))
+    (fp_line (start 0.8 -0.4) (end 0.8 0.4) (layer "F.Fab") (width 0.1))
+    (fp_line (start -0.8 -0.4) (end 0.8 -0.4) (layer "F.Fab") (width 0.1))
+    (pad "1" smd roundrect (at -0.775 0 90) (size 0.9 0.95) (layers "F.Cu" "F.Paste" "F.Mask") (roundrect_rratio 0.25)
+      (net 20 "~{RES}") (pintype "passive"))
+    (pad "2" smd roundrect (at 0.775 0 90) (size 0.9 0.95) (layers "F.Cu" "F.Paste" "F.Mask") (roundrect_rratio 0.25)
+      (net 30 "GND") (pintype "passive"))
+    (model "${KICAD6_3DMODEL_DIR}/Capacitor_SMD.3dshapes/C_0603_1608Metric.wrl"
+      (offset (xyz 0 0 0))
+      (scale (xyz 1 1 1))
+      (rotate (xyz 0 0 0))
+    )
   )
   (footprint "Package_SO:SOIC-20W_7.5x12.8mm_P1.27mm" (layer "F.Cu")
@@
   (gr_line (start 99.981802 45.005538) (end 99.981802 145.005538) (layer "Edge.Cuts") (width 0.05))
   (gr_line (start 199.981802 145.005538) (end 199.981802 45.005538) (layer "Edge.Cuts") (width 0.05))
-  (gr_text "74HCT6526\nBoard 1\nv0.1.1" (at 156.1592 139.78382) (layer "F.SilkS")
+  (gr_text "74HCT6526\nBoard 1\nv0.1.2" (at 156.1592 139.78382) (layer "F.SilkS")
     (effects (font (size 1 1) (thickness 0.25) italic))
   )
@@
   (segment (start 178.02606 137.2108) (end 178.02606 109.50702) (width 0.127) (layer "B.Cu") (net 18))
   (segment (start 167.70604 69.06514) (end 167.089079 68.448179) (width 0.127) (layer "F.Cu") (net 20))
+  (segment (start 189.96 107.305) (end 189.96 109.8) (width 0.09) (layer "F.Cu") (net 20))
   (segment (start 171.74464 109.08538) (end 187.44946 109.08538) (width 0.127) (layer "F.Cu") (net 20))
   (segment (start 167.75176 113.07826) (end 171.74464 109.08538) (width 0.127) (layer "F.Cu") (net 20))
@@
   (segment (start 158.76778 131.9022) (end 160.70222 131.9022) (width 0.127) (layer "F.Cu") (net 20))
   (segment (start 182.5498 70.56628) (end 181.04866 69.06514) (width 0.127) (layer "F.Cu") (net 20))
+  (segment (start 189.89 107.235) (end 189.96 107.305) (width 0.09) (layer "F.Cu") (net 20))
   (segment (start 187.44946 109.08538) (end 189.24538 109.08538) (width 0.127) (layer "F.Cu") (net 20))
   (segment (start 147.2312 126.9112) (end 148.5012 128.1812) (width 0.127) (layer "F.Cu") (net 20))
@@
   (segment (start 110.0836 71.0692) (end 118.628911 71.0692) (width 0.127) (layer "F.Cu") (net 30))
   (segment (start 107.92206 69.01434) (end 107.92206 70.69582) (width 0.127) (layer "F.Cu") (net 30))
+  (segment (start 189.89 105.685) (end 189.89 104.58) (width 0.254) (layer "F.Cu") (net 30))
   (segment (start 118.22788 89.5492) (end 118.84152 88.93556) (width 0.127) (layer "F.Cu") (net 30))
   (segment (start 136.38288 78.6967) (end 136.96188 78.1177) (width 0.127) (layer "F.Cu") (net 30))
@@
   (via (at 152.4 95.5294) (size 0.5) (drill 0.2) (layers "F.Cu" "B.Cu") (net 30))
   (via (at 120.6754 116.3574) (size 0.5) (drill 0.2) (layers "F.Cu" "B.Cu") (net 30))
+  (via (at 189.89 104.58) (size 0.5) (drill 0.2) (layers "F.Cu" "B.Cu") (net 30))
   (via (at 146.1008 134.5184) (size 0.5) (drill 0.2) (layers "F.Cu" "B.Cu") (net 30))
   (via (at 161.3154 90.043) (size 0.5) (drill 0.2) (layers "F.Cu" "B.Cu") (net 30))

Commit message: B0 ready for v0.2.0 release.
Connections:
- U123 pad 1: Net-(U123-Pad1) -> Net-(U123-Pad8)
- U123 pad 10: Net-(U123-Pad1) -> Net-(U123-Pad10)
- U123 pad 6: Net-(U123-Pad1) -> Net-(U123-Pad10)
- U123 pad 8: unconnected-(U123-Pad8) -> Net-(U123-Pad8)
Routing:
- net Net-(U123-Pad8): track 0.00 -> 15.5 mm
- net Net-(U123-Pad1): track 14.8 -> 0.00 mm
- net Net-(U123-Pad10): track 0.00 -> 5.48 mm
- net VCC: track 136.0 -> 141.3 mm, vias 46 -> 45
- net PHI2: track 151.3 -> 153.4 mm
- net D6: track 78.5 -> 77.5 mm
- net /~{PHI2}: track 184.3 -> 185.3 mm
- net Net-(U118-Pad2): track 29.2 -> 28.7 mm

Commit message: B1 ready for v0.2.0 release
Parts:
- removed C129: 100n, Capacitor_SMD:C_0603_1608Metric
- added C100: 100n, Capacitor_SMD:C_0603_1608Metric, F.Cu at (189.9, 106.5)
Connections:
- CONTROLBUS1 pad 18: TARUNMODE -> unconnected-(CONTROLBUS1-Pad18)
- U105 pad 15: TARUNMODE -> /crega/TARUNMODE
- U108 pad 9: TARUNMODE -> /crega/TARUNMODE
- U120 pad 12: TARUNMODE -> /crega/TARUNMODE
- U128 pad 12: TARUNMODE -> /crega/TARUNMODE
Routing:
- net TARUNMODE: track 136.6 -> 0.00 mm, vias 5 -> 0
- net /crega/TARUNMODE: track 0.00 -> 123.4 mm, vias 0 -> 4
- net TAOUT: track 66.8 -> 63.5 mm
- net D0: track 102.0 -> 104.2 mm
- net CNT: track 82.1 -> 80.3 mm
- net GND: track 177.4 -> 175.7 mm
- net /~{PHI2}: track 185.3 -> 183.8 mm
- net TAPULSE: track 80.3 -> 78.9 mm
- net DZ4: track 53.6 -> 54.8 mm
- net Net-(U124-Pad6): track 18.3 -> 17.4 mm
- net TASTART: track 138.3 -> 137.4 mm
- net PHI2: track 153.4 -> 152.5 mm
- net /crega/rTASTART: track 82.2 -> 81.3 mm
- net DZ0: track 56.1 -> 56.9 mm
- net D1: track 93.1 -> 93.9 mm, vias 0 -> 2
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Other:
- board text added: "74HCT6526 Board 1 v0.2.0"
- board text removed: "74HCT6526 Board 1 v0.1.2"

Commit message: Ready for v0.2.1
Parts:
- added C129: 100n, Capacitor_SMD:C_0603_1608Metric, F.Cu at (157.6, 79.3)
- added U129: 74HC74, Package_SO:SO-14_3.9x8.65mm_P1.27mm, F.Cu at (154.1, 85.0)
- moved C113 2.98 mm to (148.6, 79.3)
- moved U113 2.98 mm to (145.0, 85.0)
- moved U114 1.18 mm to (164.3, 85.6)
- moved C114 0.74 mm to (167.2, 78.7), turned to 90 degrees
Connections:
- U118 pad 13: Net-(U113-Pad8) -> /timera/TAPULSESET
- U119 pad 11: /~{PHI2} -> VCC
- U119 pad 13: Net-(U113-Pad8) -> VCC
- U119 pad 9: Net-(U119-Pad9) -> unconnected-(U119-Pad9)
- U127 pad 4: Net-(U119-Pad9) -> Net-(U127-Pad4)
Routing:
- net Net-(U127-Pad4): track 0.00 -> 49.3 mm, vias 0 -> 2
- net /timera/TAPULSESET: track 24.8 -> 58.0 mm, vias 2 -> 3
- net Net-(U119-Pad9): track 31.5 -> 0.00 mm, vias 2 -> 0
- net /~{PHI2}: track 183.8 -> 199.2 mm, vias 6 -> 5
- net /TALOAD: track 35.9 -> 50.3 mm
- net Net-(U113-Pad8): track 29.4 -> 16.3 mm
- net VCC: track 141.3 -> 152.9 mm, vias 45 -> 48
- net Net-(U129-Pad12): track 0.00 -> 10.9 mm
- net /crega/TAUNDERFLOW: track 91.5 -> 100.9 mm
- net GND: track 175.7 -> 182.1 mm, vias 65 -> 68
- net PHI2: track 152.5 -> 158.1 mm
- net TAPULSE: track 78.9 -> 73.7 mm
- net /timera/timer16/~{TIMER_UNDERFLOW}: track 20.2 -> 18.1 mm
- net /timera/~{WETAHI}: track 107.6 -> 109.0 mm
- net /TAOUTMODE: track 106.5 -> 105.3 mm
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Other:
- board text added: "74HCT6526 Board 1 v0.2.1"
- board text removed: "74HCT6526 Board 1 v0.2.0"

Commit message: .
Connections:
- net /timera/TAPULSESET renamed /timera/timeraOutput/TAPULSESET
- net /timera/TATOGGLE renamed /timera/timeraOutput/TATOGGLE
- net /timera/TATOGGLESET renamed /timera/timeraOutput/TATOGGLESET
- net /timera/~TATOGGLE renamed /timera/timeraOutput/~TATOGGLE
- net Net-(U124-Pad8) renamed /timera/timeraPipeline/TIMERAINPUT
- U111 pad 11: /timera/~{TALOAD} -> Net-(U111-Pad11)
- U112 pad 11: /timera/~{TALOAD} -> Net-(U111-Pad11)
- U116 pad 11: /timera/~{TALOAD} -> Net-(U111-Pad11)
- U117 pad 11: /timera/~{TALOAD} -> Net-(U111-Pad11)
- U117 pad 4: /timera/TACOUNT -> Net-(U117-Pad4)
- U119 pad 5: Net-(U119-Pad5) -> /timera/TACOUNT
- U127 pad 11: /timera/TACOUNT -> Net-(U117-Pad4)
- U127 pad 13: Net-(U119-Pad5) -> /timera/TACOUNT
- U127 pad 4: Net-(U127-Pad4) -> /timera/~{TALOAD}
- U127 pad 6: /timera/~{TALOAD} -> Net-(U111-Pad11)
- U129 pad 9: Net-(U127-Pad4) -> /timera/~{TALOAD}
Routing:
- net Net-(U111-Pad11): track 0.00 -> 96.9 mm
- net Net-(U117-Pad4): track 0.00 -> 59.1 mm
- net Net-(U127-Pad4): track 49.3 -> 0.00 mm, vias 2 -> 0
- net /timera/~{TALOAD}: track 96.9 -> 49.3 mm, vias 0 -> 2
- net Net-(U119-Pad5): track 30.0 -> 0.00 mm, vias 2 -> 0
- net /timera/TACOUNT: track 59.1 -> 30.0 mm, vias 0 -> 2

Commit message: Ready for v0.2.2
Other:
- board text added: "74HCT6526 Board 1 v0.2.2"
- board text removed: "74HCT6526 Board 1 v0.2.1"
Changed lines of the file:
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@@
   (title_block
     (title "74HCT6526 Board 1")
-    (date "2023-03-25")
-    (rev "0.2.1")
+    (date "2023-06-22")
+    (rev "0.2.2")
     (company "Daniel Molina")
     (comment 1 "https://github.com/dmolinagarcia/74HCT6526")
@@
   (gr_line (start 99.981802 45.005538) (end 99.981802 145.005538) (layer "Edge.Cuts") (width 0.05))
   (gr_line (start 199.981802 145.005538) (end 199.981802 45.005538) (layer "Edge.Cuts") (width 0.05))
-  (gr_text "74HCT6526\nBoard 1\nv0.2.1" (at 156.1592 139.78382) (layer "F.SilkS")
+  (gr_text "74HCT6526\nBoard 1\nv0.2.2" (at 156.1592 139.78382) (layer "F.SilkS")
     (effects (font (size 1 1) (thickness 0.25) italic))
   )
