File: B1/B1.kicad_sch (KiCad schematic)
At the start: 1 part, among them U110 74HC04

Commit message: B2 almost ready
Other:
- sheet buses ports: added DZ[0..7], D[0..7], ~{EN[0..15]}; removed {DATABUS}, {ENABLEBUS}
- moved on the sheet: U110A

Commit message: B0 ready for v0.2.0 release.
Other:
- sheet crega ports: added none; removed TARUNMODE
Changed lines of the file:
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@@
   (title_block
     (title "74HCT6526 Board 1")
-    (date "2022-10-08")
-    (rev "0.1.2")
+    (date "2023-01-22")
+    (rev "0.2.0")
     (company "Daniel Molina")
     (comment 1 "https://github.com/dmolinagarcia/74HCT6526")
   )
   (bus_alias "CONTROLBUS" (members "TASTART" "CNT" "SP" "PHI2" "~{FLAG}" "TOD" "TAPULSE" "TBPULSE" "TODIRQ" "~{IRQ}" "PB6ON" "PB7ON" "TAOUT" "TBOUT" "SPMODE" "TODIN" "ALARM" "ENABLE_NAND" "TARUNMODE" "~{RES}"))
+  (bus_alias "DATABUS" (members "D[0..7]" "DZ[0..7]"))
   (bus_alias "ENABLEBUS" (members "~{EN[0..15]}"))
-  (bus_alias "DATABUS" (members "D[0..7]" "DZ[0..7]"))
   (junction (at 46.99 48.26) (diameter 0) (color 0 0 0 0)
   )
@@
     (stroke (width 0) (type default) (color 0 0 0 0))
   )
-  (bus_entry (at 167.64 91.44) (size 2.54 -2.54)
-    (stroke (width 0) (type default) (color 0 0 0 0))
-  )
   (bus_entry (at 167.64 83.82) (size 2.54 -2.54)
     (stroke (width 0) (type default) (color 0 0 0 0))
@@
     (stroke (width 0) (type default) (color 0 0 0 0))
   )
-  (wire (pts (xy 154.94 91.44) (xy 167.64 91.44))
-    (stroke (width 0) (type default) (color 0 0 0 0))
-  )
   (wire (pts (xy 154.94 101.6) (xy 222.25 101.6))
     (stroke (width 0) (type default) (color 0 0 0 0))
   )
   (bus (pts (xy 170.18 78.74) (xy 170.18 81.28))
-    (stroke (width 0) (type default) (color 0 0 0 0))
-  )
-  (bus (pts (xy 170.18 86.36) (xy 170.18 88.9))
     (stroke (width 0) (type default) (color 0 0 0 0))
   )
@@
   )
   (label "TODIN" (at 156.21 83.82 0)
-    (effects (font (size 1.27 1.27)) (justify left bottom))
-  )
-  (label "TARUNMODE" (at 156.21 91.44 0)
     (effects (font (size 1.27 1.27)) (justify left bottom))
   )
@@
       (effects (font (size 1.27 1.27)) (justify right))
     )
-    (pin "TARUNMODE" output (at 154.94 91.44 0)
-      (effects (font (size 1.27 1.27)) (justify right))
-    )
     (pin "TAINMODE" output (at 154.94 101.6 0)
       (effects (font (size 1.27 1.27)) (justify right))
@@
       (reference "#PWR0171") (unit 1) (value "GND") (footprint "")
     )
+    (path "/d71e373b-2126-4572-b605-db646e364722/f601c79d-0a90-4f06-932e-aa5468725aa3"
+      (reference "C100") (unit 1) (value "100n") (footprint "Capacitor_SMD:C_0603_1608Metric")
+    )
     (path "/c09c7409-d5b2-4c4f-a820-cde0cb763f7f/12dcbe09-d7c9-470c-a39e-e8b7d1242732"
       (reference "C101") (unit 1) (value "100n") (footprint "Capacitor_SMD:C_0603_1608Metric")
@@
       (reference "C128") (unit 1) (value "100n") (footprint "Capacitor_SMD:C_0603_1608Metric")
     )
-    (path "/d71e373b-2126-4572-b605-db646e364722/f601c79d-0a90-4f06-932e-aa5468725aa3"
-      (reference "C129") (unit 1) (value "100n") (footprint "Capacitor_SMD:C_0603_1608Metric")
-    )
     (path "/d71e373b-2126-4572-b605-db646e364722/25a0a619-bd2a-4e5a-afc1-97e231f72e29"
