File: B1/crega.kicad_sch (KiCad schematic)
At the start: 9 parts, among them U105 74HC244, U108 74HC32, U110 74HC04, U115 74HC74, U120 74HC74, U124 74HC00, U125 74HC74, U127 74HC08, U128 74HC377

Commit message: B0 ready for v0.2.0 release.
Changed lines of the file:
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@@
   (title_block
     (title "74HCT6526 Board 1")
-    (date "2022-10-08")
-    (rev "0.1.2")
+    (date "2023-01-22")
+    (rev "0.2.0")
     (company "Daniel Molina")
     (comment 1 "https://github.com/dmolinagarcia/74HCT6526")
@@
   (junction (at 200.66 39.37) (diameter 0) (color 0 0 0 0)
   )
-  (junction (at 217.17 57.15) (diameter 0) (color 0 0 0 0)
-  )
   (junction (at 198.12 52.07) (diameter 0) (color 0 0 0 0)
   )
   (junction (at 20.32 57.15) (diameter 0) (color 0 0 0 0)
   )
+  (junction (at 203.2 49.53) (diameter 0) (color 0 0 0 0)
+  )
   (junction (at 215.9 57.15) (diameter 0) (color 0 0 0 0)
   )
-  (junction (at 203.2 49.53) (diameter 0) (color 0 0 0 0)
-  )
   (junction (at 195.58 92.71) (diameter 0) (color 0 0 0 0)
   )
@@
   )
   (junction (at 40.64 71.12) (diameter 0) (color 0 0 0 0)
-  )
-  (junction (at 205.74 105.41) (diameter 0) (color 0 0 0 0)
   )
   (junction (at 74.93 66.04) (diameter 0) (color 0 0 0 0)
@@
     (stroke (width 0) (type default) (color 0 0 0 0))
   )
+  (wire (pts (xy 100.33 24.13) (xy 100.33 26.67))
+    (stroke (width 0) (type default) (color 0 0 0 0))
+  )
   (wire (pts (xy 198.12 52.07) (xy 217.17 52.07))
     (stroke (width 0) (type default) (color 0 0 0 0))
@@
     (stroke (width 0) (type default) (color 0 0 0 0))
   )
+  (wire (pts (xy 215.9 57.15) (xy 217.17 57.15))
+    (stroke (width 0) (type default) (color 0 0 0 0))
+  )
   (wire (pts (xy 195.58 34.29) (xy 195.58 92.71))
     (stroke (width 0) (type default) (color 0 0 0 0))
@@
     (stroke (width 0) (type default) (color 0 0 0 0))
   )
-  (wire (pts (xy 217.17 57.15) (xy 215.9 57.15))
-    (stroke (width 0) (type default) (color 0 0 0 0))
-  )
   (wire (pts (xy 214.63 92.71) (xy 214.63 109.22))
     (stroke (width 0) (type default) (color 0 0 0 0))
@@
     (stroke (width 0) (type default) (color 0 0 0 0))
   )
-  (wire (pts (xy 205.74 135.89) (xy 257.81 135.89))
-    (stroke (width 0) (type default) (color 0 0 0 0))
-  )
   (wire (pts (xy 156.21 139.7) (xy 257.81 139.7))
     (stroke (width 0) (type default) (color 0 0 0 0))
@@
     (stroke (width 0) (type default) (color 0 0 0 0))
   )
-  (wire (pts (xy 217.17 57.15) (xy 222.25 57.15))
-    (stroke (width 0) (type default) (color 0 0 0 0))
-  )
   (wire (pts (xy 115.57 105.41) (xy 116.84 105.41))
     (stroke (width 0) (type default) (color 0 0 0 0))
@@
     (stroke (width 0) (type default) (color 0 0 0 0))
   )
-  (wire (pts (xy 205.74 135.89) (xy 205.74 105.41))
-    (stroke (width 0) (type default) (color 0 0 0 0))
-  )
   (wire (pts (xy 116.84 105.41) (xy 116.84 142.24))
     (stroke (width 0) (type default) (color 0 0 0 0))
@@
     (stroke (width 0) (type default) (color 0 0 0 0))
   )
+  (wire (pts (xy 100.33 69.85) (xy 100.33 67.31))
+    (stroke (width 0) (type default) (color 0 0 0 0))
+  )
   (wire (pts (xy 144.78 44.45) (xy 210.82 44.45))
     (stroke (width 0) (type default) (color 0 0 0 0))
@@
   (label "TALOAD" (at 184.785 139.7 0)
     (effects (font (size 1.27 1.27)) (justify left bottom))
-  )
-  (global_label "DZ[0..7]" (shape output) (at 48.26 31.75 0) (fields_autoplaced)
-    (effects (font (size 0.0254 0.0254)) (justify left))
-    (property "Intersheet References" "${INTERSHEET_REFS}" (id 0) (at 48.4681 31.7484 0)
-      (effects (font (size 0.0254 0.0254)) (justify left) hide)
-    )
   )
   (hierarchical_label "~{EN14}" (shape input) (at 35.56 71.12 180)
@@
   )
   (hierarchical_label "PB6ON" (shape output) (at 257.81 77.47 0)
-    (effects (font (size 1.27 1.27)) (justify left))
-  )
-  (hierarchical_label "TARUNMODE" (shape output) (at 257.81 135.89 0)
     (effects (font (size 1.27 1.27)) (justify left))
   )
@@
     (pin "7")
   )
-  (symbol (lib_id "power:VCC") (at 100.33 26.67 0) (unit 1)
+  (symbol (lib_id "power:VCC") (at 100.33 24.13 0) (unit 1)
     (in_bom yes) (on_board yes) (fields_autoplaced)
-    (property "Reference" "#PWR0106" (id 0) (at 100.33 30.48 0)
-      (effects (font (size 1.27 1.27)) hide)
-    )
-    (property "Value" "VCC" (id 1) (at 100.33 23.0655 0))
-    (property "Footprint" "" (id 2) (at 100.33 26.67 0)
-      (effects (font (size 1.27 1.27)) hide)
-    )
-    (property "Datasheet" "" (id 3) (at 100.33 26.67 0)
+    (property "Reference" "#PWR0106" (id 0) (at 100.33 27.94 0)
+      (effects (font (size 1.27 1.27)) hide)
+    )
+    (property "Value" "VCC" (id 1) (at 100.33 20.5255 0))
+    (property "Footprint" "" (id 2) (at 100.33 24.13 0)
+      (effects (font (size 1.27 1.27)) hide)
+    )
+    (property "Datasheet" "" (id 3) (at 100.33 24.13 0)
       (effects (font (size 1.27 1.27)) hide)
     )
@@
     (pin "7")
   )
-  (symbol (lib_id "power:GND") (at 100.33 67.31 0) (unit 1)
+  (symbol (lib_id "power:GND") (at 100.33 69.85 0) (unit 1)
     (in_bom yes) (on_board yes) (fields_autoplaced)
-    (property "Reference" "#PWR0107" (id 0) (at 100.33 73.66 0)
-      (effects (font (size 1.27 1.27)) hide)
-    )
-    (property "Value" "GND" (id 1) (at 100.33 71.8725 0))
-    (property "Footprint" "" (id 2) (at 100.33 67.31 0)
-      (effects (font (size 1.27 1.27)) hide)
-    )
-    (property "Datasheet" "" (id 3) (at 100.33 67.31 0)
-      (effects (font (size 1.27 1.27)) hide)
-    )
+    (property "Reference" "#PWR0107" (id 0) (at 100.33 76.2 0)
+      (effects (font (size 1.27 1.27)) hide)
+    )
+    (property "Value" "GND" (id 1) (at 100.33 74.4125 0))
+    (property "Footprint" "" (id 2) (at 100.33 69.85 0)
+      (effects (font (size 1.27 1.27)) hide)
+    )
+    (property "Datasheet" "" (id 3) (at 100.33 69.85 0)
+      (effects (font (size 1.27 1.27)) hide)
+    )
