File: B1/power.kicad_sch (KiCad schematic)
At the start: 43 parts, among them U103 74HCT32, U104 74HCT32, U108 74HC32, U109 74HC74, U110 74HC04, U113 74HC27, U115 74HC74, U118 74HC74, U119 74HC74, U120 74HC74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

Commit message: Almost 0.1.1
Other:
- company: (none) -> Daniel Molina
- title: (none) -> 74HCT6526 Board 1
Changed lines of the file:
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@@
 (kicad_sch (version 20211123) (generator eeschema)
   (paper "A4")
+  (title_block
+    (title "74HCT6526 Board 1")
+    (date "2022-08-17")
+    (rev "0.1")
+    (company "Daniel Molina")
+    (comment 1 "https://github.com/dmolinagarcia/74HCT6526")
+  )
   (junction (at 137.16 63.5) (diameter 0) (color 0 0 0 0)
   )

Commit message: Ready for v0.2.1
Parts:
- added C129: 100n, Capacitor_SMD:C_0603_1608Metric, symbol Device:C
- added unit 2 of U119
- added U129: 74HC74, Package_SO:SO-14_3.9x8.65mm_P1.27mm, symbol 74xx:74HC74
Connections:
- net GND: now also C129.2, U129.7 (GND)
- net VCC: now also C129.1, U119.10 (~{S}), U119.11 (C), U119.12 (D), U119.13 (~{R}), U129.14 (VCC)
- no-connect marks 2 -> 4
