File: B1/resetData.kicad_sch (KiCad schematic)
At the start: 3 parts, among them U103 74HCT32, U104 74HCT32, U110 74HC04

Commit message: Almost 0.1.1
Other:
- company: (none) -> Daniel Molina
- title: (none) -> 74HCT6526 Board 1
Changed lines of the file:
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@@
 (kicad_sch (version 20211123) (generator eeschema)
   (paper "A4")
+  (title_block
+    (title "74HCT6526 Board 1")
+    (date "2022-08-17")
+    (rev "0.1")
+    (company "Daniel Molina")
+    (comment 1 "https://github.com/dmolinagarcia/74HCT6526")
+  )
   (junction (at 133.35 99.06) (diameter 0) (color 0 0 0 0)
   )
