File: B1/timer16.kicad_sch (KiCad schematic)
At the start: 8 parts, among them U101 74HC244, U102 74HC244, U106 74HC688, U107 74HC688, U111 74HC193, U112 74HC193, U116 74HC193, U117 74HC193

Commit message: Almost 0.1.1
Other:
- company: (none) -> Daniel Molina
- title: (none) -> 74HCT6526 Board 1
Changed lines of the file:
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@@
 (kicad_sch (version 20211123) (generator eeschema)
   (paper "A4")
+  (title_block
+    (title "74HCT6526 Board 1")
+    (date "2022-08-17")
+    (rev "0.1")
+    (company "Daniel Molina")
+    (comment 1 "https://github.com/dmolinagarcia/74HCT6526")
+  )
   (junction (at 237.49 133.35) (diameter 0) (color 0 0 0 0)
   )

Commit message: .
Parts:
- added U127: 74HC08, Package_SO:SO-14_3.9x8.65mm_P1.27mm, symbol Custom 74xx:74HC08
Connections:
- net CLK: now also U127.13; no longer U117.4 (DOWN)
- net ~{LOAD}: now also U127.4; no longer U111.11 (~{LOAD}), U112.11 (~{LOAD}), U116.11 (~{LOAD}), U117.11 (~{LOAD})
- new net: U111.11 (~{LOAD}), U112.11 (~{LOAD}), U116.11 (~{LOAD}), U117.11 (~{LOAD}), U127.6
- new net: U117.4 (DOWN), U127.11
- new net PHI2: U127.12
- new net ~{RES}: U127.5
Changed lines of the file:
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@@
+    (stroke (width 0) (type default) (color 0 0 0 0))
+  )
+  (wire (pts (xy 21.59 48.26) (xy 24.13 48.26))
     (stroke (width 0) (type default) (color 0 0 0 0))
   )
@@
     (stroke (width 0) (type default) (color 0 0 0 0))
   )
+  (wire (pts (xy 71.12 50.8) (xy 71.12 46.99))
+    (stroke (width 0) (type default) (color 0 0 0 0))
+  )
   (wire (pts (xy 236.22 86.36) (xy 236.22 73.66))
     (stroke (width 0) (type default) (color 0 0 0 0))
@@
     (stroke (width 0) (type default) (color 0 0 0 0))
   )
+  (wire (pts (xy 21.59 36.83) (xy 24.13 36.83))
+    (stroke (width 0) (type default) (color 0 0 0 0))
+  )
   (wire (pts (xy 168.91 129.54) (xy 168.91 132.08))
     (stroke (width 0) (type default) (color 0 0 0 0))
@@
     (stroke (width 0) (type default) (color 0 0 0 0))
   )
+  (wire (pts (xy 21.59 41.91) (xy 24.13 41.91))
+    (stroke (width 0) (type default) (color 0 0 0 0))
+  )
   (bus (pts (xy 63.5 29.21) (xy 63.5 31.75))
     (stroke (width 0) (type default) (color 0 0 0 0))
@@
     (stroke (width 0) (type default) (color 0 0 0 0))
   )
+  (wire (pts (xy 39.37 50.8) (xy 71.12 50.8))
+    (stroke (width 0) (type default) (color 0 0 0 0))
+  )
   (bus (pts (xy 124.46 163.83) (xy 124.46 161.29))
     (stroke (width 0) (type default) (color 0 0 0 0))
@@
     (stroke (width 0) (type default) (color 0 0 0 0))
   )
-  (wire (pts (xy 74.295 46.99) (xy 85.09 46.99))
+  (wire (pts (xy 71.12 46.99) (xy 85.09 46.99))
     (stroke (width 0) (type default) (color 0 0 0 0))
   )
@@
   )
   (bus (pts (xy 63.5 72.39) (xy 63.5 74.93))
+    (stroke (width 0) (type default) (color 0 0 0 0))
+  )
+  (wire (pts (xy 21.59 53.34) (xy 24.13 53.34))
     (stroke (width 0) (type default) (color 0 0 0 0))
   )
@@
     )
   )
-  (hierarchical_label "CLK" (shape input) (at 74.295 46.99 180)
+  (hierarchical_label "PHI2" (shape input) (at 21.59 53.34 180)
     (effects (font (size 1.27 1.27)) (justify right))
   )
-  (hierarchical_label "~{LOAD}" (shape input) (at 39.37 39.37 180)
+  (hierarchical_label "CLK" (shape input) (at 21.59 48.26 180)
+    (effects (font (size 1.27 1.27)) (justify right))
+  )
+  (hierarchical_label "~{LOAD}" (shape input) (at 21.59 36.83 180)
+    (effects (font (size 1.27 1.27)) (justify right))
+  )
+  (hierarchical_label "~{RES}" (shape input) (at 21.59 41.91 180)
     (effects (font (size 1.27 1.27)) (justify right))
   )
@@
     (pin "9")
   )
+  (symbol (lib_id "Custom 74xx:74HC08") (at 31.75 39.37 0) (unit 2)
+    (in_bom yes) (on_board yes)
+    (property "Reference" "U127" (id 0) (at 31.75 39.37 0))
+    (property "Value" "74HC08" (id 1) (at 31.75 41.91 0))
+    (property "Footprint" "Package_SO:SO-14_3.9x8.65mm_P1.27mm" (id 2) (at 31.75 39.37 0)
+      (effects (font (size 1.27 1.27)) hide)
+    )
+    (property "Datasheet" "" (id 3) (at 31.75 33.02 0)
+      (effects (font (size 1.27 1.27)) hide)
+    )
+    (pin "1")
+    (pin "2")
+    (pin "3")
+    (pin "4")
+    (pin "5")
+    (pin "6")
+    (pin "10")
+    (pin "8")
+    (pin "9")
+    (pin "11")
+    (pin "12")
+    (pin "13")
+    (pin "14")
+    (pin "7")
+  )
   (symbol (lib_id "power:GND") (at 237.49 68.58 0) (unit 1)
     (in_bom yes) (on_board yes)
@@
     (pin "1")
   )
+  (symbol (lib_id "Custom 74xx:74HC08") (at 31.75 50.8 0) (mirror x) (unit 4)
+    (in_bom yes) (on_board yes)
+    (property "Reference" "U127" (id 0) (at 31.115 51.435 0))
+    (property "Value" "74HC08" (id 1) (at 31.75 55.8014 0))
+    (property "Footprint" "Package_SO:SO-14_3.9x8.65mm_P1.27mm" (id 2) (at 31.75 50.8 0)
+      (effects (font (size 1.27 1.27)) hide)
+    )
+    (property "Datasheet" "" (id 3) (at 31.75 57.15 0)
+      (effects (font (size 1.27 1.27)) hide)
+    )
+    (pin "1")
+    (pin "2")
+    (pin "3")
+    (pin "4")
+    (pin "5")
+    (pin "6")
+    (pin "10")
+    (pin "8")
+    (pin "9")
+    (pin "11")
+    (pin "12")
+    (pin "13")
+    (pin "14")
+    (pin "7")
+  )
   (symbol (lib_id "power:GND") (at 97.79 57.15 0) (unit 1)
