File: B1/timera.kicad_sch (KiCad schematic)
At the start: 14 parts, among them U108 74HC32, U109 74HC74, U110 74HC04, U113 74HC27, U114 74HC153, U115 74HC74, U118 74HC74, U119 74HC74, U121 74HC377, U122 74HC377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

Commit message: B0 ready for v0.2.0 release.
Connections:
- net at U123.10 (~{S}), U123.6 (~{Q}): no longer U123.1 (~{R})
- net at U123.8 (~{Q}): now also U123.1 (~{R})
- no-connect marks 8 -> 7
Changed lines of the file:
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@@
   (title_block
     (title "74HCT6526 Board 1")
-    (date "2022-10-08")
-    (rev "0.1.2")
+    (date "2023-01-22")
+    (rev "0.2.0")
     (company "Daniel Molina")
     (comment 1 "https://github.com/dmolinagarcia/74HCT6526")
@@
   (junction (at 30.48 86.36) (diameter 0) (color 0 0 0 0)
   )
-  (junction (at 59.69 31.75) (diameter 0) (color 0 0 0 0)
-  )
   (junction (at 135.89 53.34) (diameter 0) (color 0 0 0 0)
   )
@@
   (junction (at 72.39 134.62) (diameter 0) (color 0 0 0 0)
   )
-  (no_connect (at 80.01 31.75))
   (no_connect (at 57.15 26.67))
   (no_connect (at 100.33 26.67))
@@
     (stroke (width 0) (type default) (color 0 0 0 0))
   )
+  (wire (pts (xy 81.28 31.75) (xy 80.01 31.75))
+    (stroke (width 0) (type default) (color 0 0 0 0))
+  )
   (wire (pts (xy 190.5 69.85) (xy 190.5 73.66))
     (stroke (width 0) (type default) (color 0 0 0 0))
@@
     (stroke (width 0) (type default) (color 0 0 0 0))
   )
-  (wire (pts (xy 49.53 38.1) (xy 49.53 36.83))
+  (wire (pts (xy 49.53 39.37) (xy 49.53 36.83))
     (stroke (width 0) (type default) (color 0 0 0 0))
   )
@@
     (stroke (width 0) (type default) (color 0 0 0 0))
   )
-  (wire (pts (xy 59.69 38.1) (xy 49.53 38.1))
-    (stroke (width 0) (type default) (color 0 0 0 0))
-  )
   (wire (pts (xy 118.11 34.29) (xy 118.11 29.21))
     (stroke (width 0) (type default) (color 0 0 0 0))
@@
     (stroke (width 0) (type default) (color 0 0 0 0))
   )
+  (wire (pts (xy 81.28 39.37) (xy 81.28 31.75))
+    (stroke (width 0) (type default) (color 0 0 0 0))
+  )
   (wire (pts (xy 245.11 86.36) (xy 245.11 88.9))
     (stroke (width 0) (type default) (color 0 0 0 0))
@@
     (stroke (width 0) (type default) (color 0 0 0 0))
   )
+  (wire (pts (xy 49.53 39.37) (xy 81.28 39.37))
+    (stroke (width 0) (type default) (color 0 0 0 0))
+  )
   (wire (pts (xy 233.68 146.05) (xy 280.67 146.05))
     (stroke (width 0) (type default) (color 0 0 0 0))
@@
     (stroke (width 0) (type default) (color 0 0 0 0))
   )
-  (wire (pts (xy 59.69 31.75) (xy 59.69 38.1))
-    (stroke (width 0) (type default) (color 0 0 0 0))
-  )

Commit message: Ready for v0.2.1
Parts:
- removed unit 2 of U119
- added U129: 74HC74, Package_SO:SO-14_3.9x8.65mm_P1.27mm, symbol 74xx:74HC74
Connections:
- net TAPULSESET: now also U118.13 (~{R})
- net VCC: now also U129.10 (~{S}), U129.2 (D), U129.4 (~{S})
- net ~{PHI2}: now also U129.11 (C), U129.3 (C)
- net at U113.8: now also U129.1 (~{R}), U129.13 (~{R}); no longer U118.13 (~{R})
- net at U127.4: now also U129.9 (Q)
- new net: U129.12 (D), U129.5 (Q)
- no-connect marks 7 -> 8
Other:
- moved on the sheet: U127B

Commit message: .
Parts:
- removed U109, U115, U119, U129: 74HC74, Package_SO:SO-14_3.9x8.65mm_P1.27mm, symbol 74xx:74HC74
- removed U110: 74HC04, Package_SO:SOIC-14_3.9x8.7mm_P1.27mm, symbol 74xx:74HC04
- removed U113: 74HC27, Package_SO:SO-14_3.9x8.65mm_P1.27mm, symbol 74xx:74LS27
- removed U114: 74HC153, Package_SO:SOIC-16_3.9x9.9mm_P1.27mm, symbol 74xx:74LS153
- removed unit 2 of U118
- removed U127: 74HC08, Package_SO:SO-14_3.9x8.65mm_P1.27mm, symbol Custom 74xx:74HC08
Connections:
- net timeraPipeline/TIMERAINPUT: now reaches U124.8
- no-connect marks 8 -> 2
Other:
- added sheet timeraOutput (timeraOutput.kicad_sch)
- added sheet timeraPipeline (timeraPipeline.kicad_sch)
- sheet timer16 ports: added PHI2, ~{RES}; removed none
- moved on the sheet: U118A, U123A, U123B, U124C
