File: B4/B4.kicad_pcb (KiCad board)
At the start: 4 copper layers, 100 x 100 mm, 3 parts

Commit message: .
Connections:
- net /buses/~FLAG renamed /buses/~{FLAG}
- net /buses/~IRQ renamed /buses/~{IRQ}
- net /buses/~RES renamed /buses/~{RES}

Commit message: Ready for v0.2.1
Parts:
- added C400: 100n, Capacitor_SMD:C_0603_1608Metric, F.Cu at (190.8, 106.4)
- added U1: 74HC04, Package_SO:SOIC-14_3.9x8.7mm_P1.27mm, F.Cu at (181.0, 139.2)
- added U2: 74HC377, Package_SO:SOIC-20W_7.5x12.8mm_P1.27mm, F.Cu at (116.0, 58.5)
- added U3: 74HC377, Package_SO:SOIC-20W_7.5x12.8mm_P1.27mm, F.Cu at (115.7, 101.3)
- added U4: 74HC377, Package_SO:SOIC-20W_7.5x12.8mm_P1.27mm, F.Cu at (115.9, 81.1)
- added U5: 74HC377, Package_SO:SOIC-20W_7.5x12.8mm_P1.27mm, F.Cu at (115.9, 120.5)
Connections:
- net /buses/ALARM renamed ALARM
- net /buses/CNT renamed CNT
- net /buses/D0 renamed D0
- net /buses/D1 renamed D1
- net /buses/D2 renamed D2
- net /buses/D3 renamed D3
- net /buses/D4 renamed D4
- net /buses/D5 renamed D5
- net /buses/D6 renamed D6
- net /buses/D7 renamed D7
- net /buses/EN10 renamed ~{EN10}
- net /buses/EN11 renamed ~{EN11}
- net /buses/EN12 renamed ~{EN12}
- net /buses/EN13 renamed ~{EN13}
- net /buses/EN14 renamed ~{EN14}
- net /buses/EN15 renamed ~{EN15}
- net /buses/EN4 renamed ~{EN4}
- net /buses/EN5 renamed ~{EN5}
- net /buses/EN6 renamed ~{EN6}
- net /buses/EN7 renamed ~{EN7}
- net /buses/EN8 renamed ~{EN8}
- net /buses/EN9 renamed ~{EN9}
- net /buses/ENABLE_NAND renamed ENABLE_NAND
- net /buses/PB6ON renamed PB6ON
- net /buses/PB7ON renamed PB7ON
- net /buses/SP renamed SP
- net /buses/SPMODE renamed SPMODE
- net /buses/TAOUT renamed TAOUT
- net /buses/TAPULSE renamed TAPULSE
- net /buses/TASTART renamed TASTART
- net /buses/TBOUT renamed TBOUT
- net /buses/TBPULSE renamed TBPULSE
- net /buses/TOD renamed TOD
- net /buses/TODIN renamed TODIN
- net /buses/TODIRQ renamed TODIRQ
- net /buses/~{FLAG} renamed ~{FLAG}
- net /buses/~{IRQ} renamed ~{IRQ}
- CONTROLBUS4 pad 18: /buses/TARUNMODE -> unconnected-(CONTROLBUS4-Pad18)
- CONTROLBUS4 pad 20: /buses/~{RES} -> ~{RES}
- CONTROLBUS4 pad 7: /buses/PHI2 -> PHI2
- DATABUS4 pad 11: GND -> VCC
- DATABUS4 pad 12: VCC -> GND
- DATABUS4 pad 13: /buses/DZ0 -> DZ0
- DATABUS4 pad 14: /buses/DZ4 -> DZ4
- DATABUS4 pad 15: /buses/DZ7 -> DZ7
- DATABUS4 pad 16: /buses/DZ3 -> DZ3
- DATABUS4 pad 17: /buses/DZ1 -> DZ1
- DATABUS4 pad 18: /buses/DZ5 -> DZ5
- DATABUS4 pad 19: /buses/DZ6 -> DZ6
- DATABUS4 pad 20: /buses/DZ2 -> DZ2
- ENABLEBUS4 pad 10: GND -> VCC
- ENABLEBUS4 pad 12: GND -> VCC
- ENABLEBUS4 pad 14: VCC -> GND
- ENABLEBUS4 pad 16: VCC -> GND
- ENABLEBUS4 pad 18: VCC -> GND
- ENABLEBUS4 pad 20: VCC -> GND
- ENABLEBUS4 pad 6: GND -> VCC
- ENABLEBUS4 pad 8: GND -> VCC

Commit message: B2 refactored. B4 Added. TOD sch completed.
Parts:
- removed C400: 100n, Capacitor_SMD:C_0603_1608Metric
- removed U1: 74HC04, Package_SO:SOIC-14_3.9x8.7mm_P1.27mm
- removed U2, U3, U4, U5: 74HC377, Package_SO:SOIC-20W_7.5x12.8mm_P1.27mm
- added C401: 100n, Capacitor_SMD:C_0603_1608Metric, F.Cu at (255.5, 113.3)
- added U401: 74HC00, Package_SO:SOIC-14_3.9x8.7mm_P1.27mm, F.Cu at (309.3, 116.7)
- added U402: 74HC00, Package_SO:SOIC-14_3.9x8.7mm_P1.27mm, F.Cu at (309.3, 84.8)
- added U403: 74HC04, Package_SO:SOIC-14_3.9x8.7mm_P1.27mm, F.Cu at (329.1, 116.2)
- added U404: 74HC32, Package_SO:SOIC-14_3.9x8.7mm_P1.27mm, F.Cu at (309.3, 73.9)
- added U405: 74HC32, Package_SO:SOIC-14_3.9x8.7mm_P1.27mm, F.Cu at (309.3, 63.7)
- added U406: 74HC32, Package_SO:SOIC-14_3.9x8.7mm_P1.27mm, F.Cu at (309.3, 106.5)
- added U407: 74HC377, Package_SO:SOIC-20W_7.5x12.8mm_P1.27mm, F.Cu at (117.0, 59.0)
- added U408: 74HC377, Package_SO:SOIC-20W_7.5x12.8mm_P1.27mm, F.Cu at (117.2, 92.3)
- added U409: 74HC377, Package_SO:SOIC-20W_7.5x12.8mm_P1.27mm, F.Cu at (117.2, 75.4)
- added U410: 74HC377, Package_SO:SOIC-20W_7.5x12.8mm_P1.27mm, F.Cu at (117.2, 109.5)
- added U411: 74HC08, Package_SO:SOIC-14_3.9x8.7mm_P1.27mm, F.Cu at (319.2, 116.6)
- added U412: 74HC193, Package_SO:SOIC-16_3.9x9.9mm_P1.27mm, F.Cu at (129.8, 59.0)
- added U413: 74HC193, Package_SO:SOIC-16_3.9x9.9mm_P1.27mm, F.Cu at (139.8, 59.0)
- added U414: 74HC11, Package_SO:SOIC-14_3.9x8.7mm_P1.27mm, F.Cu at (309.3, 53.0)
- added U415: 74HC32, Package_SO:SOIC-14_3.9x8.7mm_P1.27mm, F.Cu at (349.4, 141.3)
- added U416: 74HC193, Package_SO:SOIC-16_3.9x9.9mm_P1.27mm, F.Cu at (129.5, 75.3)
- added U417: 74HC193, Package_SO:SOIC-16_3.9x9.9mm_P1.27mm, F.Cu at (140.0, 75.3)
- added U418: 74HC08, Package_SO:SOIC-14_3.9x8.7mm_P1.27mm, F.Cu at (338.8, 116.5)
- added U419: 74HC193, Package_SO:SOIC-16_3.9x9.9mm_P1.27mm, F.Cu at (129.6, 92.5)
- added U420: 74HC193, Package_SO:SOIC-16_3.9x9.9mm_P1.27mm, F.Cu at (140.2, 92.4)
- added U421: 74HC373, Package_SO:SOIC-20W_7.5x12.8mm_P1.27mm, F.Cu at (177.5, 59.1)
- added U422: 74HC373, Package_SO:SOIC-20W_7.5x12.8mm_P1.27mm, F.Cu at (177.5, 92.1)
- added U423: 74HC373, Package_SO:SOIC-20W_7.5x12.8mm_P1.27mm, F.Cu at (177.3, 75.6)
- added U424: 74HC373, Package_SO:SOIC-20W_7.5x12.8mm_P1.27mm, F.Cu at (177.1, 109.2)
- added U425: 74HC688, Package_SO:SOIC-20W_7.5x12.8mm_P1.27mm, F.Cu at (162.8, 58.9)
- added U426: 74HC688, Package_SO:SOIC-20W_7.5x12.8mm_P1.27mm, F.Cu at (163.0, 75.5)
- added U427: 74HC688, Package_SO:SOIC-20W_7.5x12.8mm_P1.27mm, F.Cu at (163.0, 92.4)
- added U428: 74HC688, Package_SO:SOIC-20W_7.5x12.8mm_P1.27mm, F.Cu at (163.0, 109.5)
- added U429: 74HC74, Package_SO:SOIC-14_3.9x8.7mm_P1.27mm, F.Cu at (309.3, 95.4)
- added U430: 74HC193, Package_SO:SOIC-16_3.9x9.9mm_P1.27mm, F.Cu at (129.4, 109.5)
- added U431: 74HC04, Package_SO:SOIC-14_3.9x8.7mm_P1.27mm, F.Cu at (315.9, 141.1)
- added U432: 74HC08, Package_SO:SOIC-14_3.9x8.7mm_P1.27mm, F.Cu at (332.6, 140.9)
- added U433: 74HC74, Package_SO:SOIC-14_3.9x8.7mm_P1.27mm, F.Cu at (140.2, 109.5)
- added U434: 74HC74, Package_SO:SOIC-14_3.9x8.7mm_P1.27mm, F.Cu at (341.1, 140.9)
- added U435: 74HC11, Package_SO:SOIC-14_3.9x8.7mm_P1.27mm, F.Cu at (307.4, 141.1)
- added U436: 74HC00, Package_SO:SOIC-14_3.9x8.7mm_P1.27mm, F.Cu at (324.2, 140.9)

Commit message: TOD is here
Parts:
- added C400: 100n, Capacitor_SMD:C_0603_1608Metric, F.Cu at (190.7, 106.7)
- added C402: 100n, Capacitor_SMD:C_0603_1608Metric, F.Cu at (144.5, 49.8)
- added C403: 100n, Capacitor_SMD:C_0603_1608Metric, F.Cu at (154.6, 49.8)
- added C404: 100n, Capacitor_SMD:C_0603_1608Metric, F.Cu at (168.8, 48.5)
- added C405: 100n, Capacitor_SMD:C_0603_1608Metric, F.Cu at (182.9, 48.5)
- added C406: 100n, Capacitor_SMD:C_0603_1608Metric, F.Cu at (169.7, 111.6)
- added C407: 100n, Capacitor_SMD:C_0603_1608Metric, F.Cu at (168.8, 80.5)
- added C408: 100n, Capacitor_SMD:C_0603_1608Metric, F.Cu at (111.7, 98.0)
- added C409: 100n, Capacitor_SMD:C_0603_1608Metric, F.Cu at (115.1, 75.3)
- added C410: 100n, Capacitor_SMD:C_0603_1608Metric, F.Cu at (143.1, 123.5)
- added C411: 100n, Capacitor_SMD:C_0603_1608Metric, F.Cu at (111.9, 123.5)
- added C412: 100n, Capacitor_SMD:C_0603_1608Metric, F.Cu at (180.7, 111.6)
- added C413: 100n, Capacitor_SMD:C_0603_1608Metric, F.Cu at (144.9, 66.0)
- added C414: 100n, Capacitor_SMD:C_0603_1608Metric, F.Cu at (154.7, 66.0)
- added C416: 100n, Capacitor_SMD:C_0603_1608Metric, F.Cu at (134.0, 95.9)
- added C417: 100n, Capacitor_SMD:C_0603_1608Metric, F.Cu at (144.6, 81.8)
- added C418: 100n, Capacitor_SMD:C_0603_1608Metric, F.Cu at (133.7, 80.5)
- added C419: 100n, Capacitor_SMD:C_0603_1608Metric, F.Cu at (120.5, 123.5)
- added C420: 100n, Capacitor_SMD:C_0603_1608Metric, F.Cu at (133.9, 64.6)
- added C421: 100n, Capacitor_SMD:C_0603_1608Metric, F.Cu at (154.6, 81.7)
- added C422: 100n, Capacitor_SMD:C_0603_1608Metric, F.Cu at (182.9, 80.5)
- added C423: 100n, Capacitor_SMD:C_0603_1608Metric, F.Cu at (128.3, 111.6)
- added C424: 100n, Capacitor_SMD:C_0603_1608Metric, F.Cu at (182.9, 96.0)
- added C426: 100n, Capacitor_SMD:C_0603_1608Metric, F.Cu at (159.2, 123.5)
- added C427: 100n, Capacitor_SMD:C_0603_1608Metric, F.Cu at (116.8, 50.5)
- added C428: 100n, Capacitor_SMD:C_0603_1608Metric, F.Cu at (168.7, 96.0)
- added C429: 100n, Capacitor_SMD:C_0603_1608Metric, F.Cu at (180.3, 123.5)
- added C430: 100n, Capacitor_SMD:C_0603_1608Metric, F.Cu at (140.5, 111.6)
- added C431: 100n, Capacitor_SMD:C_0603_1608Metric, F.Cu at (129.5, 123.5)
- added C432: 100n, Capacitor_SMD:C_0603_1608Metric, F.Cu at (144.7, 97.2)
- added C433: 100n, Capacitor_SMD:C_0603_1608Metric, F.Cu at (154.7, 97.4)
- added C434: 100n, Capacitor_SMD:C_0603_1608Metric, F.Cu at (159.0, 111.6)
- added C435: 100n, Capacitor_SMD:C_0603_1608Metric, F.Cu at (120.4, 98.0)
- added C436: 100n, Capacitor_SMD:C_0603_1608Metric, F.Cu at (168.7, 64.7)
- added C504: 100n, Capacitor_SMD:C_0603_1608Metric, F.Cu at (116.3, 111.6)
- added C505: 100n, Capacitor_SMD:C_0603_1608Metric, F.Cu at (182.9, 64.6)
- added GND101: GND, MountingHole:MountingHole_2.2mm_M2_DIN965_Pad, F.Cu at (103.4, 56.9)
- added GND102: GND, MountingHole:MountingHole_2.2mm_M2_DIN965_Pad, F.Cu at (196.4, 56.9)
- added VCC101: VCC, MountingHole:MountingHole_2.2mm_M2_DIN965_Pad, F.Cu at (103.4, 139.6)
- added VCC102: VCC, MountingHole:MountingHole_2.2mm_M2_DIN965_Pad, F.Cu at (196.4, 139.9)
- moved U415 244.0 mm to (108.3, 103.5)
- moved U418 228.5 mm to (113.1, 80.8)
- moved U432 218.6 mm to (117.3, 103.5)
- moved U431 204.2 mm to (113.1, 117.0)
- moved U498 201.1 mm to (108.6, 129.0)
- moved U436 200.4 mm to (125.2, 117.0)
- moved U497 196.9 mm to (117.5, 129.0)
- moved U414 195.9 mm to (113.4, 56.0)
- moved U434 186.9 mm to (155.7, 117.0)
- moved U406 184.4 mm to (126.3, 129.0)
- moved U505 181.5 mm to (139.9, 129.0)
- moved U411 163.8 mm to (155.9, 129.0)
- moved U503 162.5 mm to (166.6, 117.0)
- moved U435 160.7 mm to (151.4, 102.8)
- moved U504 138.7 mm to (177.4, 117.0)
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- renumbered U407 to U401, U412 to U402, U413 to U403, U425 to U404, U421 to U405, U402 to U497, U401 to U498, U403 to U503, U404 to U504, U405 to U505
Connections:
- C401 pad 1: ~{RES} -> VCC
- U401 pad 12: /todAlarm/ALARM4 -> unconnected-(U401-Pad12)
- U401 pad 13: DZ0 -> GND
- U401 pad 14: DZ1 -> GND
- U401 pad 15: /todAlarm/ALARM5 -> unconnected-(U401-Pad15)
- U401 pad 16: /todAlarm/ALARM6 -> unconnected-(U401-Pad16)
- U401 pad 17: DZ2 -> GND
- U401 pad 18: DZ3 -> GND
- U401 pad 19: /todAlarm/ALARM7 -> unconnected-(U401-Pad19)
- U401 pad 2: /todAlarm/ALARM0 -> /todAlarm/ALARM5
- U401 pad 3: GND -> DZ1
- U401 pad 4: GND -> DZ0
- U401 pad 5: /todAlarm/ALARM1 -> /todAlarm/ALARM4
- U401 pad 6: /todAlarm/ALARM2 -> /todAlarm/ALARM6
- U401 pad 7: GND -> DZ2
- U401 pad 8: GND -> DZ3
- U401 pad 9: /todAlarm/ALARM3 -> /todAlarm/ALARM7
- U402 pad 2: Net-(U412-Pad2) -> /todCounter/todTenths/TODBUS1
- U402 pad 3: Net-(U412-Pad3) -> /todCounter/todTenths/TODBUS0
- U402 pad 6: Net-(U412-Pad6) -> /todCounter/todTenths/TODBUS2
- U404 pad 11: /todComparator/TODBUS4 -> /todComparator/TODBUS7
- U404 pad 12: /todAlarm/ALARM4 -> /todAlarm/ALARM7
- U404 pad 13: /todComparator/TODBUS5 -> /todComparator/TODBUS6
- U404 pad 14: /todAlarm/ALARM5 -> /todAlarm/ALARM6
- U404 pad 15: /todComparator/TODBUS6 -> GND
- U404 pad 16: /todAlarm/ALARM6 -> GND
- U404 pad 17: /todComparator/TODBUS7 -> GND
- U404 pad 18: /todAlarm/ALARM7 -> GND
- U404 pad 2: GND -> /todComparator/TODBUS5
- U404 pad 3: GND -> /todAlarm/ALARM5
- U404 pad 4: GND -> /todComparator/TODBUS4
- U404 pad 5: GND -> /todAlarm/ALARM4
- U405 pad 12: D4 -> D6
- U405 pad 15: D5 -> D4
- U405 pad 16: D6 -> D5
- U405 pad 2: D0 -> D1
- U405 pad 3: /todComparator/TODBUS4 -> /todComparator/TODBUS5
- U405 pad 4: /todComparator/TODBUS5 -> /todComparator/TODBUS4
- U405 pad 5: D1 -> D0
- U406 pad 1: Net-(U401-Pad6) -> Net-(U406-Pad1)
- U406 pad 10: Net-(U403-Pad4) -> /todControl/~{ALARM}
- U406 pad 13: Net-(U403-Pad4) -> /todControl/~{ALARM}
- U406 pad 2: Net-(U403-Pad4) -> /todControl/~{ALARM}
- U406 pad 4: Net-(U401-Pad11) -> Net-(U406-Pad4)
- U406 pad 5: Net-(U403-Pad4) -> /todControl/~{ALARM}
- U406 pad 7: Net-(U401-Pad7) -> GND
- U406 pad 9: Net-(U402-Pad6) -> Net-(U406-Pad9)
- U408 pad 12: /todAlarm/ALARM20 -> /todAlarm/ALARM22
- U408 pad 13: DZ4 -> DZ6
- U408 pad 16: /todAlarm/ALARM22 -> /todAlarm/ALARM20
- U408 pad 17: DZ6 -> DZ4
- U408 pad 19: /todAlarm/ALARM23 -> unconnected-(U408-Pad19)
- U408 pad 2: /todAlarm/ALARM16 -> /todAlarm/ALARM17
- U408 pad 3: DZ0 -> DZ1
- U408 pad 4: DZ1 -> DZ0
- U408 pad 5: /todAlarm/ALARM17 -> /todAlarm/ALARM16
- U409 pad 12: /todAlarm/ALARM12 -> /todAlarm/ALARM14
- U409 pad 13: DZ4 -> DZ6
- U409 pad 16: /todAlarm/ALARM14 -> /todAlarm/ALARM12
- U409 pad 17: DZ6 -> DZ4
- U409 pad 19: /todAlarm/ALARM15 -> unconnected-(U409-Pad19)
- U409 pad 2: /todAlarm/ALARM8 -> /todAlarm/ALARM9
- U409 pad 3: DZ0 -> DZ1
- U409 pad 4: DZ1 -> DZ0
- U409 pad 5: /todAlarm/ALARM9 -> /todAlarm/ALARM8
- U410 pad 12: /todAlarm/ALARM28 -> unconnected-(U410-Pad12)
- U410 pad 13: DZ4 -> GND
- U410 pad 15: /todAlarm/ALARM29 -> unconnected-(U410-Pad15)
- U410 pad 16: /todAlarm/ALARM30 -> /todAlarm/ALARM28
- U410 pad 17: GND -> DZ4
- U410 pad 2: /todAlarm/ALARM24 -> /todAlarm/ALARM25
- U410 pad 3: DZ0 -> DZ1
- U410 pad 4: DZ1 -> DZ0
- U410 pad 5: /todAlarm/ALARM25 -> /todAlarm/ALARM24
- U411 pad 1: TOD -> GND
- U411 pad 10: Net-(U401-Pad7) -> /todControl/COUNT
- U411 pad 12: Net-(U401-Pad7) -> GND
- U411 pad 14: unconnected-(U411-Pad14) -> VCC
- U411 pad 2: /todControl/COUNT -> GND
- U411 pad 3: /todCounter/TICK -> unconnected-(U411-Pad3)
- U411 pad 4: /todComparator/TODBUS5 -> GND
- U411 pad 5: /todComparator/TODBUS7 -> GND
- U411 pad 6: /todCounter/todSeconds/SEC_TK -> unconnected-(U411-Pad6)
- U411 pad 7: Net-(U401-Pad7) -> GND
- U411 pad 8: unconnected-(U411-Pad8) -> /todCounter/TICK
- U411 pad 9: Net-(U401-Pad7) -> TOD
- U414 pad 10: Net-(U401-Pad7) -> /todCounter/todTenths/TODBUS0
- U414 pad 11: Net-(U401-Pad7) -> TODIN
- U414 pad 13: Net-(U412-Pad6) -> /todCounter/todTenths/TODBUS1
- U414 pad 2: Net-(U412-Pad2) -> /todCounter/todTenths/TODBUS2
- U414 pad 3: Net-(U412-Pad6) -> /todComparator/TODBUS5
- U414 pad 4: Net-(U412-Pad3) -> /todComparator/TODBUS5
- U414 pad 5: TODIN -> /todComparator/TODBUS7
- U414 pad 6: Net-(U414-Pad6) -> /todCounter/todSeconds/SEC_TK
- U414 pad 7: Net-(U401-Pad7) -> GND
- U414 pad 8: unconnected-(U414-Pad8) -> Net-(U414-Pad8)
- U414 pad 9: Net-(U401-Pad7) -> /todCounter/todTenths/TODBUS2
- U415 pad 10: DZ0 -> Net-(U415-Pad10)
- U415 pad 11: /todCounter/todHours/H4_FLIP -> Net-(U415-Pad11)
- U415 pad 12: Net-(U430-Pad14) -> Net-(U415-Pad12)
- U415 pad 13: Net-(U435-Pad6) -> DZ0
- U415 pad 2: Net-(U414-Pad6) -> Net-(U414-Pad8)
- U415 pad 4: Net-(U431-Pad2) -> /todControl/~{LOADH}
- U415 pad 5: /todControl/~{LOADH} -> Net-(U415-Pad5)
- U415 pad 6: Net-(U415-Pad6) -> Net-(U415-Pad12)
- U415 pad 8: Net-(U415-Pad8) -> /todCounter/todHours/H4_FLIP
- U415 pad 9: Net-(U415-Pad6) -> Net-(U415-Pad9)
- U418 pad 1: /todComparator/TODBUS9 -> /todComparator/TODBUS13
- U418 pad 10: /todComparator/TODBUS19 -> /todComparator/TODBUS21
- U418 pad 11: /todCounter/todHours/HOU_TK -> Net-(U416-Pad14)
- U418 pad 12: /todComparator/TODBUS21 -> /todComparator/TODBUS11
- U418 pad 13: /todComparator/TODBUS22 -> /todComparator/TODBUS9
- U418 pad 2: /todComparator/TODBUS11 -> /todComparator/TODBUS14
- U418 pad 3: Net-(U416-Pad14) -> /todCounter/todMinutes/MIN_TK
- U418 pad 4: /todComparator/TODBUS13 -> /todComparator/TODBUS17
- U418 pad 5: /todComparator/TODBUS14 -> /todComparator/TODBUS19
- U418 pad 6: /todCounter/todMinutes/MIN_TK -> Net-(U418-Pad6)
- U418 pad 7: Net-(U401-Pad7) -> GND
- U418 pad 8: Net-(U418-Pad8) -> /todCounter/todHours/HOU_TK
- U418 pad 9: /todComparator/TODBUS17 -> /todComparator/TODBUS22
- U419 pad 14: Net-(U418-Pad8) -> Net-(U418-Pad6)
- U420 pad 5: Net-(U418-Pad8) -> Net-(U418-Pad6)
- U422 pad 12: D4 -> D6
- U422 pad 13: /todComparator/TODBUS20 -> /todComparator/TODBUS22
- U422 pad 14: /todComparator/TODBUS21 -> /todComparator/TODBUS20
- U422 pad 15: D5 -> D4
- U422 pad 16: D6 -> D5
- U422 pad 17: /todComparator/TODBUS22 -> /todComparator/TODBUS21
- U422 pad 2: D0 -> D1
- U422 pad 3: /todComparator/TODBUS16 -> /todComparator/TODBUS17
- U422 pad 4: /todComparator/TODBUS17 -> /todComparator/TODBUS16
- U422 pad 5: D1 -> D0
- U423 pad 12: D4 -> D6
- U423 pad 13: /todComparator/TODBUS12 -> /todComparator/TODBUS14
- U423 pad 14: /todComparator/TODBUS13 -> /todComparator/TODBUS12
- U423 pad 15: D5 -> D4
- U423 pad 16: D6 -> D5
- U423 pad 17: /todComparator/TODBUS14 -> /todComparator/TODBUS13
- U423 pad 2: D0 -> D1
- U423 pad 3: /todComparator/TODBUS8 -> /todComparator/TODBUS9
- U423 pad 4: /todComparator/TODBUS9 -> /todComparator/TODBUS8
- U423 pad 5: D1 -> D0
- U424 pad 12: D4 -> D6
- U424 pad 13: /todComparator/TODBUS28 -> GND
- U424 pad 14: GND -> /todComparator/TODBUS28
- U424 pad 15: D5 -> D4
- U424 pad 16: D6 -> D5
- U424 pad 2: D0 -> D1
- U424 pad 3: /todComparator/TODBUS24 -> /todComparator/TODBUS25
- U424 pad 4: /todComparator/TODBUS25 -> /todComparator/TODBUS24
- U424 pad 5: D1 -> D0
- U426 pad 11: /todComparator/TODBUS12 -> /todComparator/TODBUS11
- U426 pad 12: /todAlarm/ALARM12 -> /todAlarm/ALARM11
- U426 pad 13: /todComparator/TODBUS13 -> /todComparator/TODBUS10
- U426 pad 14: /todAlarm/ALARM13 -> /todAlarm/ALARM10
- U426 pad 15: /todComparator/TODBUS14 -> /todComparator/TODBUS12
- U426 pad 16: /todAlarm/ALARM14 -> /todAlarm/ALARM12
- U426 pad 2: /todComparator/TODBUS8 -> /todComparator/TODBUS9
- U426 pad 3: /todAlarm/ALARM8 -> /todAlarm/ALARM9
- U426 pad 4: /todComparator/TODBUS9 -> /todComparator/TODBUS8
- U426 pad 5: /todAlarm/ALARM9 -> /todAlarm/ALARM8
- U426 pad 6: /todComparator/TODBUS10 -> /todComparator/TODBUS13
- U426 pad 7: /todAlarm/ALARM10 -> /todAlarm/ALARM13
- U426 pad 8: /todComparator/TODBUS11 -> /todComparator/TODBUS14
- U426 pad 9: /todAlarm/ALARM11 -> /todAlarm/ALARM14
- U427 pad 11: /todComparator/TODBUS20 -> /todComparator/TODBUS19
- U427 pad 12: /todAlarm/ALARM20 -> /todAlarm/ALARM19
- U427 pad 13: /todComparator/TODBUS21 -> /todComparator/TODBUS18
- U427 pad 14: /todAlarm/ALARM21 -> /todAlarm/ALARM18
- U427 pad 15: /todComparator/TODBUS22 -> /todComparator/TODBUS20
- U427 pad 16: /todAlarm/ALARM22 -> /todAlarm/ALARM20
- U427 pad 2: /todComparator/TODBUS16 -> /todComparator/TODBUS17
- U427 pad 3: /todAlarm/ALARM16 -> /todAlarm/ALARM17
- U427 pad 4: /todComparator/TODBUS17 -> /todComparator/TODBUS16
- U427 pad 5: /todAlarm/ALARM17 -> /todAlarm/ALARM16
- U427 pad 6: /todComparator/TODBUS18 -> /todComparator/TODBUS21
- U427 pad 7: /todAlarm/ALARM18 -> /todAlarm/ALARM21
- U427 pad 8: /todComparator/TODBUS19 -> /todComparator/TODBUS22
- U427 pad 9: /todAlarm/ALARM19 -> /todAlarm/ALARM22
- U428 pad 11: /todComparator/TODBUS28 -> /todComparator/TODBUS27
- U428 pad 12: /todAlarm/ALARM28 -> /todAlarm/ALARM27
- U428 pad 13: /todComparator/TODBUS31 -> /todComparator/TODBUS26
- U428 pad 14: /todAlarm/ALARM31 -> /todAlarm/ALARM26
- U428 pad 15: GND -> /todComparator/TODBUS28
- U428 pad 16: GND -> /todAlarm/ALARM28
- U428 pad 17: GND -> /todComparator/TODBUS31
- U428 pad 18: GND -> /todAlarm/ALARM31
- U428 pad 19: Net-(U403-Pad9) -> Net-(U428-Pad19)
- U428 pad 2: /todComparator/TODBUS24 -> /todComparator/TODBUS25
- U428 pad 3: /todAlarm/ALARM24 -> /todAlarm/ALARM25
- U428 pad 4: /todComparator/TODBUS25 -> /todComparator/TODBUS24
- U428 pad 5: /todAlarm/ALARM25 -> /todAlarm/ALARM24
- U428 pad 6: /todComparator/TODBUS26 -> GND
- U428 pad 7: /todAlarm/ALARM26 -> GND
- U428 pad 8: /todComparator/TODBUS27 -> GND
- U428 pad 9: /todAlarm/ALARM27 -> GND
- U429 pad 7: Net-(U401-Pad7) -> GND
- U430 pad 14: Net-(U430-Pad14) -> Net-(U415-Pad9)
- U430 pad 15: Net-(U415-Pad8) -> Net-(U415-Pad11)
- U431 pad 13: Net-(U435-Pad6) -> Net-(U415-Pad10)
- U431 pad 2: Net-(U431-Pad2) -> Net-(U415-Pad5)
- U431 pad 3: Net-(U415-Pad6) -> Net-(U415-Pad12)
- U431 pad 7: Net-(U401-Pad7) -> GND
- U432 pad 4: Net-(U431-Pad4) -> DZ2
- U432 pad 5: DZ2 -> Net-(U431-Pad4)
- U432 pad 7: Net-(U401-Pad7) -> GND
- U433 pad 1: Net-(U436-Pad6) -> Net-(U433-Pad1)
- U433 pad 4: Net-(U436-Pad3) -> Net-(U433-Pad4)
- U433 pad 7: Net-(U401-Pad7) -> GND
- U434 pad 13: Net-(U403-Pad12) -> Net-(U434-Pad13)
- U434 pad 7: Net-(U401-Pad7) -> GND
- U435 pad 12: Net-(U430-Pad14) -> Net-(U415-Pad9)
- U435 pad 6: Net-(U435-Pad6) -> Net-(U415-Pad10)
- U436 pad 10: DZ7 -> Net-(U431-Pad4)
- U436 pad 12: Net-(U431-Pad4) -> Net-(U431-Pad8)
- U436 pad 13: Net-(U431-Pad8) -> Net-(U431-Pad4)
- U436 pad 2: DZ4 -> Net-(U431-Pad6)
- U436 pad 3: Net-(U436-Pad3) -> Net-(U433-Pad1)
- U436 pad 5: Net-(U431-Pad6) -> DZ4
- U436 pad 6: Net-(U436-Pad6) -> Net-(U433-Pad4)
- U436 pad 9: Net-(U431-Pad4) -> DZ7
- U497 pad 1: ~{RES} -> Net-(U497-Pad1)
- U497 pad 10: ~{EN11} -> ENABLE_NAND
- U497 pad 12: Net-(U402-Pad12) -> Net-(U497-Pad12)
- U497 pad 2: ~{EN10} -> ENABLE_NAND
- U497 pad 3: Net-(U402-Pad3) -> Net-(U406-Pad1)
- U497 pad 4: Net-(U402-Pad3) -> Net-(U497-Pad4)
- U497 pad 6: Net-(U402-Pad6) -> Net-(U406-Pad4)
- U497 pad 8: Net-(U402-Pad12) -> Net-(U406-Pad9)
- U497 pad 9: ~{RES} -> Net-(U497-Pad9)
- U498 pad 1: ~{RES} -> ~{EN8}
- U498 pad 10: ~{EN9} -> ~{RES}
- U498 pad 11: Net-(U401-Pad11) -> Net-(U497-Pad12)
- U498 pad 12: Net-(U401-Pad12) -> ~{RES}
- U498 pad 13: ENABLE_NAND -> ~{EN11}
- U498 pad 2: ~{EN8} -> ~{RES}
- U498 pad 3: Net-(U401-Pad3) -> Net-(U497-Pad1)
- U498 pad 4: Net-(U401-Pad3) -> ~{RES}
- U498 pad 5: ENABLE_NAND -> ~{EN9}
- U498 pad 6: Net-(U401-Pad6) -> Net-(U497-Pad4)
- U498 pad 7: Net-(U401-Pad7) -> GND
- U498 pad 8: Net-(U401-Pad12) -> Net-(U497-Pad9)
- U498 pad 9: ~{RES} -> ~{EN10}
- U503 pad 1: PHI2 -> GND
- U503 pad 10: unconnected-(U403-Pad10) -> /todControl/~{ALARM}
- U503 pad 11: Net-(U401-Pad7) -> ALARM
- U503 pad 12: Net-(U403-Pad12) -> TODIRQ
- U503 pad 13: Net-(U435-Pad8) -> Net-(U428-Pad19)
- U503 pad 2: /~{PHI2} -> unconnected-(U503-Pad2)
- U503 pad 3: ALARM -> Net-(U435-Pad8)
- U503 pad 4: Net-(U403-Pad4) -> Net-(U434-Pad13)
- U503 pad 8: TODIRQ -> /~{PHI2}
- U503 pad 9: Net-(U403-Pad9) -> PHI2
- U504 pad 7: Net-(U401-Pad7) -> GND
- U505 pad 1: Net-(U401-Pad6) -> Net-(U406-Pad1)
- U505 pad 4: Net-(U401-Pad11) -> Net-(U406-Pad4)
- U505 pad 7: Net-(U401-Pad7) -> GND
- U505 pad 9: Net-(U402-Pad6) -> Net-(U406-Pad9)
Routing:
- net VCC: track 0.00 -> 815.0 mm, vias 0 -> 9
- net DZ0: track 0.00 -> 236.6 mm, vias 0 -> 9
- net DZ2: track 0.00 -> 235.7 mm, vias 0 -> 9
- net DZ3: track 0.00 -> 232.9 mm, vias 0 -> 9
- net DZ1: track 0.00 -> 229.5 mm, vias 0 -> 9
- net DZ4: track 0.00 -> 223.2 mm, vias 0 -> 5
- net ~{RES}: track 0.00 -> 219.4 mm, vias 0 -> 2
- net DZ7: track 0.00 -> 194.1 mm, vias 0 -> 3
- net ENABLE_NAND: track 0.00 -> 173.3 mm, vias 0 -> 2
- net DZ6: track 0.00 -> 165.7 mm, vias 0 -> 3
- net DZ5: track 0.00 -> 157.9 mm, vias 0 -> 5
- net TODIN: track 0.00 -> 138.1 mm, vias 0 -> 2
- net GND: track 0.00 -> 133.7 mm, vias 4 -> 88
- net /todControl/~{LOADT}: track 0.00 -> 123.5 mm, vias 0 -> 2
- net Net-(U414-Pad1): track 0.00 -> 120.6 mm, vias 0 -> 2
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
Commit message: Ready for v0.2.2
Parts:
- U435: renamed from U411; value 74HC08 -> 74HCT08
- renumbered U414 to U401, U401 to U402, U402 to U403, U403 to U404, U404 to U405, U405 to U406, U418 to U407, U409 to U408, U417 to U409, U416 to U410, U426 to U411, U423 to U412, U408 to U413, U420 to U414, U419 to U415, U427 to U416, U422 to U417, U415 to U418, U432 to U419, U410 to U420, U430 to U421, U435 to U422, U428 to U423, U431 to U425, U436 to U426, U433 to U427, U434 to U428, U503 to U429, U504 to U430, U498 to U431, U497 to U432, U406 to U433, U505 to U434, U429 to U436
Routing:
- net GND: track 133.7 -> 151.8 mm, vias 88 -> 85
- net /todComparator/TODBUS19: track 77.9 -> 71.5 mm
- net /todControl/~{ALARM}: track 60.7 -> 57.9 mm
- net D1: track 102.3 -> 99.6 mm
- net D3: track 100.3 -> 98.0 mm
- net D2: track 95.0 -> 92.7 mm
- net D0: track 107.4 -> 105.5 mm
- net /todControl/~{OEH}: track 33.4 -> 34.2 mm
Other:
- board text added: "74HCT6526 Board 4 v0.2.2"
