File: B4/buses.kicad_sch (KiCad schematic)
At the start: 3 parts

Commit message: B1 CREGA added
Work started on b1. CREGA added.
Minor changes to B0 schematic properties.
Connections:
- net ~EN10 renamed ~{EN10}
- net ~EN11 renamed ~{EN11}
- net ~EN12 renamed ~{EN12}
- net ~EN13 renamed ~{EN13}
- net ~EN14 renamed ~{EN14}
- net ~EN15 renamed ~{EN15}
- net ~EN4 renamed ~{EN4}
- net ~EN5 renamed ~{EN5}
- net ~EN6 renamed ~{EN6}
- net ~EN7 renamed ~{EN7}
- net ~EN8 renamed ~{EN8}
- net ~EN9 renamed ~{EN9}
- net ~FLAG renamed ~{FLAG}
- net ~IRQ renamed ~{IRQ}
- net ~RES renamed ~{RES}

Commit message: .
Parts:
- renumbered CONTROLBUS1 to CONTROLBUS4, DATABUS1 to DATABUS4, ENABLEBUS1 to ENABLEBUS4
Changed lines of the file:
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@@
   (symbol (lib_id "Connector_Generic:Conn_02x10_Odd_Even") (at 104.14 78.74 0) (unit 1)
     (in_bom yes) (on_board yes)
-    (property "Reference" "ENABLEBUS1" (id 0) (at 105.41 63.1 0))
+    (property "Reference" "ENABLEBUS4" (id 0) (at 105.41 63.1 0))
     (property "Value" "Conn_02x10_Odd_Even" (id 1) (at 105.41 65.3985 0))
     (property "Footprint" "Connector_PinHeader_2.54mm:PinHeader_2x10_P2.54mm_Vertical" (id 2) (at 104.14 78.74 0)
@@
   (symbol (lib_id "Connector_Generic:Conn_02x10_Odd_Even") (at 157.48 78.74 0) (unit 1)
     (in_bom yes) (on_board yes)
-    (property "Reference" "DATABUS1" (id 0) (at 158.75 63.1 0))
+    (property "Reference" "DATABUS4" (id 0) (at 158.75 63.1 0))
     (property "Value" "Conn_02x10_Odd_Even" (id 1) (at 158.75 65.3985 0))
     (property "Footprint" "Connector_PinHeader_2.54mm:PinHeader_2x10_P2.54mm_Vertical" (id 2) (at 157.48 78.74 0)
@@
   (symbol (lib_id "Connector_Generic:Conn_02x10_Odd_Even") (at 231.14 78.74 0) (unit 1)
     (in_bom yes) (on_board yes)
-    (property "Reference" "CONTROLBUS1" (id 0) (at 232.41 63.1 0))
+    (property "Reference" "CONTROLBUS4" (id 0) (at 232.41 63.1 0))
     (property "Value" "Conn_02x10_Odd_Even" (id 1) (at 232.41 65.3985 0))
     (property "Footprint" "Connector_PinHeader_2.54mm:PinHeader_2x10_P2.54mm_Vertical" (id 2) (at 231.14 78.74 0)

Commit message: B0 ready for v0.2.0 release.
Parts:
- added C400: 100n, symbol Device:C
Connections:
- net GND: now also C400.2
- net ~{RES}: now also C400.1
- net TARUNMODE: no longer names the net of CONTROLBUS4.18 (Pin_18)
Other:
- company: (none) -> Daniel Molina
- title: (none) -> 74HCT6526 Board 4
Changed lines of the file:
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@@
 (kicad_sch (version 20211123) (generator eeschema)
   (paper "A4")
+  (title_block
+    (title "74HCT6526 Board 4")
+    (date "2023-01-22")
+    (rev "0.2.0")
+    (company "Daniel Molina")
+    (comment 1 "https://github.com/dmolinagarcia/74HCT6526")
+  )
   (junction (at 208.28 33.02) (diameter 1.016) (color 0 0 0 0)
   )
@@
   (junction (at 165.1 78.74) (diameter 1.016) (color 0 0 0 0)
   )
+  (junction (at 134.62 101.6) (diameter 0) (color 0 0 0 0)
+  )
   (junction (at 111.76 86.36) (diameter 1.016) (color 0 0 0 0)
   )
   (junction (at 78.74 38.1) (diameter 1.016) (color 0 0 0 0)
   )
+  (junction (at 246.38 91.44) (diameter 0) (color 0 0 0 0)
+  )
   (junction (at 111.76 88.9) (diameter 1.016) (color 0 0 0 0)
   )
@@
     (stroke (width 0.1524) (type solid) (color 0 0 0 0))
   )
-  (bus_entry (at 259.08 86.36) (size -2.54 2.54)
-    (stroke (width 0.1524) (type solid) (color 0 0 0 0))
-  )
   (bus_entry (at 134.62 66.04) (size 2.54 2.54)
     (stroke (width 0.1524) (type solid) (color 0 0 0 0))
@@
     (stroke (width 0) (type solid) (color 0 0 0 0))
   )
-  (wire (pts (xy 238.76 91.44) (xy 256.54 91.44))
+  (wire (pts (xy 238.76 91.44) (xy 246.38 91.44))
     (stroke (width 0) (type solid) (color 0 0 0 0))
   )
@@
     (stroke (width 0) (type solid) (color 0 0 0 0))
   )
+  (bus (pts (xy 134.62 101.6) (xy 180.34 101.6))
+    (stroke (width 0) (type default) (color 0 0 0 0))
+  )
   (wire (pts (xy 111.76 73.66) (xy 111.76 76.2))
     (stroke (width 0) (type solid) (color 0 0 0 0))
@@
     (stroke (width 0) (type solid) (color 0 0 0 0))
   )
-  (bus (pts (xy 259.08 86.36) (xy 259.08 88.9))
+  (bus (pts (xy 259.08 83.82) (xy 259.08 88.9))
     (stroke (width 0) (type solid) (color 0 0 0 0))
   )
@@
     (stroke (width 0) (type solid) (color 0 0 0 0))
   )
-  (wire (pts (xy 238.76 88.9) (xy 256.54 88.9))
-    (stroke (width 0) (type solid) (color 0 0 0 0))
-  )
   (bus (pts (xy 180.34 81.28) (xy 180.34 83.82))
     (stroke (width 0) (type solid) (color 0 0 0 0))
@@
     (stroke (width 0) (type solid) (color 0 0 0 0))
   )
+  (wire (pts (xy 246.38 91.44) (xy 256.54 91.44))
+    (stroke (width 0) (type solid) (color 0 0 0 0))
+  )
   (wire (pts (xy 137.16 71.12) (xy 152.4 71.12))
     (stroke (width 0) (type solid) (color 0 0 0 0))
@@
     (stroke (width 0) (type solid) (color 0 0 0 0))
   )
-  (bus (pts (xy 134.62 73.66) (xy 134.62 81.28))
-    (stroke (width 0) (type solid) (color 0 0 0 0))
-  )
   (bus (pts (xy 208.28 73.66) (xy 208.28 76.2))
     (stroke (width 0) (type solid) (color 0 0 0 0))
@@
     (stroke (width 0) (type solid) (color 0 0 0 0))
   )
+  (bus (pts (xy 27.94 101.6) (xy 134.62 101.6))
+    (stroke (width 0) (type default) (color 0 0 0 0))
+  )
+  (bus (pts (xy 134.62 88.9) (xy 134.62 101.6))
+    (stroke (width 0) (type default) (color 0 0 0 0))
+  )
   (wire (pts (xy 111.76 71.12) (xy 129.54 71.12))
     (stroke (width 0) (type solid) (color 0 0 0 0))
@@
     (stroke (width 0) (type solid) (color 0 0 0 0))
   )
+  (bus (pts (xy 180.34 101.6) (xy 180.34 88.9))
+    (stroke (width 0) (type default) (color 0 0 0 0))
+  )
   (bus (pts (xy 259.08 78.74) (xy 259.08 81.28))
     (stroke (width 0) (type solid) (color 0 0 0 0))
   )
-  (bus (pts (xy 180.34 73.66) (xy 180.34 81.28))
-    (stroke (width 0) (type solid) (color 0 0 0 0))
-  )
   (bus (pts (xy 208.28 78.74) (xy 208.28 81.28))
     (stroke (width 0) (type solid) (color 0 0 0 0))
@@
     (stroke (width 0) (type solid) (color 0 0 0 0))
   )
-  (bus (pts (xy 259.08 83.82) (xy 259.08 86.36))
-    (stroke (width 0) (type solid) (color 0 0 0 0))
-  )
   (bus (pts (xy 259.08 76.2) (xy 259.08 78.74))
     (stroke (width 0) (type solid) (color 0 0 0 0))
@@
     (effects (font (size 1.27 1.27)) (justify right bottom))
   )
-  (label "TARUNMODE" (at 251.46 88.9 180)
-    (effects (font (size 1.27 1.27)) (justify right bottom))
-  )
   (label "PHI2" (at 223.52 76.2 180)
     (effects (font (size 1.27 1.27)) (justify right bottom))
@@
     (effects (font (size 1.27 1.27)) (justify right bottom))
   )
-  (label "{DATABUS}" (at 180.34 35.56 180)
-    (effects (font (size 1.27 1.27)) (justify right bottom))
-  )
   (label "{ENABLEBUS}" (at 132.08 38.1 180)
     (effects (font (size 1.27 1.27)) (justify right bottom))
@@
     (effects (font (size 1.27 1.27)) (justify right bottom))
   )
-  (hierarchical_label "{ENABLEBUS}" (shape input) (at 27.94 38.1 180)
+  (hierarchical_label "~{EN[0..15]}" (shape input) (at 27.94 38.1 180)
+    (effects (font (size 1.27 1.27)) (justify right))
+  )
+  (hierarchical_label "DZ[0..7]" (shape bidirectional) (at 27.94 101.6 180)
     (effects (font (size 1.27 1.27)) (justify right))
   )
@@
     (effects (font (size 1.27 1.27)) (justify right))
   )
-  (hierarchical_label "{DATABUS}" (shape bidirectional) (at 27.94 35.56 180)
+  (hierarchical_label "D[0..7]" (shape bidirectional) (at 27.94 35.56 180)
     (effects (font (size 1.27 1.27)) (justify right))
   )
@@
     (pin "9")
   )
+  (symbol (lib_id "power:GND") (at 246.38 99.06 0) (unit 1)
+    (in_bom yes) (on_board yes) (fields_autoplaced)
+    (property "Reference" "#PWR?" (id 0) (at 246.38 105.41 0)
+      (effects (font (size 1.27 1.27)) hide)
+    )
+    (property "Value" "GND" (id 1) (at 246.38 104.14 0))
+    (property "Footprint" "" (id 2) (at 246.38 99.06 0)
+      (effects (font (size 1.27 1.27)) hide)
+    )
+    (property "Datasheet" "" (id 3) (at 246.38 99.06 0)
+      (effects (font (size 1.27 1.27)) hide)
+    )
+    (pin "1")
+  )
+  (symbol (lib_id "Device:C") (at 246.38 95.25 0) (unit 1)
+    (in_bom yes) (on_board yes) (fields_autoplaced)
+    (property "Reference" "C400" (id 0) (at 250.19 93.9799 0)
+      (effects (font (size 1.27 1.27)) (justify left))
+    )
+    (property "Value" "100n" (id 1) (at 250.19 96.5199 0)
+      (effects (font (size 1.27 1.27)) (justify left))
+    )
+    (property "Footprint" "" (id 2) (at 247.3452 99.06 0)
+      (effects (font (size 1.27 1.27)) hide)
+    )
+    (property "Datasheet" "~" (id 3) (at 246.38 95.25 0)
+      (effects (font (size 1.27 1.27)) hide)
+    )
+    (pin "1")
+    (pin "2")
+  )
   (symbol (lib_id "Connector_Generic:Conn_02x10_Odd_Even") (at 157.48 78.74 0) (unit 1)

Commit message: Ready for v0.2.1
Parts:
- C401: renamed from C400; footprint (none) -> Capacitor_SMD:C_0603_1608Metric
- renumbered CONTROLBUS4 to CONTROLBUS401, DATABUS4 to DATABUS401, ENABLEBUS4 to ENABLEBUS401
Connections:
- no-connect marks 0 -> 1
Changed lines of the file:
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@@
   (junction (at 152.4 81.28) (diameter 1.016) (color 0 0 0 0)
   )
+  (no_connect (at 238.76 88.9))
   (bus_entry (at 78.74 83.82) (size 2.54 2.54)
     (stroke (width 0.1524) (type solid) (color 0 0 0 0))
@@
     (effects (font (size 1.27 1.27)) (justify right bottom))
   )
-  (label "{ENABLEBUS}" (at 132.08 38.1 180)
-    (effects (font (size 1.27 1.27)) (justify right bottom))
-  )
   (label "TBOUT" (at 251.46 76.2 180)
     (effects (font (size 1.27 1.27)) (justify right bottom))
@@
   (symbol (lib_id "Connector_Generic:Conn_02x10_Odd_Even") (at 104.14 78.74 0) (unit 1)
     (in_bom yes) (on_board yes)
-    (property "Reference" "ENABLEBUS4" (id 0) (at 105.41 63.1 0))
+    (property "Reference" "ENABLEBUS401" (id 0) (at 105.41 63.1 0))
     (property "Value" "Conn_02x10_Odd_Even" (id 1) (at 105.41 65.3985 0))
     (property "Footprint" "Connector_PinHeader_2.54mm:PinHeader_2x10_P2.54mm_Vertical" (id 2) (at 104.14 78.74 0)
@@
   (symbol (lib_id "power:GND") (at 246.38 99.06 0) (unit 1)
     (in_bom yes) (on_board yes) (fields_autoplaced)
-    (property "Reference" "#PWR?" (id 0) (at 246.38 105.41 0)
+    (property "Reference" "#PWR0405" (id 0) (at 246.38 105.41 0)
       (effects (font (size 1.27 1.27)) hide)
     )
@@
   (symbol (lib_id "Device:C") (at 246.38 95.25 0) (unit 1)
     (in_bom yes) (on_board yes) (fields_autoplaced)
-    (property "Reference" "C400" (id 0) (at 250.19 93.9799 0)
+    (property "Reference" "C401" (id 0) (at 250.19 93.9799 0)
       (effects (font (size 1.27 1.27)) (justify left))
     )
@@
       (effects (font (size 1.27 1.27)) (justify left))
     )
-    (property "Footprint" "" (id 2) (at 247.3452 99.06 0)
+    (property "Footprint" "Capacitor_SMD:C_0603_1608Metric" (id 2) (at 247.3452 99.06 0)
       (effects (font (size 1.27 1.27)) hide)
     )
@@
   (symbol (lib_id "Connector_Generic:Conn_02x10_Odd_Even") (at 157.48 78.74 0) (unit 1)
     (in_bom yes) (on_board yes)
-    (property "Reference" "DATABUS4" (id 0) (at 158.75 63.1 0))
+    (property "Reference" "DATABUS401" (id 0) (at 158.75 63.1 0))
     (property "Value" "Conn_02x10_Odd_Even" (id 1) (at 158.75 65.3985 0))
     (property "Footprint" "Connector_PinHeader_2.54mm:PinHeader_2x10_P2.54mm_Vertical" (id 2) (at 157.48 78.74 0)
@@
   (symbol (lib_id "power:GND") (at 173.99 78.74 0) (unit 1)
     (in_bom yes) (on_board yes)
-    (property "Reference" "#PWR04" (id 0) (at 173.99 85.09 0)
+    (property "Reference" "#PWR0404" (id 0) (at 173.99 85.09 0)
       (effects (font (size 1.27 1.27)) hide)
     )
@@
   (symbol (lib_id "power:GND") (at 118.11 83.82 0) (unit 1)
     (in_bom yes) (on_board yes)
-    (property "Reference" "#PWR02" (id 0) (at 118.11 90.17 0)
+    (property "Reference" "#PWR0402" (id 0) (at 118.11 90.17 0)
       (effects (font (size 1.27 1.27)) hide)
     )
@@
   (symbol (lib_id "power:VCC") (at 143.51 81.28 0) (unit 1)
     (in_bom yes) (on_board yes)
-    (property "Reference" "#PWR03" (id 0) (at 143.51 85.09 0)
+    (property "Reference" "#PWR0403" (id 0) (at 143.51 85.09 0)
       (effects (font (size 1.27 1.27)) hide)
     )
@@
   (symbol (lib_id "Connector_Generic:Conn_02x10_Odd_Even") (at 231.14 78.74 0) (unit 1)
     (in_bom yes) (on_board yes)
-    (property "Reference" "CONTROLBUS4" (id 0) (at 232.41 63.1 0))
+    (property "Reference" "CONTROLBUS401" (id 0) (at 232.41 63.1 0))
     (property "Value" "Conn_02x10_Odd_Even" (id 1) (at 232.41 65.3985 0))
     (property "Footprint" "Connector_PinHeader_2.54mm:PinHeader_2x10_P2.54mm_Vertical" (id 2) (at 231.14 78.74 0)
@@
   (symbol (lib_id "power:VCC") (at 118.11 81.28 0) (unit 1)
     (in_bom yes) (on_board yes)
-    (property "Reference" "#PWR01" (id 0) (at 118.11 85.09 0)
-      (effects (font (size 1.27 1.27)) hide)
-    )
+    (property "Reference" "#PWR0401" (id 0) (at 118.11 85.09 0)
+      (effects (font (size 1.27 1.27)) hide)
+    )

Commit message: B2 refactored. B4 Added. TOD sch completed.
Parts:
- renumbered CONTROLBUS401 to CONTROLBUS4, DATABUS401 to DATABUS4, ENABLEBUS401 to ENABLEBUS4
Changed lines of the file:
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@@
   (symbol (lib_id "Connector_Generic:Conn_02x10_Odd_Even") (at 104.14 78.74 0) (unit 1)
     (in_bom yes) (on_board yes)
-    (property "Reference" "ENABLEBUS401" (id 0) (at 105.41 63.1 0))
+    (property "Reference" "ENABLEBUS4" (id 0) (at 105.41 63.1 0))
     (property "Value" "Conn_02x10_Odd_Even" (id 1) (at 105.41 65.3985 0))
     (property "Footprint" "Connector_PinHeader_2.54mm:PinHeader_2x10_P2.54mm_Vertical" (id 2) (at 104.14 78.74 0)
@@
   (symbol (lib_id "Connector_Generic:Conn_02x10_Odd_Even") (at 157.48 78.74 0) (unit 1)
     (in_bom yes) (on_board yes)
-    (property "Reference" "DATABUS401" (id 0) (at 158.75 63.1 0))
+    (property "Reference" "DATABUS4" (id 0) (at 158.75 63.1 0))
     (property "Value" "Conn_02x10_Odd_Even" (id 1) (at 158.75 65.3985 0))
     (property "Footprint" "Connector_PinHeader_2.54mm:PinHeader_2x10_P2.54mm_Vertical" (id 2) (at 157.48 78.74 0)
@@
   (symbol (lib_id "Connector_Generic:Conn_02x10_Odd_Even") (at 231.14 78.74 0) (unit 1)
     (in_bom yes) (on_board yes)
-    (property "Reference" "CONTROLBUS401" (id 0) (at 232.41 63.1 0))
+    (property "Reference" "CONTROLBUS4" (id 0) (at 232.41 63.1 0))
     (property "Value" "Conn_02x10_Odd_Even" (id 1) (at 232.41 65.3985 0))
     (property "Footprint" "Connector_PinHeader_2.54mm:PinHeader_2x10_P2.54mm_Vertical" (id 2) (at 231.14 78.74 0)

Commit message: TOD is here
Parts:
- renumbered C401 to C400
Changed lines of the file:
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@@
   (symbol (lib_id "Device:C") (at 246.38 95.25 0) (unit 1)
     (in_bom yes) (on_board yes) (fields_autoplaced)
-    (property "Reference" "C401" (id 0) (at 250.19 93.9799 0)
+    (property "Reference" "C400" (id 0) (at 250.19 93.9799 0)
       (effects (font (size 1.27 1.27)) (justify left))
     )
