File: B4/todControl.kicad_sch (KiCad schematic)
At the start: 6 parts, among them U401 74HC00, U402 74HC00, U403 74HC04, U404 74HC32, U405 74HC32, U406 74HC32

Commit message: B2 refactored. B4 Added. TOD sch completed.
Parts:
- added U429: 74HC74, Package_SO:SOIC-14_3.9x8.7mm_P1.27mm, symbol 74xx:74HC74
- U401, U402, U404, U405, U406: footprint (none) -> Package_SO:SOIC-14_3.9x8.7mm_P1.27mm
Connections:
- net COUNT: now also U429.5 (Q)
- net LATCH: now also U429.9 (Q)
- net ~{LOADH}: now also U429.1 (~{R})
- net ~{LOADT}: now also U429.4 (~{S})
- net ~{OEH}: now also U429.13 (~{R})
- net ~{OET}: now also U429.10 (~{S})
- net ~{RES}: now also U429.11 (C), U429.3 (C)
- new net GND: U429.2 (D)
- new net VCC: U429.12 (D)
- no-connect marks 0 -> 2
Other:
- moved on the sheet: U401A, U401B, U401C, U401D, U402A, U402B, U402C, U402D, U403B, U404A, U404B, U404C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

Commit message: TOD is here
Parts:
- renumbered U402 to U497, U401 to U498, U403 to U503, U404 to U504, U405 to U505
Connections:
- net ALARM: now also U503.11; no longer U503.3
- net ENABLE_NAND: now also U497.10, U497.2; no longer U498.13, U498.5
- net ~{EN10}: now also U498.9; no longer U497.2
- net ~{EN11}: now also U498.13; no longer U497.10
- net ~{EN8}: now also U498.1; no longer U498.2
- net ~{EN9}: now also U498.5; no longer U498.10
- net ~{RES}: now also U498.10, U498.12, U498.2, U498.4; no longer U497.1, U497.9, U498.1, U498.9
- net at U498.8: now also U497.9; no longer U498.12
- net at U497.3: now also U406.1, U505.1; no longer U497.4
- net at U497.8: now also U406.9, U505.9; no longer U497.12
- net ~{ALARM: now reaches U406.10, U406.13, U406.2, U406.5
- net ~{ALARM: now also U503.10; no longer U503.4
- net at U498.3: now also U497.1; no longer U498.4
- net at U406.4, U505.4: now also U497.6; no longer U498.11
- new net: U497.12, U498.11
- new net: U497.4, U498.6
Other:
- moved on the sheet: U497A, U497B, U497C, U498B, U498C, U498D

Commit message: Ready for v0.2.2
Parts:
- renumbered U503 to U429, U504 to U430, U498 to U431, U497 to U432, U406 to U433, U505 to U434, U429 to U436
Other:
- company: (none) -> Daniel Molina
- title: (none) -> 74HCT6526 Board 4
Changed lines of the file:
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@@
 (kicad_sch (version 20211123) (generator eeschema)
   (paper "A4")
+  (title_block
+    (title "74HCT6526 Board 4")
+    (date "2023-06-22")
+    (rev "0.2.2")
+    (company "Daniel Molina")
+    (comment 1 "https://github.com/dmolinagarcia/74HCT6526")
+  )
   (junction (at 96.52 31.75) (diameter 0) (color 0 0 0 0)
   )
@@
   (symbol (lib_id "74xx:74HC00") (at 111.76 64.77 0) (mirror x) (unit 3)
     (in_bom yes) (on_board yes) (fields_autoplaced)
-    (property "Reference" "U498" (id 0) (at 111.76 55.88 0))
+    (property "Reference" "U431" (id 0) (at 111.76 55.88 0))
     (property "Value" "74HC00" (id 1) (at 111.76 58.42 0))
     (property "Footprint" "Package_SO:SOIC-14_3.9x8.7mm_P1.27mm" (id 2) (at 111.76 64.77 0)
@@
   (symbol (lib_id "74xx:74HC00") (at 127 36.83 0) (unit 1)
     (in_bom yes) (on_board yes) (fields_autoplaced)
-    (property "Reference" "U497" (id 0) (at 127 27.94 0))
+    (property "Reference" "U432" (id 0) (at 127 27.94 0))
     (property "Value" "74HC00" (id 1) (at 127 30.48 0))
     (property "Footprint" "Package_SO:SOIC-14_3.9x8.7mm_P1.27mm" (id 2) (at 127 36.83 0)
@@
   (symbol (lib_id "74xx:74HC00") (at 127 67.31 0) (unit 3)
     (in_bom yes) (on_board yes) (fields_autoplaced)
-    (property "Reference" "U497" (id 0) (at 127 58.42 0))
+    (property "Reference" "U432" (id 0) (at 127 58.42 0))
     (property "Value" "74HC00" (id 1) (at 127 60.96 0))
     (property "Footprint" "Package_SO:SOIC-14_3.9x8.7mm_P1.27mm" (id 2) (at 127 67.31 0)
@@
   (symbol (lib_id "74xx:74LS32") (at 165.1 99.06 0) (unit 1)
     (in_bom yes) (on_board yes) (fields_autoplaced)
-    (property "Reference" "U406" (id 0) (at 165.1 90.17 0))
+    (property "Reference" "U433" (id 0) (at 165.1 90.17 0))
     (property "Value" "74HC32" (id 1) (at 165.1 92.71 0))
     (property "Footprint" "Package_SO:SOIC-14_3.9x8.7mm_P1.27mm" (id 2) (at 165.1 99.06 0)
@@
   (symbol (lib_id "74xx:74HC00") (at 127 82.55 0) (unit 4)
     (in_bom yes) (on_board yes) (fields_autoplaced)
-    (property "Reference" "U497" (id 0) (at 127 73.66 0))
+    (property "Reference" "U432" (id 0) (at 127 73.66 0))
     (property "Value" "74HC00" (id 1) (at 127 76.2 0))
     (property "Footprint" "Package_SO:SOIC-14_3.9x8.7mm_P1.27mm" (id 2) (at 127 82.55 0)
@@
   (symbol (lib_id "74xx:74LS32") (at 165.1 39.37 0) (unit 1)
     (in_bom yes) (on_board yes) (fields_autoplaced)
-    (property "Reference" "U505" (id 0) (at 165.1 30.48 0))
+    (property "Reference" "U434" (id 0) (at 165.1 30.48 0))
     (property "Value" "74HC32" (id 1) (at 165.1 33.02 0))
     (property "Footprint" "Package_SO:SOIC-14_3.9x8.7mm_P1.27mm" (id 2) (at 165.1 39.37 0)
@@
   (symbol (lib_id "74xx:74HC04") (at 73.66 22.86 0) (unit 5)
     (in_bom yes) (on_board yes)
-    (property "Reference" "U503" (id 0) (at 76.2 19.05 0))
+    (property "Reference" "U429" (id 0) (at 76.2 19.05 0))
     (property "Value" "74HC04" (id 1) (at 77.47 26.67 0))
     (property "Footprint" "Package_SO:SOIC-14_3.9x8.7mm_P1.27mm" (id 2) (at 73.66 22.86 0)
@@
   (symbol (lib_id "74xx:74LS32") (at 165.1 69.85 0) (unit 3)
     (in_bom yes) (on_board yes) (fields_autoplaced)
-    (property "Reference" "U505" (id 0) (at 165.1 60.96 0))
+    (property "Reference" "U434" (id 0) (at 165.1 60.96 0))
     (property "Value" "74HC32" (id 1) (at 165.1 63.5 0))
     (property "Footprint" "Package_SO:SOIC-14_3.9x8.7mm_P1.27mm" (id 2) (at 165.1 69.85 0)
@@
   (symbol (lib_id "74xx:74HC00") (at 111.76 34.29 0) (mirror x) (unit 1)
     (in_bom yes) (on_board yes) (fields_autoplaced)
-    (property "Reference" "U498" (id 0) (at 111.76 25.4 0))
+    (property "Reference" "U431" (id 0) (at 111.76 25.4 0))
     (property "Value" "74HC00" (id 1) (at 111.76 27.94 0))
     (property "Footprint" "Package_SO:SOIC-14_3.9x8.7mm_P1.27mm" (id 2) (at 111.76 34.29 0)
@@
   (symbol (lib_id "74xx:74HC00") (at 127 52.07 0) (unit 2)
     (in_bom yes) (on_board yes) (fields_autoplaced)
-    (property "Reference" "U497" (id 0) (at 127 43.18 0))
+    (property "Reference" "U432" (id 0) (at 127 43.18 0))
     (property "Value" "74HC00" (id 1) (at 127 45.72 0))
     (property "Footprint" "Package_SO:SOIC-14_3.9x8.7mm_P1.27mm" (id 2) (at 127 52.07 0)
@@
   (symbol (lib_id "74xx:74LS32") (at 165.1 129.54 0) (unit 3)
     (in_bom yes) (on_board yes) (fields_autoplaced)
-    (property "Reference" "U406" (id 0) (at 165.1 120.65 0))
+    (property "Reference" "U433" (id 0) (at 165.1 120.65 0))
     (property "Value" "74HC32" (id 1) (at 165.1 123.19 0))
     (property "Footprint" "Package_SO:SOIC-14_3.9x8.7mm_P1.27mm" (id 2) (at 165.1 129.54 0)
@@
   (symbol (lib_id "74xx:74LS32") (at 165.1 114.3 0) (unit 2)
     (in_bom yes) (on_board yes) (fields_autoplaced)
-    (property "Reference" "U406" (id 0) (at 165.1 105.41 0))
+    (property "Reference" "U433" (id 0) (at 165.1 105.41 0))
     (property "Value" "74HC32" (id 1) (at 165.1 107.95 0))
     (property "Footprint" "Package_SO:SOIC-14_3.9x8.7mm_P1.27mm" (id 2) (at 165.1 114.3 0)
@@
   (symbol (lib_id "74xx:74LS32") (at 165.1 144.78 0) (unit 4)
     (in_bom yes) (on_board yes) (fields_autoplaced)
-    (property "Reference" "U406" (id 0) (at 165.1 135.89 0))
+    (property "Reference" "U433" (id 0) (at 165.1 135.89 0))
     (property "Value" "74HC32" (id 1) (at 165.1 138.43 0))
     (property "Footprint" "Package_SO:SOIC-14_3.9x8.7mm_P1.27mm" (id 2) (at 165.1 144.78 0)
@@
   (symbol (lib_id "74xx:74HC74") (at 247.65 68.58 0) (unit 1)
     (in_bom yes) (on_board yes) (fields_autoplaced)
-    (property "Reference" "U429" (id 0) (at 249.6694 58.42 0)
+    (property "Reference" "U436" (id 0) (at 249.6694 58.42 0)
       (effects (font (size 1.27 1.27)) (justify left))
     )
@@
   (symbol (lib_id "74xx:74LS32") (at 111.76 132.08 0) (unit 1)
     (in_bom yes) (on_board yes) (fields_autoplaced)
-    (property "Reference" "U504" (id 0) (at 111.76 123.19 0))
+    (property "Reference" "U430" (id 0) (at 111.76 123.19 0))
     (property "Value" "74HC32" (id 1) (at 111.76 125.73 0))
     (property "Footprint" "Package_SO:SOIC-14_3.9x8.7mm_P1.27mm" (id 2) (at 111.76 132.08 0)
@@
   (symbol (lib_id "74xx:74LS32") (at 165.1 85.09 0) (unit 4)
     (in_bom yes) (on_board yes) (fields_autoplaced)
-    (property "Reference" "U505" (id 0) (at 165.1 76.2 0))
+    (property "Reference" "U434" (id 0) (at 165.1 76.2 0))
     (property "Value" "74HC32" (id 1) (at 165.1 78.74 0))
     (property "Footprint" "Package_SO:SOIC-14_3.9x8.7mm_P1.27mm" (id 2) (at 165.1 85.09 0)
@@
   (symbol (lib_id "74xx:74LS32") (at 165.1 54.61 0) (unit 2)
     (in_bom yes) (on_board yes) (fields_autoplaced)
-    (property "Reference" "U505" (id 0) (at 165.1 45.72 0))
+    (property "Reference" "U434" (id 0) (at 165.1 45.72 0))
     (property "Value" "74HC32" (id 1) (at 165.1 48.26 0))
     (property "Footprint" "Package_SO:SOIC-14_3.9x8.7mm_P1.27mm" (id 2) (at 165.1 54.61 0)
@@
   (symbol (lib_id "74xx:74LS32") (at 111.76 148.59 0) (unit 2)
     (in_bom yes) (on_board yes) (fields_autoplaced)
-    (property "Reference" "U504" (id 0) (at 111.76 139.7 0))
+    (property "Reference" "U430" (id 0) (at 111.76 139.7 0))
     (property "Value" "74HC32" (id 1) (at 111.76 142.24 0))
     (property "Footprint" "Package_SO:SOIC-14_3.9x8.7mm_P1.27mm" (id 2) (at 111.76 148.59 0)
@@
   (symbol (lib_id "74xx:74LS32") (at 111.76 181.61 0) (unit 4)
     (in_bom yes) (on_board yes) (fields_autoplaced)
-    (property "Reference" "U504" (id 0) (at 111.76 172.72 0))
+    (property "Reference" "U430" (id 0) (at 111.76 172.72 0))
     (property "Value" "74HC32" (id 1) (at 111.76 175.26 0))
     (property "Footprint" "Package_SO:SOIC-14_3.9x8.7mm_P1.27mm" (id 2) (at 111.76 181.61 0)
@@
   (symbol (lib_id "74xx:74HC74") (at 165.1 165.1 0) (unit 2)
     (in_bom yes) (on_board yes) (fields_autoplaced)
-    (property "Reference" "U429" (id 0) (at 167.1194 154.94 0)
+    (property "Reference" "U436" (id 0) (at 167.1194 154.94 0)
       (effects (font (size 1.27 1.27)) (justify left))
     )
@@
   (symbol (lib_id "74xx:74HC00") (at 111.76 49.53 0) (unit 2)
     (in_bom yes) (on_board yes) (fields_autoplaced)
-    (property "Reference" "U498" (id 0) (at 111.76 40.64 0))
+    (property "Reference" "U431" (id 0) (at 111.76 40.64 0))
     (property "Value" "74HC00" (id 1) (at 111.76 43.18 0))
     (property "Footprint" "Package_SO:SOIC-14_3.9x8.7mm_P1.27mm" (id 2) (at 111.76 49.53 0)
@@
   (symbol (lib_id "74xx:74HC00") (at 111.76 80.01 0) (unit 4)
     (in_bom yes) (on_board yes) (fields_autoplaced)
-    (property "Reference" "U498" (id 0) (at 111.76 71.12 0))
+    (property "Reference" "U431" (id 0) (at 111.76 71.12 0))
     (property "Value" "74HC00" (id 1) (at 111.76 73.66 0))
     (property "Footprint" "Package_SO:SOIC-14_3.9x8.7mm_P1.27mm" (id 2) (at 111.76 80.01 0)
@@
   (symbol (lib_id "74xx:74LS32") (at 111.76 165.1 0) (unit 3)
     (in_bom yes) (on_board yes) (fields_autoplaced)
-    (property "Reference" "U504" (id 0) (at 111.76 156.21 0))
+    (property "Reference" "U430" (id 0) (at 111.76 156.21 0))
     (property "Value" "74HC32" (id 1) (at 111.76 158.75 0))
     (property "Footprint" "Package_SO:SOIC-14_3.9x8.7mm_P1.27mm" (id 2) (at 111.76 165.1 0)
