File: B4/todHours.kicad_sch (KiCad schematic)
At the start: 9 parts, among them U403 74HC04, U415 74HC32, U430 74HC193, U431 74HC04, U432 74HC08, U433 74HC74, U434 74HC74, U435 74HC11, U436 74HC00

Commit message: TOD is here
Parts:
- renumbered U403 to U503
Connections:
- net DZ0: now also U415.13; no longer U415.10
- net DZ2: now also U432.4; no longer U432.5
- net DZ4: now also U436.5; no longer U436.2
- net DZ7: now also U436.9; no longer U436.10
- net H4_FLIP: now also U415.8; no longer U415.11
- net ~{LOADH}: now also U415.4; no longer U415.5
- net at U430.14 (CLR), U435.12: now also U415.9; no longer U415.12
- net at U431.13, U435.6: now also U415.10; no longer U415.13
- net at U435.8: now also U503.3; no longer U503.13
- net at U431.4, U432.1, U432.9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: now also U432.5, U436.10, U436.13; no longer U432.4, U436.12, U436.9
- net at U436.3: now also U433.1 (~{R}); no longer U433.4 (~{S})
- net at U431.8: now also U436.12; no longer U436.13
- net at U431.6: now also U436.2; no longer U436.5
- net at U434.13 (~{R}): now also U503.4; no longer U503.12
- net at U436.6: now also U433.4 (~{S}); no longer U433.1 (~{R})
- net at U415.6, U431.3: now also U415.12; no longer U415.9
- net at U430.15 (A): now also U415.11; no longer U415.8
- net at U431.2: now also U415.5; no longer U415.4
Other:
- moved on the sheet: U415C, U415D, U436A, U436B

Commit message: Ready for v0.2.2
Parts:
- renumbered U415 to U418, U432 to U419, U430 to U421, U435 to U422, U431 to U425, U436 to U426, U433 to U427, U434 to U428, U503 to U429
Other:
- company: (none) -> Daniel Molina
- title: (none) -> 74HCT6526 Board 4
Changed lines of the file:
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@@
 (kicad_sch (version 20211123) (generator eeschema)
   (paper "A4")
+  (title_block
+    (title "74HCT6526 Board 4")
+    (date "2023-06-22")
+    (rev "0.2.2")
+    (company "Daniel Molina")
+    (comment 1 "https://github.com/dmolinagarcia/74HCT6526")
+  )
   (junction (at 90.17 49.53) (diameter 0) (color 0 0 0 0)
   )
@@
   (symbol (lib_id "74xx:74HC04") (at 177.8 107.95 0) (unit 5)
     (in_bom yes) (on_board yes)
-    (property "Reference" "U431" (id 0) (at 177.8 106.68 0))
+    (property "Reference" "U425" (id 0) (at 177.8 106.68 0))
     (property "Value" "74HC04" (id 1) (at 177.8 109.22 0))
     (property "Footprint" "Package_SO:SOIC-14_3.9x8.7mm_P1.27mm" (id 2) (at 177.8 107.95 0)
@@
   (symbol (lib_id "74xx:74LS32") (at 104.14 26.67 0) (unit 4)
     (in_bom yes) (on_board yes) (fields_autoplaced)
-    (property "Reference" "U415" (id 0) (at 104.14 17.78 0))
+    (property "Reference" "U418" (id 0) (at 104.14 17.78 0))
     (property "Value" "74HC32" (id 1) (at 104.14 20.32 0))
     (property "Footprint" "Package_SO:SOIC-14_3.9x8.7mm_P1.27mm" (id 2) (at 104.14 26.67 0)
@@
   (symbol (lib_id "74xx:74LS11") (at 194.31 113.03 0) (unit 3)
     (in_bom yes) (on_board yes)
-    (property "Reference" "U435" (id 0) (at 194.31 111.76 0))
+    (property "Reference" "U422" (id 0) (at 194.31 111.76 0))
     (property "Value" "74HC11" (id 1) (at 194.31 114.3 0))
     (property "Footprint" "Package_SO:SOIC-14_3.9x8.7mm_P1.27mm" (id 2) (at 194.31 113.03 0)
@@
   (symbol (lib_id "74xx:74HC00") (at 102.87 120.65 0) (unit 1)
     (in_bom yes) (on_board yes)
-    (property "Reference" "U436" (id 0) (at 102.87 119.38 0))
+    (property "Reference" "U426" (id 0) (at 102.87 119.38 0))
     (property "Value" "74HC00" (id 1) (at 102.87 121.92 0))
     (property "Footprint" "Package_SO:SOIC-14_3.9x8.7mm_P1.27mm" (id 2) (at 102.87 120.65 0)
@@
   (symbol (lib_id "Custom 74xx:74HC08") (at 104.14 52.07 0) (mirror x) (unit 2)
     (in_bom yes) (on_board yes)
-    (property "Reference" "U432" (id 0) (at 104.14 53.34 0))
+    (property "Reference" "U419" (id 0) (at 104.14 53.34 0))
     (property "Value" "74HC08" (id 1) (at 104.14 50.8 0))
     (property "Footprint" "Package_SO:SOIC-14_3.9x8.7mm_P1.27mm" (id 2) (at 104.14 52.07 0)
@@
   (symbol (lib_id "74xx:74HC74") (at 137.16 144.78 0) (unit 2)
     (in_bom yes) (on_board yes) (fields_autoplaced)
-    (property "Reference" "U433" (id 0) (at 139.1794 134.62 0)
+    (property "Reference" "U427" (id 0) (at 139.1794 134.62 0)
       (effects (font (size 1.27 1.27)) (justify left))
     )
@@
   (symbol (lib_id "Custom 74xx:74HC08") (at 104.14 43.18 0) (unit 1)
     (in_bom yes) (on_board yes)
-    (property "Reference" "U432" (id 0) (at 104.14 41.91 0))
+    (property "Reference" "U419" (id 0) (at 104.14 41.91 0))
     (property "Value" "74HC08" (id 1) (at 104.14 44.45 0))
     (property "Footprint" "Package_SO:SOIC-14_3.9x8.7mm_P1.27mm" (id 2) (at 104.14 43.18 0)
@@
   (symbol (lib_id "74xx:74HC04") (at 52.07 157.48 0) (unit 4)
     (in_bom yes) (on_board yes)
-    (property "Reference" "U431" (id 0) (at 52.07 156.21 0))
+    (property "Reference" "U425" (id 0) (at 52.07 156.21 0))
     (property "Value" "74HC04" (id 1) (at 52.07 158.75 0))
     (property "Footprint" "Package_SO:SOIC-14_3.9x8.7mm_P1.27mm" (id 2) (at 52.07 157.48 0)
@@
   (symbol (lib_id "74xx:74HC04") (at 52.07 123.19 0) (mirror x) (unit 3)
     (in_bom yes) (on_board yes)
-    (property "Reference" "U431" (id 0) (at 52.07 121.92 0))
+    (property "Reference" "U425" (id 0) (at 52.07 121.92 0))
     (property "Value" "74HC04" (id 1) (at 52.07 124.46 0))
     (property "Footprint" "Package_SO:SOIC-14_3.9x8.7mm_P1.27mm" (id 2) (at 52.07 123.19 0)
@@
   (symbol (lib_id "Custom 74xx:74HC08") (at 259.08 106.68 0) (unit 4)
     (in_bom yes) (on_board yes) (fields_autoplaced)
-    (property "Reference" "U432" (id 0) (at 259.08 97.79 0))
+    (property "Reference" "U419" (id 0) (at 259.08 97.79 0))
     (property "Value" "74HC08" (id 1) (at 259.08 100.33 0))
     (property "Footprint" "Package_SO:SOIC-14_3.9x8.7mm_P1.27mm" (id 2) (at 259.08 106.68 0)
@@
   (symbol (lib_id "74xx:74HC04") (at 208.28 123.19 270) (unit 2)
     (in_bom yes) (on_board yes) (fields_autoplaced)
-    (property "Reference" "U503" (id 0) (at 213.36 121.9199 90)
+    (property "Reference" "U429" (id 0) (at 213.36 121.9199 90)
       (effects (font (size 1.27 1.27)) (justify left))
     )
@@
   (symbol (lib_id "74xx:74HC74") (at 137.16 110.49 0) (unit 1)
     (in_bom yes) (on_board yes) (fields_autoplaced)
-    (property "Reference" "U433" (id 0) (at 139.1794 100.33 0)
+    (property "Reference" "U427" (id 0) (at 139.1794 100.33 0)
       (effects (font (size 1.27 1.27)) (justify left))
     )
@@
   (symbol (lib_id "74xx:74HC04") (at 80.01 40.64 0) (unit 2)
     (in_bom yes) (on_board yes)
-    (property "Reference" "U431" (id 0) (at 76.2 41.91 0)
+    (property "Reference" "U425" (id 0) (at 76.2 41.91 0)
       (effects (font (size 1.27 1.27)) (justify left))
     )
@@
   (symbol (lib_id "74xx:74HC00") (at 102.87 154.94 0) (mirror x) (unit 4)
     (in_bom yes) (on_board yes)
-    (property "Reference" "U436" (id 0) (at 102.87 156.21 0))
+    (property "Reference" "U426" (id 0) (at 102.87 156.21 0))
     (property "Value" "74HC00" (id 1) (at 102.87 153.67 0))
     (property "Footprint" "Package_SO:SOIC-14_3.9x8.7mm_P1.27mm" (id 2) (at 102.87 154.94 0)
@@
   (symbol (lib_id "74xx:74HC00") (at 102.87 100.33 0) (unit 2)
     (in_bom yes) (on_board yes)
-    (property "Reference" "U436" (id 0) (at 102.87 99.06 0))
+    (property "Reference" "U426" (id 0) (at 102.87 99.06 0))
     (property "Value" "74HC00" (id 1) (at 102.87 101.6 0))
     (property "Footprint" "Package_SO:SOIC-14_3.9x8.7mm_P1.27mm" (id 2) (at 102.87 100.33 0)
@@
   (symbol (lib_id "74xx:74HC00") (at 102.87 134.62 0) (mirror x) (unit 3)
     (in_bom yes) (on_board yes)
-    (property "Reference" "U436" (id 0) (at 102.87 135.89 0))
+    (property "Reference" "U426" (id 0) (at 102.87 135.89 0))
     (property "Value" "74HC00" (id 1) (at 102.87 133.35 0))
     (property "Footprint" "Package_SO:SOIC-14_3.9x8.7mm_P1.27mm" (id 2) (at 102.87 134.62 0)
@@
   (symbol (lib_id "74xx:74LS193") (at 137.16 57.15 0) (unit 1)
     (in_bom yes) (on_board yes) (fields_autoplaced)
-    (property "Reference" "U430" (id 0) (at 139.1794 39.37 0)
+    (property "Reference" "U421" (id 0) (at 139.1794 39.37 0)
       (effects (font (size 1.27 1.27)) (justify left))
     )
@@
   (symbol (lib_id "74xx:74LS11") (at 194.31 95.25 0) (unit 2)
     (in_bom yes) (on_board yes)
-    (property "Reference" "U435" (id 0) (at 194.31 93.98 0))
+    (property "Reference" "U422" (id 0) (at 194.31 93.98 0))
     (property "Value" "74HC11" (id 1) (at 194.31 96.52 0))
     (property "Footprint" "Package_SO:SOIC-14_3.9x8.7mm_P1.27mm" (id 2) (at 194.31 95.25 0)
@@
   (symbol (lib_id "Custom 74xx:74HC08") (at 104.14 60.96 0) (unit 3)
     (in_bom yes) (on_board yes)
-    (property "Reference" "U432" (id 0) (at 104.14 59.69 0))
+    (property "Reference" "U419" (id 0) (at 104.14 59.69 0))
     (property "Value" "74HC08" (id 1) (at 104.14 62.23 0))
     (property "Footprint" "Package_SO:SOIC-14_3.9x8.7mm_P1.27mm" (id 2) (at 104.14 60.96 0)
@@
   (symbol (lib_id "74xx:74HC74") (at 236.22 137.16 0) (unit 2)
     (in_bom yes) (on_board yes) (fields_autoplaced)
-    (property "Reference" "U434" (id 0) (at 238.2394 127 0)
+    (property "Reference" "U428" (id 0) (at 238.2394 127 0)
       (effects (font (size 1.27 1.27)) (justify left))
     )
@@
   (symbol (lib_id "74xx:74LS11") (at 194.31 78.74 0) (unit 1)
     (in_bom yes) (on_board yes)
-    (property "Reference" "U435" (id 0) (at 194.31 77.47 0))
+    (property "Reference" "U422" (id 0) (at 194.31 77.47 0))
     (property "Value" "74HC11" (id 1) (at 194.31 80.01 0))
     (property "Footprint" "Package_SO:SOIC-14_3.9x8.7mm_P1.27mm" (id 2) (at 194.31 78.74 0)
@@
   (symbol (lib_id "74xx:74LS32") (at 62.23 24.13 0) (mirror x) (unit 2)
     (in_bom yes) (on_board yes)
-    (property "Reference" "U415" (id 0) (at 62.23 26.67 0))
+    (property "Reference" "U418" (id 0) (at 62.23 26.67 0))
     (property "Value" "74HC32" (id 1) (at 62.23 24.13 0))
     (property "Footprint" "Package_SO:SOIC-14_3.9x8.7mm_P1.27mm" (id 2) (at 62.23 24.13 0)
@@
   (symbol (lib_id "74xx:74HC04") (at 45.72 21.59 0) (unit 1)
     (in_bom yes) (on_board yes)
-    (property "Reference" "U431" (id 0) (at 45.72 21.59 0))
+    (property "Reference" "U425" (id 0) (at 45.72 21.59 0))
     (property "Value" "74HC04" (id 1) (at 49.53 24.13 0))
     (property "Footprint" "Package_SO:SOIC-14_3.9x8.7mm_P1.27mm" (id 2) (at 45.72 21.59 0)
@@
   (symbol (lib_id "74xx:74LS32") (at 226.06 81.28 0) (unit 3)
     (in_bom yes) (on_board yes)
-    (property "Reference" "U415" (id 0) (at 226.06 80.01 0))
+    (property "Reference" "U418" (id 0) (at 226.06 80.01 0))
     (property "Value" "74HC32" (id 1) (at 226.06 82.55 0))
     (property "Footprint" "Package_SO:SOIC-14_3.9x8.7mm_P1.27mm" (id 2) (at 226.06 81.28 0)
@@
   (symbol (lib_id "74xx:74HC04") (at 214.63 95.25 0) (unit 6)
     (in_bom yes) (on_board yes) (fields_autoplaced)
-    (property "Reference" "U431" (id 0) (at 214.63 86.36 0))
+    (property "Reference" "U425" (id 0) (at 214.63 86.36 0))
     (property "Value" "74HC04" (id 1) (at 214.63 88.9 0))
     (property "Footprint" "Package_SO:SOIC-14_3.9x8.7mm_P1.27mm" (id 2) (at 214.63 95.25 0)
@@
   (symbol (lib_id "74xx:74HC74") (at 236.22 106.68 0) (unit 1)
     (in_bom yes) (on_board yes) (fields_autoplaced)
-    (property "Reference" "U434" (id 0) (at 238.2394 96.52 0)
+    (property "Reference" "U428" (id 0) (at 238.2394 96.52 0)
       (effects (font (size 1.27 1.27)) (justify left))
     )
