File: B4/todMinutes.kicad_sch (KiCad schematic)
At the start: 3 parts, among them U418 74HC08, U419 74HC193, U420 74HC193

Commit message: TOD is here
Connections:
- net HOU_TK: now also U418.8; no longer U418.11
- net M1: now also U418.4; no longer U418.9
- net M3: now also U418.5; no longer U418.10
- net M5: now also U418.10; no longer U418.12
- net M6: now also U418.9; no longer U418.13
- net at U419.14 (CLR), U420.5 (UP): now also U418.6; no longer U418.8
Changed lines of the file:
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@@
     (pin "1")
   )
-  (symbol (lib_id "Custom 74xx:74HC08") (at 189.23 69.85 0) (unit 3)
+  (symbol (lib_id "Custom 74xx:74HC08") (at 189.23 69.85 0) (unit 2)
     (in_bom yes) (on_board yes) (fields_autoplaced)
     (property "Reference" "U418" (id 0) (at 189.23 60.96 0))
@@
     (pin "9")
   )
-  (symbol (lib_id "Custom 74xx:74HC08") (at 189.23 137.16 0) (unit 4)
+  (symbol (lib_id "Custom 74xx:74HC08") (at 189.23 137.16 0) (mirror x) (unit 3)
     (in_bom yes) (on_board yes) (fields_autoplaced)
     (property "Reference" "U418" (id 0) (at 189.23 128.27 0))
@@
       (effects (font (size 1.27 1.27)) hide)
     )
-    (property "Datasheet" "" (id 3) (at 189.23 130.81 0)
+    (property "Datasheet" "" (id 3) (at 189.23 143.51 0)
       (effects (font (size 1.27 1.27)) hide)
     )

Commit message: Ready for v0.2.2
Parts:
- renumbered U418 to U407, U420 to U414, U419 to U415
Other:
- company: (none) -> Daniel Molina
- title: (none) -> 74HCT6526 Board 4
Changed lines of the file:
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@@
 (kicad_sch (version 20211123) (generator eeschema)
   (paper "A4")
+  (title_block
+    (title "74HCT6526 Board 4")
+    (date "2023-06-22")
+    (rev "0.2.2")
+    (company "Daniel Molina")
+    (comment 1 "https://github.com/dmolinagarcia/74HCT6526")
+  )
   (junction (at 92.71 81.28) (diameter 0) (color 0 0 0 0)
   )
@@
   (symbol (lib_id "Custom 74xx:74HC08") (at 189.23 69.85 0) (unit 2)
     (in_bom yes) (on_board yes) (fields_autoplaced)
-    (property "Reference" "U418" (id 0) (at 189.23 60.96 0))
+    (property "Reference" "U407" (id 0) (at 189.23 60.96 0))
     (property "Value" "74HC08" (id 1) (at 189.23 63.5 0))
     (property "Footprint" "Package_SO:SOIC-14_3.9x8.7mm_P1.27mm" (id 2) (at 189.23 69.85 0)
@@
   (symbol (lib_id "74xx:74LS193") (at 118.11 109.22 0) (unit 1)
     (in_bom yes) (on_board yes) (fields_autoplaced)
-    (property "Reference" "U420" (id 0) (at 120.1294 91.44 0)
+    (property "Reference" "U414" (id 0) (at 120.1294 91.44 0)
       (effects (font (size 1.27 1.27)) (justify left))
     )
@@
   (symbol (lib_id "74xx:74LS193") (at 118.11 44.45 0) (unit 1)
     (in_bom yes) (on_board yes) (fields_autoplaced)
-    (property "Reference" "U419" (id 0) (at 120.1294 26.67 0)
+    (property "Reference" "U415" (id 0) (at 120.1294 26.67 0)
       (effects (font (size 1.27 1.27)) (justify left))
     )
@@
   (symbol (lib_id "Custom 74xx:74HC08") (at 189.23 137.16 0) (mirror x) (unit 3)
     (in_bom yes) (on_board yes) (fields_autoplaced)
-    (property "Reference" "U418" (id 0) (at 189.23 128.27 0))
+    (property "Reference" "U407" (id 0) (at 189.23 128.27 0))
     (property "Value" "74HC08" (id 1) (at 189.23 130.81 0))
     (property "Footprint" "Package_SO:SOIC-14_3.9x8.7mm_P1.27mm" (id 2) (at 189.23 137.16 0)
