File: B4/todPower.kicad_sch (KiCad schematic)
At the start: 17 parts, among them U401 74HC00, U402 74HC00, U403 74HC04, U404 74HC32, U405 74HC32, U406 74HC32, U411 74HC08, U414 74HC11, U415 74HC32, U418 74HC08, U429 74HC74, U431 74HC04, U432 74HC08, U433 74HC74, U434 74HC74, U435 74HC11, U436 74HC00

Commit message: TOD is here
Parts:
- removed unit 3 of U414
- added C401, C402, C403, C404, C405, C406, C407, C408, C409, C410, C411, C412, C413, C414, C416, C417, C418, C419, C420, C421, C422, C423, C424, C426, C427, C428, C429, C430, C431, C432, C433, C434, C435, C436, C504, C505: 100n, Capacitor_SMD:C_0603_1608Metric, symbol Device:C
- added unit 2 of U411
- renumbered U402 to U497, U401 to U498, U403 to U503, U404 to U504, U405 to U505
Connections:
- net GND: now also U406.7 (GND), U411.1, U411.12, U411.13, U411.2, U411.7 (GND), U414.7 (GND), U418.7 (GND), U429.7 (GND), U431.7 (GND), U432.7 (GND), U433.7 (GND), U434.7 (GND), U498.7 (GND), U503.1, U504.7 (GND), U505.7 (GND), C401.2, C402.2, C403.2, C404.2, C405.2, C406.2, C407.2, C408.2, C409.2, C410.2, C411.2, C412.2, C413.2, C414.2, C416.2, C417.2, C418.2, C419.2, C420.2, C421.2, C422.2, C423.2, C424.2, C426.2, C427.2, C428.2, C429.2, C430.2, C431.2, C432.2, C433.2, C434.2, C435.2, C436.2, C504.2, C505.2, U411.4, U411.5; no longer U411.13
- net VCC: now also U411.14 (VCC), C401.1, C402.1, C403.1, C404.1, C405.1, C406.1, C407.1, C408.1, C409.1, C410.1, C411.1, C412.1, C413.1, C414.1, C416.1, C417.1, C418.1, C419.1, C420.1, C421.1, C422.1, C423.1, C424.1, C426.1, C427.1, C428.1, C429.1, C430.1, C431.1, C432.1, C433.1, C434.1, C435.1, C436.1, C504.1, C505.1

Commit message: .
Parts:
- U411: value 74HC08 -> 74HCT08
Changed lines of the file:
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@@
     (in_bom yes) (on_board yes) (fields_autoplaced)
     (property "Reference" "U411" (id 0) (at 181.61 67.31 0))
-    (property "Value" "74HC08" (id 1) (at 181.61 69.85 0))
+    (property "Value" "74HCT08" (id 1) (at 181.61 69.85 0))
     (property "Footprint" "Package_SO:SOIC-14_3.9x8.7mm_P1.27mm" (id 2) (at 181.61 76.2 0)
       (effects (font (size 1.27 1.27)) hide)
@@
       (effects (font (size 1.27 1.27)) (justify left))
     )
-    (property "Value" "74HC08" (id 1) (at 85.09 80.0099 0)
+    (property "Value" "74HCT08" (id 1) (at 85.09 80.0099 0)
       (effects (font (size 1.27 1.27)) (justify left))
     )
@@
     (in_bom yes) (on_board yes) (fields_autoplaced)
     (property "Reference" "U411" (id 0) (at 181.61 97.79 0))
-    (property "Value" "74HC08" (id 1) (at 181.61 100.33 0))
+    (property "Value" "74HCT08" (id 1) (at 181.61 100.33 0))
     (property "Footprint" "Package_SO:SOIC-14_3.9x8.7mm_P1.27mm" (id 2) (at 181.61 106.68 0)
       (effects (font (size 1.27 1.27)) hide)
@@
     (in_bom yes) (on_board yes) (fields_autoplaced)
     (property "Reference" "U411" (id 0) (at 181.61 113.03 0))
-    (property "Value" "74HC08" (id 1) (at 181.61 115.57 0))
+    (property "Value" "74HCT08" (id 1) (at 181.61 115.57 0))
     (property "Footprint" "Package_SO:SOIC-14_3.9x8.7mm_P1.27mm" (id 2) (at 181.61 121.92 0)
       (effects (font (size 1.27 1.27)) hide)

Commit message: Ready for v0.2.2
Parts:
- renumbered U414 to U401, U418 to U407, U415 to U418, U432 to U419, U435 to U422, U431 to U425, U436 to U426, U433 to U427, U434 to U428, U503 to U429, U504 to U430, U498 to U431, U497 to U432, U406 to U433, U505 to U434, U411 to U435, U429 to U436
Other:
- company: (none) -> Daniel Molina
- title: (none) -> 74HCT6526 Board 4
Changed lines of the file:
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@@
 (kicad_sch (version 20211123) (generator eeschema)
   (paper "A4")
+  (title_block
+    (title "74HCT6526 Board 4")
+    (date "2023-06-22")
+    (rev "0.2.2")
+    (company "Daniel Molina")
+    (comment 1 "https://github.com/dmolinagarcia/74HCT6526")
+  )
   (junction (at 54.61 133.35) (diameter 0) (color 0 0 0 0)
   )
@@
   (symbol (lib_id "74xx:74HC04") (at 31.75 40.64 0) (unit 7)
     (in_bom yes) (on_board yes) (fields_autoplaced)
-    (property "Reference" "U431" (id 0) (at 38.1 39.3699 0)
+    (property "Reference" "U425" (id 0) (at 38.1 39.3699 0)
       (effects (font (size 1.27 1.27)) (justify left))
     )
@@
   (symbol (lib_id "74xx:74HC74") (at 147.32 41.91 0) (unit 3)
     (in_bom yes) (on_board yes) (fields_autoplaced)
-    (property "Reference" "U434" (id 0) (at 153.67 40.6399 0)
+    (property "Reference" "U428" (id 0) (at 153.67 40.6399 0)
       (effects (font (size 1.27 1.27)) (justify left))
     )
@@
   (symbol (lib_id "Custom 74xx:74HC08") (at 181.61 76.2 0) (unit 2)
     (in_bom yes) (on_board yes) (fields_autoplaced)
-    (property "Reference" "U411" (id 0) (at 181.61 67.31 0))
+    (property "Reference" "U435" (id 0) (at 181.61 67.31 0))
     (property "Value" "74HCT08" (id 1) (at 181.61 69.85 0))
     (property "Footprint" "Package_SO:SOIC-14_3.9x8.7mm_P1.27mm" (id 2) (at 181.61 76.2 0)
@@
   (symbol (lib_id "Custom 74xx:74HC08") (at 31.75 78.74 0) (unit 5)
     (in_bom yes) (on_board yes) (fields_autoplaced)
-    (property "Reference" "U418" (id 0) (at 38.1 77.4699 0)
+    (property "Reference" "U407" (id 0) (at 38.1 77.4699 0)
       (effects (font (size 1.27 1.27)) (justify left))
     )
@@
   (symbol (lib_id "74xx:74HC04") (at 54.61 118.11 0) (unit 7)
     (in_bom yes) (on_board yes) (fields_autoplaced)
-    (property "Reference" "U503" (id 0) (at 62.23 116.8399 0)
+    (property "Reference" "U429" (id 0) (at 62.23 116.8399 0)
       (effects (font (size 1.27 1.27)) (justify left))
     )
@@
   (symbol (lib_id "Custom 74xx:74HC08") (at 77.47 78.74 0) (unit 5)
     (in_bom yes) (on_board yes) (fields_autoplaced)
-    (property "Reference" "U411" (id 0) (at 85.09 77.4699 0)
+    (property "Reference" "U435" (id 0) (at 85.09 77.4699 0)
       (effects (font (size 1.27 1.27)) (justify left))
     )
@@
   (symbol (lib_id "74xx:74LS11") (at 54.61 78.74 0) (unit 4)
     (in_bom yes) (on_board yes) (fields_autoplaced)
-    (property "Reference" "U414" (id 0) (at 60.96 77.4699 0)
+    (property "Reference" "U401" (id 0) (at 60.96 77.4699 0)
       (effects (font (size 1.27 1.27)) (justify left))
     )
@@
   (symbol (lib_id "Custom 74xx:74HC08") (at 181.61 106.68 0) (unit 4)
     (in_bom yes) (on_board yes) (fields_autoplaced)
-    (property "Reference" "U411" (id 0) (at 181.61 97.79 0))
+    (property "Reference" "U435" (id 0) (at 181.61 97.79 0))
     (property "Value" "74HCT08" (id 1) (at 181.61 100.33 0))
     (property "Footprint" "Package_SO:SOIC-14_3.9x8.7mm_P1.27mm" (id 2) (at 181.61 106.68 0)
@@
   (symbol (lib_id "74xx:74HC74") (at 100.33 41.91 0) (unit 3)
     (in_bom yes) (on_board yes) (fields_autoplaced)
-    (property "Reference" "U433" (id 0) (at 106.68 40.6399 0)
+    (property "Reference" "U427" (id 0) (at 106.68 40.6399 0)
       (effects (font (size 1.27 1.27)) (justify left))
     )
@@
   (symbol (lib_id "Custom 74xx:74HC08") (at 54.61 41.91 0) (unit 5)
     (in_bom yes) (on_board yes) (fields_autoplaced)
-    (property "Reference" "U432" (id 0) (at 60.96 40.6399 0)
+    (property "Reference" "U419" (id 0) (at 60.96 40.6399 0)
       (effects (font (size 1.27 1.27)) (justify left))
     )
@@
   (symbol (lib_id "74xx:74LS11") (at 100.33 118.11 0) (unit 4)
     (in_bom yes) (on_board yes) (fields_autoplaced)
-    (property "Reference" "U435" (id 0) (at 106.68 116.8399 0)
+    (property "Reference" "U422" (id 0) (at 106.68 116.8399 0)
       (effects (font (size 1.27 1.27)) (justify left))
     )
@@
   (symbol (lib_id "74xx:74HC04") (at 181.61 91.44 0) (unit 1)
     (in_bom yes) (on_board yes) (fields_autoplaced)
-    (property "Reference" "U503" (id 0) (at 181.61 82.55 0))
+    (property "Reference" "U429" (id 0) (at 181.61 82.55 0))
     (property "Value" "74HC04" (id 1) (at 181.61 85.09 0))
     (property "Footprint" "Package_SO:SOIC-14_3.9x8.7mm_P1.27mm" (id 2) (at 181.61 91.44 0)
@@
   (symbol (lib_id "74xx:74LS32") (at 31.75 118.11 0) (unit 5)
     (in_bom yes) (on_board yes) (fields_autoplaced)
-    (property "Reference" "U415" (id 0) (at 39.37 116.8399 0)
+    (property "Reference" "U418" (id 0) (at 39.37 116.8399 0)
       (effects (font (size 1.27 1.27)) (justify left))
     )
@@
   (symbol (lib_id "Custom 74xx:74HC08") (at 181.61 121.92 0) (unit 1)
     (in_bom yes) (on_board yes) (fields_autoplaced)
-    (property "Reference" "U411" (id 0) (at 181.61 113.03 0))
+    (property "Reference" "U435" (id 0) (at 181.61 113.03 0))
     (property "Value" "74HCT08" (id 1) (at 181.61 115.57 0))
     (property "Footprint" "Package_SO:SOIC-14_3.9x8.7mm_P1.27mm" (id 2) (at 181.61 121.92 0)
@@
   (symbol (lib_id "74xx:74LS32") (at 123.19 41.91 0) (unit 5)
     (in_bom yes) (on_board yes) (fields_autoplaced)
-    (property "Reference" "U504" (id 0) (at 130.81 40.6399 0)
+    (property "Reference" "U430" (id 0) (at 130.81 40.6399 0)
       (effects (font (size 1.27 1.27)) (justify left))
     )
@@
   (symbol (lib_id "74xx:74HC00") (at 100.33 78.74 0) (unit 5)
     (in_bom yes) (on_board yes) (fields_autoplaced)
-    (property "Reference" "U498" (id 0) (at 107.95 77.4699 0)
+    (property "Reference" "U431" (id 0) (at 107.95 77.4699 0)
       (effects (font (size 1.27 1.27)) (justify left))
     )
@@
   (symbol (lib_id "74xx:74LS32") (at 123.19 78.74 0) (unit 5)
     (in_bom yes) (on_board yes) (fields_autoplaced)
-    (property "Reference" "U505" (id 0) (at 130.81 77.4699 0)
+    (property "Reference" "U434" (id 0) (at 130.81 77.4699 0)
       (effects (font (size 1.27 1.27)) (justify left))
     )
@@
   (symbol (lib_id "74xx:74LS32") (at 147.32 80.01 0) (unit 5)
     (in_bom yes) (on_board yes) (fields_autoplaced)
-    (property "Reference" "U406" (id 0) (at 154.94 78.7399 0)
+    (property "Reference" "U433" (id 0) (at 154.94 78.7399 0)
       (effects (font (size 1.27 1.27)) (justify left))
     )
@@
   (symbol (lib_id "74xx:74HC00") (at 123.19 118.11 0) (unit 5)
     (in_bom yes) (on_board yes) (fields_autoplaced)
-    (property "Reference" "U436" (id 0) (at 129.54 116.8399 0)
+    (property "Reference" "U426" (id 0) (at 129.54 116.8399 0)
       (effects (font (size 1.27 1.27)) (justify left))
     )
@@
   (symbol (lib_id "74xx:74HC00") (at 77.47 118.11 0) (unit 5)
     (in_bom yes) (on_board yes) (fields_autoplaced)
-    (property "Reference" "U497" (id 0) (at 85.09 116.8399 0)
+    (property "Reference" "U432" (id 0) (at 85.09 116.8399 0)
       (effects (font (size 1.27 1.27)) (justify left))
     )
@@
   (symbol (lib_id "74xx:74HC74") (at 77.47 41.91 0) (unit 3)
     (in_bom yes) (on_board yes) (fields_autoplaced)
-    (property "Reference" "U429" (id 0) (at 83.82 40.6399 0)
-      (effects (font (size 1.27 1.27)) (justify left))
-    )
+    (property "Reference" "U436" (id 0) (at 83.82 40.6399 0)
+      (effects (font (size 1.27 1.27)) (justify left))
+    )
