File: B4/todSeconds.kicad_sch (KiCad schematic)
At the start: 3 parts, among them U416 74HC193, U417 74HC193, U418 74HC08

Commit message: TOD is here
Connections:
- net MIN_TK: now also U418.3; no longer U418.6
- net S1: now also U418.13; no longer U418.1
- net S3: now also U418.12; no longer U418.2
- net S5: now also U418.1; no longer U418.4
- net S6: now also U418.2; no longer U418.5
- net at U416.14 (CLR), U417.5 (UP): now also U418.11; no longer U418.3
Changed lines of the file:
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@@
     (effects (font (size 1.27 1.27)) (justify left))
   )
-  (symbol (lib_id "Custom 74xx:74HC08") (at 177.8 144.78 0) (unit 2)
+  (symbol (lib_id "Custom 74xx:74HC08") (at 177.8 144.78 0) (unit 1)
     (in_bom yes) (on_board yes) (fields_autoplaced)
     (property "Reference" "U418" (id 0) (at 177.8 135.89 0))
@@
     (pin "9")
   )
-  (symbol (lib_id "Custom 74xx:74HC08") (at 177.8 77.47 0) (unit 1)
+  (symbol (lib_id "Custom 74xx:74HC08") (at 177.8 77.47 0) (mirror x) (unit 4)
     (in_bom yes) (on_board yes) (fields_autoplaced)
     (property "Reference" "U418" (id 0) (at 177.8 68.58 0))
@@
       (effects (font (size 1.27 1.27)) hide)
     )
-    (property "Datasheet" "" (id 3) (at 177.8 71.12 0)
+    (property "Datasheet" "" (id 3) (at 177.8 83.82 0)
       (effects (font (size 1.27 1.27)) hide)
     )

Commit message: Ready for v0.2.2
Parts:
- renumbered U418 to U407, U417 to U409, U416 to U410
Other:
- company: (none) -> Daniel Molina
- title: (none) -> 74HCT6526 Board 4
Changed lines of the file:
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@@
 (kicad_sch (version 20211123) (generator eeschema)
   (paper "A4")
+  (title_block
+    (title "74HCT6526 Board 4")
+    (date "2023-06-22")
+    (rev "0.2.2")
+    (company "Daniel Molina")
+    (comment 1 "https://github.com/dmolinagarcia/74HCT6526")
+  )
   (junction (at 190.5 144.78) (diameter 0) (color 0 0 0 0)
   )
@@
   (symbol (lib_id "Custom 74xx:74HC08") (at 177.8 144.78 0) (unit 1)
     (in_bom yes) (on_board yes) (fields_autoplaced)
-    (property "Reference" "U418" (id 0) (at 177.8 135.89 0))
+    (property "Reference" "U407" (id 0) (at 177.8 135.89 0))
     (property "Value" "74HC08" (id 1) (at 177.8 138.43 0))
     (property "Footprint" "Package_SO:SOIC-14_3.9x8.7mm_P1.27mm" (id 2) (at 177.8 144.78 0)
@@
   (symbol (lib_id "74xx:74LS193") (at 106.68 116.84 0) (unit 1)
     (in_bom yes) (on_board yes) (fields_autoplaced)
-    (property "Reference" "U417" (id 0) (at 108.6994 99.06 0)
+    (property "Reference" "U409" (id 0) (at 108.6994 99.06 0)
       (effects (font (size 1.27 1.27)) (justify left))
     )
@@
   (symbol (lib_id "74xx:74LS193") (at 106.68 52.07 0) (unit 1)
     (in_bom yes) (on_board yes) (fields_autoplaced)
-    (property "Reference" "U416" (id 0) (at 108.6994 34.29 0)
+    (property "Reference" "U410" (id 0) (at 108.6994 34.29 0)
       (effects (font (size 1.27 1.27)) (justify left))
     )
@@
   (symbol (lib_id "Custom 74xx:74HC08") (at 177.8 77.47 0) (mirror x) (unit 4)
     (in_bom yes) (on_board yes) (fields_autoplaced)
-    (property "Reference" "U418" (id 0) (at 177.8 68.58 0))
+    (property "Reference" "U407" (id 0) (at 177.8 68.58 0))
     (property "Value" "74HC08" (id 1) (at 177.8 71.12 0))
     (property "Footprint" "Package_SO:SOIC-14_3.9x8.7mm_P1.27mm" (id 2) (at 177.8 77.47 0)
