File: B4/todTenths.kicad_sch (KiCad schematic)
At the start: 6 parts, among them U403 74HC04, U411 74HC08, U412 74HC193, U413 74HC193, U414 74HC11, U415 74HC32

Commit message: TOD is here
Parts:
- removed U411: 74HC08, Package_SO:SOIC-14_3.9x8.7mm_P1.27mm, symbol Custom 74xx:74HC08
- added unit 3 of U414
- renumbered U412 to U402, U413 to U403, U403 to U503
Connections:
- net SEC_TK: now also U414.6
- net T5: now also U414.3, U414.4
- net T7: now also U414.5
- net TODIN: now also U414.11; no longer U414.5
- net at U415.2: now also U414.8; no longer U414.6
- net TODBUS1: now reaches U402.2 (QB)
- net TODBUS1: now also U414.13; no longer U414.2
- net TODBUS0: now reaches U402.3 (QA)
- net TODBUS0: now also U414.10; no longer U414.4
- new net TODBUS2: U402.6 (QC), U414.2, U414.9
Other:
- moved on the sheet: U414B
Changed lines of the file:
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@@
 (kicad_sch (version 20211123) (generator eeschema)
   (paper "A4")
+  (junction (at 173.99 132.08) (diameter 0) (color 0 0 0 0)
+  )
   (junction (at 101.6 39.37) (diameter 0) (color 0 0 0 0)
   )
@@
   (junction (at 101.6 44.45) (diameter 0) (color 0 0 0 0)
   )
-  (junction (at 171.45 62.23) (diameter 0) (color 0 0 0 0)
-  )
   (junction (at 90.17 57.15) (diameter 0) (color 0 0 0 0)
   )
@@
   )
   (junction (at 173.99 107.95) (diameter 0) (color 0 0 0 0)
+  )
+  (junction (at 171.45 59.69) (diameter 0) (color 0 0 0 0)
   )
   (junction (at 101.6 41.91) (diameter 0) (color 0 0 0 0)
@@
     (stroke (width 0) (type default) (color 0 0 0 0))
   )
-  (wire (pts (xy 171.45 62.23) (xy 171.45 41.91))
+  (wire (pts (xy 171.45 41.91) (xy 171.45 59.69))
+    (stroke (width 0) (type default) (color 0 0 0 0))
+  )
+  (wire (pts (xy 168.91 36.83) (xy 168.91 77.47))
     (stroke (width 0) (type default) (color 0 0 0 0))
   )
@@
     (stroke (width 0) (type default) (color 0 0 0 0))
   )
-  (wire (pts (xy 176.53 62.23) (xy 171.45 62.23))
+  (wire (pts (xy 171.45 74.93) (xy 176.53 74.93))
     (stroke (width 0) (type default) (color 0 0 0 0))
   )
@@
     (stroke (width 0) (type default) (color 0 0 0 0))
   )
+  (wire (pts (xy 171.45 59.69) (xy 176.53 59.69))
+    (stroke (width 0) (type default) (color 0 0 0 0))
+  )
   (wire (pts (xy 148.59 80.01) (xy 176.53 80.01))
     (stroke (width 0) (type default) (color 0 0 0 0))
@@
     (stroke (width 0) (type default) (color 0 0 0 0))
   )
+  (wire (pts (xy 173.99 62.23) (xy 176.53 62.23))
+    (stroke (width 0) (type default) (color 0 0 0 0))
+  )
   (wire (pts (xy 171.45 113.03) (xy 227.33 113.03))
     (stroke (width 0) (type default) (color 0 0 0 0))
@@
     (stroke (width 0) (type default) (color 0 0 0 0))
   )
-  (wire (pts (xy 176.53 74.93) (xy 171.45 74.93))
-    (stroke (width 0) (type default) (color 0 0 0 0))
-  )
   (wire (pts (xy 101.6 44.45) (xy 106.68 44.45))
     (stroke (width 0) (type default) (color 0 0 0 0))
@@
     (stroke (width 0) (type default) (color 0 0 0 0))
   )
-  (wire (pts (xy 168.91 77.47) (xy 168.91 36.83))
-    (stroke (width 0) (type default) (color 0 0 0 0))
-  )
-  (wire (pts (xy 176.53 77.47) (xy 168.91 77.47))
+  (wire (pts (xy 171.45 59.69) (xy 171.45 74.93))
     (stroke (width 0) (type default) (color 0 0 0 0))
   )
@@
     (stroke (width 0) (type default) (color 0 0 0 0))
   )
+  (wire (pts (xy 173.99 134.62) (xy 176.53 134.62))
+    (stroke (width 0) (type default) (color 0 0 0 0))
+  )
   (bus (pts (xy 97.79 107.95) (xy 97.79 110.49))
     (stroke (width 0) (type default) (color 0 0 0 0))
@@
     (stroke (width 0) (type default) (color 0 0 0 0))
   )
-  (wire (pts (xy 173.99 59.69) (xy 173.99 39.37))
-    (stroke (width 0) (type default) (color 0 0 0 0))
-  )
-  (wire (pts (xy 171.45 74.93) (xy 171.45 62.23))
+  (wire (pts (xy 173.99 39.37) (xy 173.99 62.23))
     (stroke (width 0) (type default) (color 0 0 0 0))
   )
@@
     (stroke (width 0) (type default) (color 0 0 0 0))
   )
+  (wire (pts (xy 173.99 132.08) (xy 173.99 134.62))
+    (stroke (width 0) (type default) (color 0 0 0 0))
+  )
   (wire (pts (xy 173.99 107.95) (xy 227.33 107.95))
     (stroke (width 0) (type default) (color 0 0 0 0))
@@
     (stroke (width 0) (type default) (color 0 0 0 0))
   )
+  (wire (pts (xy 168.91 77.47) (xy 176.53 77.47))
+    (stroke (width 0) (type default) (color 0 0 0 0))
+  )
   (wire (pts (xy 100.33 107.95) (xy 106.68 107.95))
     (stroke (width 0) (type default) (color 0 0 0 0))
@@
     (stroke (width 0) (type default) (color 0 0 0 0))
   )
-  (wire (pts (xy 176.53 59.69) (xy 173.99 59.69))
-    (stroke (width 0) (type default) (color 0 0 0 0))
-  )
   (wire (pts (xy 100.33 105.41) (xy 106.68 105.41))
     (stroke (width 0) (type default) (color 0 0 0 0))
@@
     (effects (font (size 1.27 1.27)) (justify left bottom))
   )
+  (label "TODBUS0" (at 146.05 36.83 0)
+    (effects (font (size 1.27 1.27)) (justify left bottom))
+  )
+  (label "TODBUS2" (at 146.05 41.91 0)
+    (effects (font (size 1.27 1.27)) (justify left bottom))
+  )
   (label "DZ2" (at 102.87 110.49 0)
+    (effects (font (size 1.27 1.27)) (justify left bottom))
+  )
+  (label "TODBUS1" (at 146.05 39.37 0)
     (effects (font (size 1.27 1.27)) (justify left bottom))
   )
@@
     )
     (pin "1")
-  )
-  (symbol (lib_id "Custom 74xx:74HC08") (at 184.15 134.62 0) (unit 2)
-    (in_bom yes) (on_board yes) (fields_autoplaced)
-    (property "Reference" "U411" (id 0) (at 184.15 125.73 0))
-    (property "Value" "74HC08" (id 1) (at 184.15 128.27 0))
-    (property "Footprint" "Package_SO:SOIC-14_3.9x8.7mm_P1.27mm" (id 2) (at 184.15 134.62 0)
-      (effects (font (size 1.27 1.27)) hide)
-    )
-    (property "Datasheet" "" (id 3) (at 184.15 128.27 0)
-      (effects (font (size 1.27 1.27)) hide)
-    )
-    (pin "1")
-    (pin "2")
-    (pin "3")
-    (pin "4")
-    (pin "5")
-    (pin "6")
-    (pin "10")
-    (pin "8")
-    (pin "9")
-    (pin "11")
-    (pin "12")
-    (pin "13")
-    (pin "14")
-    (pin "7")
   )
   (symbol (lib_id "power:GND") (at 101.6 44.45 0) (unit 1)
@@
   (symbol (lib_id "74xx:74LS193") (at 119.38 115.57 0) (unit 1)
     (in_bom yes) (on_board yes)
-    (property "Reference" "U413" (id 0) (at 121.3994 97.79 0)
+    (property "Reference" "U403" (id 0) (at 121.3994 97.79 0)
       (effects (font (size 1.27 1.27)) (justify left))
     )
@@
   (symbol (lib_id "74xx:74HC04") (at 157.48 57.15 0) (unit 3)
     (in_bom yes) (on_board yes) (fields_autoplaced)
-    (property "Reference" "U403" (id 0) (at 157.48 48.26 0))
+    (property "Reference" "U503" (id 0) (at 157.48 48.26 0))
     (property "Value" "74HC04" (id 1) (at 157.48 50.8 0))
     (property "Footprint" "Package_SO:SOIC-14_3.9x8.7mm_P1.27mm" (id 2) (at 157.48 57.15 0)
@@
   (symbol (lib_id "74xx:74LS193") (at 119.38 46.99 0) (unit 1)
     (in_bom yes) (on_board yes) (fields_autoplaced)
-    (property "Reference" "U412" (id 0) (at 121.3994 30.48 0)
+    (property "Reference" "U402" (id 0) (at 121.3994 30.48 0)
       (effects (font (size 1.27 1.27)) (justify left))
     )
@@
     (pin "9")
   )
-  (symbol (lib_id "74xx:74LS11") (at 184.15 59.69 0) (unit 1)
-    (in_bom yes) (on_board yes) (fields_autoplaced)
-    (property "Reference" "U414" (id 0) (at 184.15 50.8 0))
-    (property "Value" "74HC11" (id 1) (at 184.15 53.34 0))
-    (property "Footprint" "Package_SO:SOIC-14_3.9x8.7mm_P1.27mm" (id 2) (at 184.15 59.69 0)
-      (effects (font (size 1.27 1.27)) hide)
-    )
-    (property "Datasheet" "http://www.ti.com/lit/gpn/sn74LS11" (id 3) (at 184.15 59.69 0)
+  (symbol (lib_id "74xx:74LS11") (at 184.15 77.47 0) (unit 3)
+    (in_bom yes) (on_board yes) (fields_autoplaced)
+    (property "Reference" "U414" (id 0) (at 184.15 68.58 0))
+    (property "Value" "74HC11" (id 1) (at 184.15 71.12 0))
+    (property "Footprint" "Package_SO:SOIC-14_3.9x8.7mm_P1.27mm" (id 2) (at 184.15 77.47 0)
+      (effects (font (size 1.27 1.27)) hide)
+    )
+    (property "Datasheet" "http://www.ti.com/lit/gpn/sn74LS11" (id 3) (at 184.15 77.47 0)
       (effects (font (size 1.27 1.27)) hide)
     )
@@
     (pin "7")
   )
+  (symbol (lib_id "74xx:74LS11") (at 184.15 59.69 0) (unit 1)
+    (in_bom yes) (on_board yes) (fields_autoplaced)
+    (property "Reference" "U414" (id 0) (at 184.15 50.8 0))
+    (property "Value" "74HC11" (id 1) (at 184.15 53.34 0))
+    (property "Footprint" "Package_SO:SOIC-14_3.9x8.7mm_P1.27mm" (id 2) (at 184.15 59.69 0)
+      (effects (font (size 1.27 1.27)) hide)
+    )
+    (property "Datasheet" "http://www.ti.com/lit/gpn/sn74LS11" (id 3) (at 184.15 59.69 0)
+      (effects (font (size 1.27 1.27)) hide)
+    )
+    (pin "1")
+    (pin "12")
+    (pin "13")
+    (pin "2")
+    (pin "3")
+    (pin "4")
+    (pin "5")
+    (pin "6")
+    (pin "10")
+    (pin "11")
+    (pin "8")
+    (pin "9")
+    (pin "14")
+    (pin "7")
+  )
   (symbol (lib_id "power:GND") (at 119.38 67.31 0) (unit 1)
     (in_bom yes) (on_board yes) (fields_autoplaced)
@@
     (pin "1")
   )
-  (symbol (lib_id "74xx:74LS11") (at 184.15 77.47 0) (unit 2)
-    (in_bom yes) (on_board yes) (fields_autoplaced)
-    (property "Reference" "U414" (id 0) (at 184.15 68.58 0))
-    (property "Value" "74HC11" (id 1) (at 184.15 71.12 0))
-    (property "Footprint" "Package_SO:SOIC-14_3.9x8.7mm_P1.27mm" (id 2) (at 184.15 77.47 0)
-      (effects (font (size 1.27 1.27)) hide)
-    )
-    (property "Datasheet" "http://www.ti.com/lit/gpn/sn74LS11" (id 3) (at 184.15 77.47 0)
-      (effects (font (size 1.27 1.27)) hide)
-    )
+  (symbol (lib_id "74xx:74LS11") (at 184.15 134.62 0) (unit 2)
+    (in_bom yes) (on_board yes) (fields_autoplaced)
+    (property "Reference" "U414" (id 0) (at 184.15 125.73 0))
+    (property "Value" "74HC11" (id 1) (at 184.15 128.27 0))
+    (property "Footprint" "Package_SO:SOIC-14_3.9x8.7mm_P1.27mm" (id 2) (at 184.15 134.62 0)
+      (effects (font (size 1.27 1.27)) hide)
+    )
+    (property "Datasheet" "http://www.ti.com/lit/gpn/sn74LS11" (id 3) (at 184.15 134.62 0)
+      (effects (font (size 1.27 1.27)) hide)
+    )

Commit message: Ready for v0.2.2
Parts:
- renumbered U414 to U401, U402 to U403, U403 to U404, U415 to U418, U503 to U429
Other:
- company: (none) -> Daniel Molina
- title: (none) -> 74HCT6526 Board 4
Changed lines of the file:
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@@
 (kicad_sch (version 20211123) (generator eeschema)
   (paper "A4")
+  (title_block
+    (title "74HCT6526 Board 4")
+    (date "2023-06-22")
+    (rev "0.2.2")
+    (company "Daniel Molina")
+    (comment 1 "https://github.com/dmolinagarcia/74HCT6526")
+  )
   (junction (at 173.99 132.08) (diameter 0) (color 0 0 0 0)
   )
@@
   (symbol (lib_id "74xx:74LS193") (at 119.38 115.57 0) (unit 1)
     (in_bom yes) (on_board yes)
-    (property "Reference" "U403" (id 0) (at 121.3994 97.79 0)
+    (property "Reference" "U404" (id 0) (at 121.3994 97.79 0)
       (effects (font (size 1.27 1.27)) (justify left))
     )
@@
   (symbol (lib_id "74xx:74HC04") (at 157.48 57.15 0) (unit 3)
     (in_bom yes) (on_board yes) (fields_autoplaced)
-    (property "Reference" "U503" (id 0) (at 157.48 48.26 0))
+    (property "Reference" "U429" (id 0) (at 157.48 48.26 0))
     (property "Value" "74HC04" (id 1) (at 157.48 50.8 0))
     (property "Footprint" "Package_SO:SOIC-14_3.9x8.7mm_P1.27mm" (id 2) (at 157.48 57.15 0)
@@
   (symbol (lib_id "74xx:74LS32") (at 209.55 68.58 0) (unit 1)
     (in_bom yes) (on_board yes) (fields_autoplaced)
-    (property "Reference" "U415" (id 0) (at 209.55 59.69 0))
+    (property "Reference" "U418" (id 0) (at 209.55 59.69 0))
     (property "Value" "74HC32" (id 1) (at 209.55 62.23 0))
     (property "Footprint" "Package_SO:SOIC-14_3.9x8.7mm_P1.27mm" (id 2) (at 209.55 68.58 0)
@@
   (symbol (lib_id "74xx:74LS193") (at 119.38 46.99 0) (unit 1)
     (in_bom yes) (on_board yes) (fields_autoplaced)
-    (property "Reference" "U402" (id 0) (at 121.3994 30.48 0)
+    (property "Reference" "U403" (id 0) (at 121.3994 30.48 0)
       (effects (font (size 1.27 1.27)) (justify left))
     )
@@
   (symbol (lib_id "74xx:74LS11") (at 184.15 77.47 0) (unit 3)
     (in_bom yes) (on_board yes) (fields_autoplaced)
-    (property "Reference" "U414" (id 0) (at 184.15 68.58 0))
+    (property "Reference" "U401" (id 0) (at 184.15 68.58 0))
     (property "Value" "74HC11" (id 1) (at 184.15 71.12 0))
     (property "Footprint" "Package_SO:SOIC-14_3.9x8.7mm_P1.27mm" (id 2) (at 184.15 77.47 0)
@@
   (symbol (lib_id "74xx:74LS11") (at 184.15 59.69 0) (unit 1)
     (in_bom yes) (on_board yes) (fields_autoplaced)
-    (property "Reference" "U414" (id 0) (at 184.15 50.8 0))
+    (property "Reference" "U401" (id 0) (at 184.15 50.8 0))
     (property "Value" "74HC11" (id 1) (at 184.15 53.34 0))
     (property "Footprint" "Package_SO:SOIC-14_3.9x8.7mm_P1.27mm" (id 2) (at 184.15 59.69 0)
@@
   (symbol (lib_id "74xx:74LS11") (at 184.15 134.62 0) (unit 2)
     (in_bom yes) (on_board yes) (fields_autoplaced)
-    (property "Reference" "U414" (id 0) (at 184.15 125.73 0))
+    (property "Reference" "U401" (id 0) (at 184.15 125.73 0))
     (property "Value" "74HC11" (id 1) (at 184.15 128.27 0))
     (property "Footprint" "Package_SO:SOIC-14_3.9x8.7mm_P1.27mm" (id 2) (at 184.15 134.62 0)
